Commit message: Rename packages

File: src/edna_description/urdf/parts/square_chassis.xacro (robot description, xacro)
@@ -15,5 +15,5 @@
         <origin xyz="0.061605 -0.34976 -0.53866" rpy="0 0 0" />
         <geometry>
-          <mesh filename="package://swerve_description/meshes/SwerveChassis.stl" scale="0.001 0.001 0.001" />
+          <mesh filename="package://edna_description/meshes/SwerveChassis.stl" scale="0.001 0.001 0.001" />
         </geometry>
         <material name="red"/>

File: src/edna_description/urdf/parts/swerve_axle.xacro (robot description, xacro)
@@ -18,5 +18,5 @@
                 <origin xyz="0 0 0" rpy="0 0 0" />
                 <geometry>
-                    <mesh filename="package://swerve_description/meshes/SwerveAxle.stl" scale="0.001 0.001 0.001" />
+                    <mesh filename="package://edna_description/meshes/SwerveAxle.stl" scale="0.001 0.001 0.001" />
                 </geometry>
                 <material name="blue" />
@@ -37,5 +37,5 @@
                 <origin xyz="0 0 0" rpy="0 ${pi / 4} 0" />
                 <geometry>
-                    <mesh filename="package://swerve_description/meshes/SwerveWheel.stl" scale="0.001 0.001 0.001" />
+                    <mesh filename="package://edna_description/meshes/SwerveWheel.stl" scale="0.001 0.001 0.001" />
                 </geometry>
                 <material name="yellow" />

File: src/edna_description/urdf/robots/edna.urdf.xacro (robot description, xacro)
@@ -1,12 +1,12 @@
 <?xml version="1.0"?>
-<robot name="swerve" xmlns:xacro="http://www.ros.org/wiki/xacro">
+<robot name="edna" xmlns:xacro="http://www.ros.org/wiki/xacro">
   <!-- Args -->
   <xacro:arg name="hw_interface_plugin" default="swerve_hardware/IsaacDriveHardware"/>
   <!-- Include Files -->
-  <xacro:include filename="$(find swerve_description)/urdf/control/drive.xacro" />
-  <xacro:include filename="$(find swerve_description)/urdf/util/macros.xacro" />
-  <xacro:include filename="$(find swerve_description)/urdf/util/materials.xacro" />
-  <xacro:include filename="$(find swerve_description)/urdf/parts/square_chassis.xacro" />
-  <xacro:include filename="$(find swerve_description)/urdf/parts/swerve_axle.xacro" />
+  <xacro:include filename="$(find edna_description)/urdf/control/drive.xacro" />
+  <xacro:include filename="$(find edna_description)/urdf/util/macros.xacro" />
+  <xacro:include filename="$(find edna_description)/urdf/util/materials.xacro" />
+  <xacro:include filename="$(find edna_description)/urdf/parts/square_chassis.xacro" />
+  <xacro:include filename="$(find edna_description)/urdf/parts/swerve_axle.xacro" />
     <!-- Axle Position Variables -->
     <xacro:property name="axle_pos" value="${301.625 / 1000}" />

Commit message: Fix urdf and controller output

File: src/edna_description/urdf/parts/square_chassis.xacro (robot description, xacro)
@@ -10,8 +10,8 @@
     <link name="${prefix}_chassis_link">
       <xacro:inertial_box mass="${chassis_weight}" x="${chassis_length}" y="${chassis_width}" z="${chassis_height}">
-        <origin xyz="0 0 0" rpy="0 0 0" />
+        <origin xyz="0 0 ${chassis_height/2}" rpy="0 0 0" />
       </xacro:inertial_box>
       <visual>
-        <origin xyz="0.061605 -0.34976 -0.53866" rpy="0 0 0" />
+        <origin xyz="0.061605 0.53866 -0.34976" rpy="${pi / 2} 0 0" />
         <geometry>
           <mesh filename="package://edna_description/meshes/SwerveChassis.stl" scale="0.001 0.001 0.001" />
@@ -20,7 +20,7 @@
       </visual>
       <collision>
-        <origin xyz="0 ${chassis_height/2} 0" rpy="0 0 0" />
+        <origin xyz="0 0 ${chassis_height/2}" rpy="0 0 0" />
         <geometry>
-          <box size="${chassis_length} ${chassis_height} ${chassis_width}" />
+          <box size="${chassis_length} ${chassis_width} ${chassis_height} " />
         </geometry>
       </collision>
@@ -29,5 +29,5 @@
       <parent link="base_link" />
       <child link="${prefix}_chassis_link" />
-      <origin xyz="0 0 0" rpy="${pi / 2} 0 0" />
+      <origin xyz="0 0 0" rpy="0 0 0" />
     </joint>
   </xacro:macro>

File: src/edna_description/urdf/parts/swerve_axle.xacro (robot description, xacro)
@@ -2,6 +2,6 @@
 <robot xmlns:xacro="http://www.ros.org/wiki/xacro">
     <!-- Chassis Properties -->
-    <xacro:property name="axle_radius" value="0.075" />
-    <xacro:property name="axle_length" value=".1" />
+    <xacro:property name="axle_radius" value="0.05" />
+    <xacro:property name="axle_length" value="0.03" />
     <xacro:property name="axle_mass" value="0.23739" />
     <xacro:property name="wheel_radius" value="0.0508" />
@@ -11,10 +11,10 @@
     <!-- NOTE: The below values are **guesses**-->
     <!-- NOTE: Pretty good **guesses**-->
-    <xacro:property name="wheel_pos_x" value="-0.022"/>
-    <xacro:property name="wheel_pos_y" value="0.065"/>
+    <xacro:property name="wheel_pos_y" value="0.022"/>
+    <xacro:property name="wheel_pos_z" value="0.063"/>
     <xacro:macro name="swerve_axle" params="prefix parent *origin">
         <link name="${prefix}_axle_link">
             <visual>
-                <origin xyz="0 0 0" rpy="0 0 0" />
+                <origin xyz="0 0 0" rpy="${pi} 0 ${pi/2}" />
                 <geometry>
                     <mesh filename="package://edna_description/meshes/SwerveAxle.stl" scale="0.001 0.001 0.001" />
@@ -22,6 +22,6 @@
                 <material name="blue" />
             </visual>
-            <xacro:inertial_cylinder mass="${axle_mass}" radius="${axle_radius}" length="${wheel_length}" >
-                <origin xyz="0 0 0" rpy="0 0 0" />
+            <xacro:inertial_cylinder mass="${axle_mass}" radius="${axle_radius}" length="${axle_length}" >
+                <origin xyz="0 0 -${axle_length/2}" rpy="0 0 0" />
             </xacro:inertial_cylinder>
         </link>
@@ -35,5 +35,5 @@
         <link name="${prefix}_wheel_link">
             <visual>
-                <origin xyz="0 0 0" rpy="0 ${pi / 4} 0" />
+                <origin xyz="0 -${wheel_pos_y} 0" rpy="0 ${pi/4} ${pi/2}" />
                 <geometry>
                     <mesh filename="package://edna_description/meshes/SwerveWheel.stl" scale="0.001 0.001 0.001" />
@@ -42,5 +42,5 @@
             </visual>
             <collision>
-                <origin xyz="0.021 0 0" rpy="0 ${pi / 2} 0"/>
+                <origin xyz="0 0 0" rpy="${pi / 2} 0 0"/>
                 <geometry>
                     <cylinder  length="${wheel_length}" radius="${wheel_radius}"/>
@@ -48,5 +48,5 @@
             </collision>
             <xacro:inertial_cylinder mass="${wheel_mass}" radius="${wheel_radius}" length="${wheel_length}" >
-                <origin xyz="0 0 0" rpy="0 ${pi / 2} 0" />
+                <origin xyz="0 0 0" rpy="${pi / 2} 0 0" />
             </xacro:inertial_cylinder>
         </link>
@@ -54,6 +54,6 @@
             <parent link="${prefix}_axle_link" />
             <child link="${prefix}_wheel_link" />
-            <origin xyz="${wheel_pos_x} 0 ${wheel_pos_y}" rpy="0 0 0"/>
-            <axis xyz="1 0 0" />
+            <origin xyz="0 0 -${wheel_pos_z}" rpy="0 0 0"/>
+            <axis xyz="0 1 0" />
             <dynamics friction="0.1" />
         </joint>

File: src/edna_description/urdf/robots/edna.urdf.xacro (robot description, xacro)
@@ -11,19 +11,22 @@
   <!-- Axle Position Variables -->
   <xacro:property name="axle_pos" value="${301.625 / 1000}" />
-  <xacro:property name="axle_pos_y" value="${69.056 / 1000}" />
+  <xacro:property name="axle_pos_z" value="${69.056 / 1000}" />
   <!-- Camera Position Variables -->
   <xacro:property name="cam_pos" value=".3575 0.085 0.0"/> <!-- Made up values, replace with real ones later. -->
+  <!-- X IS FORWARD -->
+  <!-- Y IS LEFT -->
+  <!-- Z IS UP -->
   <xacro:square_chassis prefix="swerve" />
   <xacro:swerve_axle prefix="front_left" parent="swerve_chassis_link">
-    <origin xyz="${axle_pos} ${axle_pos_y} ${axle_pos}" rpy="${pi / 2} 0 0" />
+    <origin xyz="${axle_pos} ${axle_pos} ${axle_pos_z}" rpy="0 0 0" />
   </xacro:swerve_axle>
   <xacro:swerve_axle prefix="front_right" parent="swerve_chassis_link">
-    <origin xyz="-${axle_pos} ${axle_pos_y} ${axle_pos}" rpy="${pi / 2} 0 0" />
+    <origin xyz="${axle_pos} -${axle_pos} ${axle_pos_z}" rpy="0 0 0" />
   </xacro:swerve_axle>
   <xacro:swerve_axle prefix="rear_left" parent="swerve_chassis_link">
-    <origin xyz="${axle_pos} ${axle_pos_y} -${axle_pos}" rpy="${pi / 2} 0 0" />
+    <origin xyz="-${axle_pos} ${axle_pos} ${axle_pos_z} " rpy="0 0 0" />
   </xacro:swerve_axle>
   <xacro:swerve_axle prefix="rear_right" parent="swerve_chassis_link">
-    <origin xyz="-${axle_pos} ${axle_pos_y} -${axle_pos}" rpy="${pi / 2} 0 0" />
+    <origin xyz="-${axle_pos} -${axle_pos} ${axle_pos_z}" rpy="0 0 0" />
   </xacro:swerve_axle>
   <!-- <xacro:zed_camera name="zed_camera" model="zed2i" parent="swerve_chassis_link">
