Commit message: remove more files cuz why not

File: src/edna_description/urdf/parts/arm.xacro (robot description, xacro)
@@ -4,6 +4,6 @@
     <xacro:property name="arm_link1_width" value="1" />
     <xacro:property name="arm_link1_height" value="1" />
-    <xacro:macro name = "arm" params = "prefix">
-        <link name = "${prefix}_box">
+    <xacro:macro name = "arm" params = "prefix parent *origin">
+        <link name = "${prefix}_link">
             <xacro:inertial_box mass = "1" x = "${arm_link1_length}" y = "${arm_link1_width}" z = "${arm_link1_height}">
                 <origin xyz="0 0 0" rpy="0 0 0" />
@@ -24,7 +24,7 @@
         </link>
         <joint name = "${prefix}_box_joint" type = "fixed">
-            <parent link = "${prefix}_chassis_link"/>
-            <child link = "${prefix}_box"/>
-            <origin xyz = "0 0 0" rpy = "0 0 0"/>
+            <parent link = "${parent}"/>
+            <child link = "${prefix}_link"/>
+            <xacro:insert_block name = "origin"/>
         </joint>
     </xacro:macro>

File: src/edna_description/urdf/robots/edna.urdf.xacro (robot description, xacro)
@@ -10,4 +10,5 @@
   <xacro:include filename="$(find edna_description)/urdf/parts/swerve_axle.xacro" />
   <xacro:include filename="$(find edna_description)/urdf/parts/zed_macro.urdf.xacro" />
+  <xacro:include filename="$(find edna_description)/urdf/parts/arm.xacro" />
   <!-- Axle Position Variables -->
   <xacro:property name="axle_pos" value="${301.625 / 1000}" />
@@ -41,3 +42,6 @@
   </xacro:zed_camera>
   <xacro:swerve_drive_control plugin="$(arg hw_interface_plugin)" />
+  <xacro:arm prefix="arm" parent="swerve_chassis_link">
+    <origin xyz="0 0 0" rpy="0 0 0" />
+  </xacro:arm>
 </robot>
