Commit message: urdf fixes

File: src/edna_description/urdf/parts/elevator.xacro (robot description, xacro)
@@ -14,5 +14,5 @@
             </xacro:inertial_box>
             <visual>
-                <origin xyz = "0.254264 -0.006 -0.072" rpy = "0 0 0"/>
+                <origin xyz = "0.254264 -0.07 -0.072" rpy = "0 0 0"/>
                 <geometry>
                     <mesh filename="package://edna_description/meshes/elevator_outer_updated.stl" scale="0.001 0.001 0.001"/>
@@ -32,5 +32,5 @@
             <axis xyz = "0 -1 0"/>
             <limit effort="1000.0" lower="0.0" upper="0.548" velocity="0.5"/>
-            <mimic joint = "${ns}_arm_roller_bar_joint" multiplier = "-1.8" offset = "0"/>
+            <!-- <mimic joint = "${ns}_arm_roller_bar_joint" multiplier = "-1.8" offset = "0"/> -->
             <xacro:insert_block name = "origin"/>
         </joint>
@@ -40,5 +40,5 @@
             </xacro:inertial_box>
             <visual>
-                <origin xyz = "0.365 0.066 -0.085" rpy = "0 0 0"/>
+                <origin xyz = "0.365 0.004 -0.085" rpy = "0 0 0"/>
                 <geometry>
                     <mesh filename="package://edna_description/meshes/elevator_center.stl" scale="0.001 0.001 0.001"/>
@@ -66,5 +66,5 @@
             </xacro:inertial_box>
             <visual>
-                <origin xyz = "0.469 -0.006 -0.1" rpy = "0 ${pi} 0"/>
+                <origin xyz = "0.469 -0.07 -0.1" rpy = "0 ${pi} 0"/>
                 <geometry>
                     <mesh filename="package://edna_description/meshes/elevator_outer_updated.stl" scale="0.001 0.001 0.001"/>

File: src/edna_description/urdf/parts/elevator_leg.xacro (robot description, xacro)
@@ -36,5 +36,5 @@
             </xacro:inertial_box>
             <visual>
-                <origin xyz = "0 0 0" rpy = "0 0 0"/>
+                <origin xyz = "0 -${roller_bar_height/2} 0" rpy = "0 0 0"/>
                 <geometry>
                     <mesh filename="package://edna_description/meshes/Roller_Bar.stl" scale="0.001 0.001 0.001"/>
@@ -53,5 +53,5 @@
             <child link = "${prefix}_roller_bar_link"/>
             <axis xyz = "0 1 0"/>
-            <limit effort = "100.0" lower = "0" upper = "0.06985" velocity = "0.5"/>
+            <limit effort = "100.0" lower = "-1" upper = "0.06985" velocity = "0.5"/>
             <xacro:insert_block name = "origin2"/>
         </joint>

File: src/edna_description/urdf/robots/edna.urdf.xacro (robot description, xacro)
@@ -47,21 +47,24 @@
   </xacro:zed_camera>
   <xacro:elevator_leg prefix="${ns}_arm" parent="${ns}_swerve_chassis_link">
-    <origin xyz = "-0.1905 0 ${0.527/2 + 0.03}" rpy = "0 0 ${pi}"/>
-    <origin xyz = "0 0 ${0.527/5 + 0.01}" rpy = "${pi/2} 0 0"/>
+    <origin xyz = "0.1905 0 ${0.527/2 + 0.03}" rpy = "0 0 ${pi}"/>
+    <origin xyz = "0 0 ${0.37}" rpy = "${pi/2} 0 0"/>
   </xacro:elevator_leg>
   <xacro:back_leg prefix="${ns}_arm" parent="${ns}_swerve_chassis_link">
-    <origin xyz = "${0.7366/2 - 0.0508/2} 0 ${back_leg_height/2 + 0.05588}" rpy = "0 0 ${pi}" />
+    <origin xyz = "-${0.7366/2 - 0.0508/2} 0 ${back_leg_height/2 + 0.05588}" rpy = "0 0 ${pi}" />
   </xacro:back_leg>
   <!--Right Elevator-->
   <xacro:elevator prefix="${ns}_elevator_right" parent="${ns}_arm_back_leg_link" ns="${ns}">
-    <origin xyz = "0.00253 -0.152 0.3738731" rpy = "${pi} ${(0.0174533*16.3)} 0" />
+    <origin xyz = "0.00253 0.28 0.3738731" rpy = "${pi} ${(0.0174533*15.3)} ${pi}" />
   </xacro:elevator>
+  <!-- <xacro:elevator prefix="${ns}_elevator_right" parent="base_link" ns="${ns}">
+    <origin xyz = "0.00253 0.28 0.3738731" rpy = "${pi} ${(0.0174533*15.3)} ${pi}" />
+  </xacro:elevator> -->
   <!--Left Elevator-->
   <xacro:elevator prefix="${ns}_elevator_left" parent="${ns}_arm_back_leg_link" ns="${ns}">
-    <origin xyz = "0.00253 0.28 0.3738731" rpy = "${pi} ${(0.0174533*16.3)} 0" />
+    <origin xyz = "0.00253 -0.28 0.3738731" rpy = "${pi} ${(0.0174533*15.3)} ${pi}" />
   </xacro:elevator>
   <xacro:lidar prefix="${ns}_lidar" parent="${ns}_swerve_chassis_link" radius="0.035" length="0.025">
     <origin xyz="0 0 .035" rpy="0 0 0" />
-  </xacro:lidar>
-  <xacro:swerve_drive_control plugin="$(arg hw_interface_plugin)" ns="${ns}"/>
+  </xacro:lidar> -->
+  <!-- <xacro:swerve_drive_control plugin="$(arg hw_interface_plugin)" ns="${ns}"/>
 </robot>

Commit message: urdf not dead

File: src/edna_description/urdf/parts/elevator.xacro (robot description, xacro)
@@ -32,5 +32,5 @@
             <axis xyz = "0 -1 0"/>
             <limit effort="1000.0" lower="0.0" upper="0.548" velocity="0.5"/>
-            <!-- <mimic joint = "${ns}_arm_roller_bar_joint" multiplier = "-1.8" offset = "0"/> -->
+            <mimic joint = "${ns}_arm_roller_bar_joint" multiplier = "-1.8" offset = "0"/>
             <xacro:insert_block name = "origin"/>
         </joint>

File: src/edna_description/urdf/robots/edna.urdf.xacro (robot description, xacro)
@@ -57,7 +57,4 @@
     <origin xyz = "0.00253 0.28 0.3738731" rpy = "${pi} ${(0.0174533*15.3)} ${pi}" />
   </xacro:elevator>
-  <!-- <xacro:elevator prefix="${ns}_elevator_right" parent="base_link" ns="${ns}">
-    <origin xyz = "0.00253 0.28 0.3738731" rpy = "${pi} ${(0.0174533*15.3)} ${pi}" />
-  </xacro:elevator> -->
   <!--Left Elevator-->
   <xacro:elevator prefix="${ns}_elevator_left" parent="${ns}_arm_back_leg_link" ns="${ns}">
@@ -66,5 +63,5 @@
   <xacro:lidar prefix="${ns}_lidar" parent="${ns}_swerve_chassis_link" radius="0.035" length="0.025">
     <origin xyz="0 0 .035" rpy="0 0 0" />
-  </xacro:lidar> -->
-  <!-- <xacro:swerve_drive_control plugin="$(arg hw_interface_plugin)" ns="${ns}"/>
+  </xacro:lidar>
+  <xacro:swerve_drive_control plugin="$(arg hw_interface_plugin)" ns="${ns}"/>
 </robot>
