Commit message: Collisions, Joint mimics

File: src/edna_description/urdf/parts/back_leg.xacro (robot description, xacro)
@@ -10,5 +10,5 @@
             </xacro:inertial_box>
             <visual>
-                <origin xyz = "0 0 0" rpy = "0 0 0"/>
+                <origin xyz = "0 0 0" rpy = "0 0 ${pi}"/>
                 <geometry>
                     <mesh filename="package://edna_description/meshes/back_legs.stl" scale="0.001 0.001 0.001"/>

File: src/edna_description/urdf/parts/elevator.xacro (robot description, xacro)
@@ -2,11 +2,15 @@
 <robot xmlns:xacro = "http://www.ros.org/wiki/xacro">
     <xacro:property name="elevator_outer_length" value="0.685" />
-    <xacro:property name="elevator_outer_width" value="0.457" />
-    <xacro:property name="elevator_outer_height" value="0.812" />
-    <xacro:property name="elevator_center_length" value="0.0508"/>
-    <xacro:property name="elevator_center_width" value="0.457"/>
-    <xacro:property name="elevator_center_height" value="0.812"/>
+    <xacro:property name="elevator_outer_width" value="0.025" />
+    <xacro:property name="elevator_outer_height" value="0.082" />
+    <xacro:property name="elevator_center_length" value="0.685"/>
+    <xacro:property name="elevator_center_width" value="0.025"/>
+    <xacro:property name="elevator_center_height" value="0.215"/>
+    <xacro:property name="elevator_center_offset_x" value="0.05"/>
+    <xacro:property name="elevator_center_offset_z" value="0.08"/>
+    <xacro:property name="elevator_outer_offset_x" value="0.04"/>
+    <xacro:property name="elevator_outer_offset_z" value="0.07"/>
     <xacro:include filename="$(find edna_description)/urdf/parts/elevator_leg.xacro" />
-    <xacro:macro name = "elevator" params = "ns prefix parent *origin">
+    <xacro:macro name = "elevator" params = "ns prefix parent *origin suffix">
         <link name = "${prefix}_elevator_outer_1_link">
             <xacro:inertial_box mass = "1" x = "${elevator_outer_length}" y = "${elevator_outer_width}" z = "${elevator_outer_height}">
@@ -14,14 +18,15 @@
             </xacro:inertial_box>
             <visual>
-                <origin xyz = "0.254264 -0.07 -0.072" rpy = "0 0 0"/>
+                <!-- <origin xyz = "0.254264 -0.07 -0.072" rpy = "${pi} 0 0"/> -->
+                <origin xyz = "${elevator_outer_length/2 - 0.08} 0.07 0.062" rpy = "${pi} 0 0"/>
                 <geometry>
                     <mesh filename="package://edna_description/meshes/elevator_outer_updated.stl" scale="0.001 0.001 0.001"/>
                 </geometry>
-                <material name = "blue"/>}
+                <material name = "blue"/>
             </visual>
             <collision>
-                <xacro:insert_block name = "origin"/>
+                <origin xyz = "${elevator_outer_length/2 - 0.0104} -0.0025 0.023" rpy = "0 0 0"/>
                 <geometry>
-                    <box size = "0.1 0.1 0.1"/>
+                    <box size = "${elevator_outer_length + 0.0004} ${elevator_outer_width + 0.0004} ${elevator_outer_height+0.002}"/>
                 </geometry>
             </collision>
@@ -32,5 +37,5 @@
             <axis xyz = "0 -1 0"/>
             <limit effort="1000.0" lower="0.0" upper="0.548" velocity="0.5"/>
-            <mimic joint = "${ns}_arm_roller_bar_joint" multiplier = "-1.8" offset = "0"/>
+            <mimic joint = "${ns}_arm_roller_bar_joint" multiplier = "1.8" offset = "0"/>
             <xacro:insert_block name = "origin"/>
         </joint>
@@ -40,5 +45,5 @@
             </xacro:inertial_box>
             <visual>
-                <origin xyz = "0.365 0.004 -0.085" rpy = "0 0 0"/>
+                <origin xyz = "${0.265+elevator_center_offset_x} 0.004 ${-0.085+elevator_center_offset_z}" rpy = "0 0 ${pi}"/>
                 <geometry>
                     <mesh filename="package://edna_description/meshes/elevator_center.stl" scale="0.001 0.001 0.001"/>
@@ -47,8 +52,9 @@
             </visual>
             <collision>
-                <origin xyz = "0 0 0" rpy = "0 0 0"/>
+                <origin xyz = "${elevator_center_length/2 - 0.03} 0 0" rpy = "0 0 0"/>
                 <geometry>
-                    <box size = "${elevator_outer_length} ${elevator_outer_width} ${elevator_outer_height}"/>
+                    <box size = "${elevator_center_length + 0.01} ${elevator_center_width} ${elevator_center_height}"/>
                 </geometry>
+                <material name="ghost"/>
             </collision>
         </link>
@@ -57,7 +63,9 @@
             <child link = "${prefix}_elevator_center_link"/>
             <axis xyz = "1 0 0"/>
-            <!-- 0.56 -->
             <limit effort="1000.0" lower="0.0" upper="0.56" velocity="0.5"/>
-            <origin xyz = "0 0 0" rpy = "0 0 0"/>
+            <xacro:if value="${suffix == 'right'}">
+                <mimic joint = "${ns}_elevator_left_elevator_center_joint" multiplier = "1" offset = "0"/>
+            </xacro:if>
+            <origin xyz = "${0.1-elevator_center_offset_x} 0 ${elevator_center_offset_z}" rpy = "0 0 0"/>
         </joint>
         <link name = "${prefix}_elevator_outer_2_link">
@@ -66,5 +74,6 @@
             </xacro:inertial_box>
             <visual>
-                <origin xyz = "0.469 -0.07 -0.1" rpy = "0 ${pi} 0"/>
+                <!-- <origin xyz = "${elevator_outer_offset_x+0.34} -0.07 ${-1*(elevator_outer_offset_z+0.015)}" rpy = "0 0 ${pi}"/> -->
+                 <origin xyz = "${elevator_outer_length/2 + 0.045} 0.075 -0.06" rpy = "0 0 ${pi}"/>
                 <geometry>
                     <mesh filename="package://edna_description/meshes/elevator_outer_updated.stl" scale="0.001 0.001 0.001"/>
@@ -73,7 +82,7 @@
             </visual>
             <collision>
-                <origin xyz = "0 0 0" rpy = "0 0 0"/>
+                <origin xyz = "${elevator_outer_length/2 - 0.025} 0 0" rpy = "0 0 ${pi}"/>
                 <geometry>
-                    <box size = "${elevator_outer_length} ${elevator_outer_width} ${elevator_outer_height}"/>
+                    <box size = "${elevator_outer_length + 0.025} ${elevator_outer_width} ${elevator_outer_height}"/>
                 </geometry>
             </collision>
@@ -81,8 +90,9 @@
         <joint name = "${prefix}_elevator_outer_2_joint" type = "prismatic">
             <axis xyz = "1 0 0"/>
-            <!-- 0.568 -->
             <limit effort="1000.0" lower="0.0" upper="0.568" velocity="0.5"/>
             <parent link = "${prefix}_elevator_center_link"/>
             <child link = "${prefix}_elevator_outer_2_link"/>
+            <mimic joint = "${prefix}_elevator_center_joint" multiplier = "1" offset = "0"/>
+            <origin xyz = "${elevator_outer_offset_x} 0 ${elevator_outer_offset_z}" rpy = "0 0 0"/>
         </joint>
     </xacro:macro>

File: src/edna_description/urdf/parts/elevator_leg.xacro (robot description, xacro)
@@ -3,9 +3,11 @@
     <xacro:property name="elevator_leg_length" value="0.052" />
     <xacro:property name="elevator_leg_width" value="0.330" />
-    <xacro:property name="elevator_leg_height" value="0.527" />
+    <xacro:property name="elevator_leg_height" value="0.59" />
     <xacro:property name="roller_bar_length" value="0.0508" />
     <xacro:property name="roller_bar_width" value="0.711" />
-    <xacro:property name="roller_bar_height" value="0.527" />
-    <xacro:macro name = "elevator_leg" params = "prefix parent *origin *origin2">
+    <!-- <xacro:property name="roller_bar_height" value="0.527" /> -->
+    <xacro:property name="roller_bar_height" value="0.1" />
+    <xacro:property name="roller_bar_wheel_radius" value="0.0254"/>
+    <xacro:macro name = "elevator_leg" params = "prefix parent *origin">
         <link name = "${prefix}_elevator_leg_link">
             <xacro:inertial_box mass = "1" x = "${elevator_leg_length}" y = "${elevator_leg_width}" z = "${elevator_leg_height}">
@@ -36,5 +38,5 @@
             </xacro:inertial_box>
             <visual>
-                <origin xyz = "0 -${roller_bar_height/2} 0" rpy = "0 0 0"/>
+                <origin xyz = "0 0 -0.19" rpy = "${pi/2} 0 0"/>
                 <geometry>
                     <mesh filename="package://edna_description/meshes/Roller_Bar.stl" scale="0.001 0.001 0.001"/>
@@ -43,7 +45,13 @@
             </visual>
             <collision>
-                <origin xyz = "0 0 0" rpy = "0 0 0"/>
+                <origin xyz = "0 0 ${roller_bar_height/2 - 0.025}" rpy = "0 0 0"/>
                 <geometry>
-                    <box size = "${roller_bar_length} ${roller_bar_width} ${roller_bar_height}"/>
+                    <box size = "${roller_bar_length} ${roller_bar_width} ${roller_bar_height*0.75}"/>
+                </geometry>
+            </collision>
+            <collision>
+                <origin xyz = "0 0 0.065" rpy = "${pi/2} 0 0"/>
+                <geometry>
+                    <cylinder radius = "${0.0492125/2}" length = "${roller_bar_width}"/>
                 </geometry>
             </collision>
@@ -52,7 +60,9 @@
             <parent link = "${prefix}_elevator_leg_link"/>
             <child link = "${prefix}_roller_bar_link"/>
-            <axis xyz = "0 1 0"/>
-            <limit effort = "100.0" lower = "-1" upper = "0.06985" velocity = "0.5"/>
-            <xacro:insert_block name = "origin2"/>
+            <axis xyz = "0 0 1"/>
+            <limit effort = "100.0" lower = "0" upper = "0.06985" velocity = "1"/>
+            <!-- <limit effort = "100.0" lower = "0" upper = "1" velocity = "0.5"/> -->
+            <origin xyz = "0 0 ${elevator_leg_height/2 + 0.01}" rpy = "0 0 0"/>
+            <!-- <origin xyz = "0 0 0.37" rpy = "0 0 0"/> -->
         </joint>
     </xacro:macro>

File: src/edna_description/urdf/robots/edna.urdf.xacro (robot description, xacro)
@@ -46,18 +46,18 @@
     <origin xyz="${cam_pos}" rpy="0 0 0" />
   </xacro:zed_camera>
+  <xacro:property name="elevator_leg_z" value="0.527"/>
   <xacro:elevator_leg prefix="${ns}_arm" parent="${ns}_swerve_chassis_link">
-    <origin xyz = "0.1905 0 ${0.527/2 + 0.03}" rpy = "0 0 ${pi}"/>
-    <origin xyz = "0 0 ${0.37}" rpy = "${pi/2} 0 0"/>
+    <origin xyz = "0.1905 0 ${elevator_leg_z/2 + 0.03}" rpy = "0 0 0"/>
   </xacro:elevator_leg>
   <xacro:back_leg prefix="${ns}_arm" parent="${ns}_swerve_chassis_link">
-    <origin xyz = "-${0.7366/2 - 0.0508/2} 0 ${back_leg_height/2 + 0.05588}" rpy = "0 0 ${pi}" />
+    <origin xyz = "-${chassis_length/2 - back_leg_length/2} 0 ${back_leg_height/2 + chassis_height}" rpy = "0 0 0" />
   </xacro:back_leg>
   <!--Right Elevator-->
-  <xacro:elevator prefix="${ns}_elevator_right" parent="${ns}_arm_back_leg_link" ns="${ns}">
-    <origin xyz = "0.00253 0.28 0.3738731" rpy = "${pi} ${(0.0174533*15.3)} ${pi}" />
+  <xacro:elevator prefix="${ns}_elevator_right" parent="${ns}_arm_back_leg_link" ns="${ns}" suffix="right">
+    <origin xyz = "0 ${-back_leg_width/2 - 0.04} ${back_leg_height/2 - 0.02}" rpy = "0 0 0" />
   </xacro:elevator>
   <!--Left Elevator-->
-  <xacro:elevator prefix="${ns}_elevator_left" parent="${ns}_arm_back_leg_link" ns="${ns}">
-    <origin xyz = "0.00253 -0.28 0.3738731" rpy = "${pi} ${(0.0174533*15.3)} ${pi}" />
+  <xacro:elevator prefix="${ns}_elevator_left" parent="${ns}_arm_back_leg_link" ns="${ns}" suffix="left">
+    <origin xyz = "0 ${back_leg_width/2 + 0.04} ${back_leg_height/2 - 0.02}" rpy = "0 0 0" />
   </xacro:elevator>
   <xacro:lidar prefix="${ns}_lidar" parent="${ns}_swerve_chassis_link" radius="0.035" length="0.025">

Commit message: Fixed the URDF

File: src/edna_description/urdf/parts/back_leg.xacro (robot description, xacro)
@@ -3,5 +3,9 @@
     <xacro:property name="back_leg_length" value="0.0508" />
     <xacro:property name="back_leg_width" value="0.457" />
-    <xacro:property name="back_leg_height" value="0.812" />
+    <xacro:property name="back_leg_height" value="0.677" />
+    <xacro:property name="lower_bearing_distance" value = ".076" />
+    <xacro:property name="upper_bearing_distance" value = ".030" />
+    <xacro:property name="inside_legs_distance" value = ".279" />
+    <xacro:property name="each_leg_width" value = ".0254" />
     <xacro:macro name = "back_leg" params = "prefix parent *origin">
         <link name = "${prefix}_back_leg_link">
@@ -10,12 +14,12 @@
             </xacro:inertial_box>
             <visual>
-                <origin xyz = "0 0 0" rpy = "0 0 ${pi}"/>
+                <origin xyz = "0 -${(inside_legs_distance + (each_leg_width * 2)) / 2} 0" rpy = "${pi /2} 0 0"/>
                 <geometry>
-                    <mesh filename="package://edna_description/meshes/back_legs.stl" scale="0.001 0.001 0.001"/>
+                    <mesh filename="package://edna_description/meshes/Back_Legs_V6.stl" scale="0.001 0.001 0.001"/>
                 </geometry>
                 <material name = "red"/>
             </visual>
             <collision>
-                <origin xyz = "0 0 0" rpy = "0 0 0"/>
+                <origin xyz = "0 0 ${back_leg_height / 2}" rpy = "0 0 0"/>
                 <geometry>
                     <box size = "${back_leg_length} ${back_leg_width} ${back_leg_height}"/>

File: src/edna_description/urdf/robots/edna.urdf.xacro (robot description, xacro)
@@ -17,4 +17,6 @@
   <xacro:property name="axle_pos" value="${301.625 / 1000}" />
   <xacro:property name="axle_pos_z" value="${69.056 / 1000}" />
+  <xacro:property name="elevator_middle_distance" value = ".457" />
+  <xacro:property name= "chassis_side_width" value = ".0254" />
   <!-- Camera Position Variables -->
   <xacro:property name="cam_pos" value="0 0 0.3"/> <!-- Made up values, replace with real ones later. -->
@@ -53,13 +55,13 @@
   </xacro:elevator_leg>
   <xacro:back_leg prefix="arm" parent="swerve_chassis_link">
-    <origin xyz = "-${chassis_length/2 - back_leg_length/2} 0 ${back_leg_height/2 + chassis_height}" rpy = "0 0 0" />
+    <origin xyz = "-${chassis_length/2 - each_leg_width * 2} 0 ${chassis_height}" rpy = "0 0 0" />
   </xacro:back_leg>
   <!--Right Elevator-->
   <xacro:elevator prefix="elevator_right" parent="arm_back_leg_link" suffix="right">
-    <origin xyz = "0 ${-back_leg_width/2 - 0.04} ${back_leg_height/2 - 0.02}" rpy = "0 0 0" />
+    <origin xyz = "-.03 -${elevator_middle_distance / 2} ${back_leg_height - .0215}" rpy = "0 0 0" />
   </xacro:elevator>
   <!--Left Elevator-->
   <xacro:elevator prefix="elevator_left" parent="arm_back_leg_link" suffix="left">
-    <origin xyz = "0 ${back_leg_width/2 + 0.04} ${back_leg_height/2 - 0.02}" rpy = "0 0 0" />
+    <origin xyz = "-.03 ${elevator_middle_distance / 2} ${back_leg_height - .0215}" rpy = "0 0 0" />
   </xacro:elevator>
   <!-- Control -->
