Commit message: needs fixing

File: src/edna_description/urdf/parts/elevator_leg.xacro (robot description, xacro)
@@ -1,9 +1,9 @@
 <?xml version = "1.0"?>
 <robot xmlns:xacro = "http://www.ros.org/wiki/xacro">
-    <xacro:property name="elevator_leg_length" value="0.052" />
-    <xacro:property name="elevator_leg_width" value="0.330" />
-    <xacro:property name="elevator_leg_height" value="0.59" />
+    <xacro:property name="elevator_leg_length" value="0.0508" />
+    <xacro:property name="elevator_leg_width" value="0.3302" />
+    <xacro:property name="elevator_leg_height" value="0.5842" />
     <xacro:property name="roller_bar_length" value="0.0508" />
-    <xacro:property name="roller_bar_width" value="0.711" />
+    <xacro:property name="roller_bar_width" value="0.7112" />
     <!-- <xacro:property name="roller_bar_height" value="0.527" /> -->
     <xacro:property name="roller_bar_height" value="0.1" />

File: src/edna_description/urdf/robots/edna.urdf.xacro (robot description, xacro)
@@ -16,4 +16,5 @@
   <xacro:include filename="$(find edna_description)/urdf/parts/gripper.xacro" />
   <xacro:include filename="$(find edna_description)/urdf/parts/slider.xacro" />
+  <xacro:include filename="$(find edna_description)/urdf/parts/intake.xacro" />
   <!-- Axle Position Variables -->
   <xacro:property name="axle_pos" value="${301.625 / 1000}" />
@@ -48,7 +49,7 @@
     <origin xyz="${cam_pos}" rpy="0 0 0" />
   </xacro:zed_camera>
-  <xacro:lidar prefix="lidar" parent="swerve_chassis_link" radius="0.035" length="0.025">
+  <!-- <xacro:lidar prefix="lidar" parent="swerve_chassis_link" radius="0.035" length="0.025">
     <origin xyz="${lidar_pos}" rpy="0 0 0" />
-  </xacro:lidar>
+  </xacro:lidar> -->
   <!-- Arm -->
   <xacro:property name="elevator_leg_z" value="0.527"/>
@@ -68,4 +69,9 @@
     <origin xyz = "${slider_pos}" rpy = "0 0 0" />
   </xacro:slider>
+  <!-- Bottom Intake + Gripper -->
+  <xacro:property name= "intake_pos" value = "${chassis_length/2} 0 -${elevator_leg_height/2}" />
+  <xacro:intake prefix="bottom" parent="elevator_outer_1_link">
+    <origin xyz = "${intake_pos}" rpy = "0 0 0" />
+  </xacro:intake>
   <!-- Control -->
   <xacro:swerve_drive_control plugin="$(arg hw_interface_plugin)"/>

Commit message: bottom gripper

File: src/edna_description/urdf/parts/elevator_leg.xacro (robot description, xacro)
@@ -17,5 +17,5 @@
                 <origin xyz = "0 0 0" rpy = "0 0 0"/>
                 <geometry>
-                    <mesh filename="package://edna_description/meshes/elevator_legs.stl" scale="0.001 0.001 0.001"/>
+                    <mesh filename="package://edna_description/meshes/Front_Legs_V2.stl" scale="0.001 0.001 0.001"/>
                 </geometry>
                 <material name = "red"/>
@@ -38,7 +38,7 @@
             </xacro:inertial_box>
             <visual>
-                <origin xyz = "0 0 -0.19" rpy = "${pi/2} 0 0"/>
+                <origin xyz = "0 0 -0.24" rpy = "0 0 0"/>
                 <geometry>
-                    <mesh filename="package://edna_description/meshes/Roller_Bar.stl" scale="0.001 0.001 0.001"/>
+                    <mesh filename="package://edna_description/meshes/Roller_Bar_V2.stl" scale="0.001 0.001 0.001"/>
                 </geometry>
                 <material name = "red"/>

File: src/edna_description/urdf/parts/intake.xacro (robot description, xacro)
@@ -10,5 +10,5 @@
         </xacro:inertial_box>
         <visual>
-            <origin xyz = "0 0 0" rpy = "${pi/2} 0 0"/>
+            <origin xyz = "${intake_block_length} ${intake_block_width/2} 0" rpy = "${pi/2} 0 0"/>
             <geometry>
                 <mesh filename = "package://edna_description/meshes/Front_Intake_V2.stl" scale="0.001 0.001 0.001"/>
@@ -19,5 +19,5 @@
             <origin xyz = "0 0 0" rpy = "0 0 0"/>
             <geometry>
-                <box size="${intake_block_length} ${intake_block_length} ${intake_block_height}"/>
+                <box size="${intake_block_length} ${intake_block_width} ${intake_block_height}"/>
             </geometry>
         </collision>
@@ -31,5 +31,5 @@
     </joint>
     <xacro:gripper prefix="${prefix}" parent="${prefix}_intake_link">
-        <origin xyz = "0 -${intake_block_width/2} ${intake_block_height/2}" rpy = "0 0 0" />
+        <origin xyz = "${intake_block_length} 0 0.0127" rpy = "0 0 0" />
     </xacro:gripper>
   </xacro:macro>

File: src/edna_description/urdf/robots/edna.urdf.xacro (robot description, xacro)
@@ -70,5 +70,5 @@
   </xacro:slider>
   <!-- Bottom Intake + Gripper -->
-  <xacro:property name= "intake_pos" value = "${chassis_length/2} 0 -${elevator_leg_height/2}" />
+  <xacro:property name= "intake_pos" value = "${chassis_length/2 + 0.17} ${intake_block_width/2 + 0.025} -${elevator_leg_height/2 + 0.23}" />
   <xacro:intake prefix="bottom" parent="elevator_outer_1_link">
     <origin xyz = "${intake_pos}" rpy = "0 0 0" />
