Commit message: Make bottom intake up by default

File: src/edna_description/urdf/parts/intake.xacro (robot description, xacro)
@@ -27,6 +27,6 @@
         <parent link="${parent}"/>
         <child link="${prefix}_intake_link"/>
-        <axis xyz = "0 -1 0"/>
-        <limit effort = "100.0" lower = "0" upper = "1.42" velocity = "1"/>
+        <axis xyz = "0 1 0"/>
+        <limit effort = "100.0" lower = "0" upper = "${pi/2 - 0.05}" velocity = "1"/>
     </joint>
     <!-- <xacro:gripper prefix="${prefix}" parent="${prefix}_intake_link">

File: src/edna_description/urdf/robots/edna.urdf.xacro (robot description, xacro)
@@ -72,5 +72,5 @@
   <xacro:property name= "intake_pos" value = "0 0 -${elevator_leg_height/4 + 0.01}" />
   <xacro:intake prefix="bottom" parent="arm_elevator_leg_link">
-    <origin xyz = "${intake_pos}" rpy = "0 0 0" />
+    <origin xyz = "${intake_pos}" rpy = "0 -${pi/2 - 0.05} 0" />
   </xacro:intake>
   <!-- Control -->
