Commit message: zed launch

File: src/edna_description/urdf/parts/zed_macro.urdf.xacro (robot description, xacro)
@@ -106,31 +106,10 @@
       <child link="${prefix}_right_camera_optical_frame"/>
     </joint>
-    <!-- ZED2 Sensors -->
-    <xacro:if value="${model == 'zed2'}">
-      <link name="${prefix}_mag_link" />
-      <joint name="${prefix}_mag_joint" type="fixed">
-        <parent link="${prefix}_camera_center"/>
-        <child link="${prefix}_mag_link"/>
-        <origin xyz="0 0 0" rpy="0 0 0" />
-      </joint>
-      <link name="${prefix}_baro_link" />
-      <joint name="${prefix}_baro_joint" type="fixed">
-        <parent link="${prefix}_camera_center"/>
-        <child link="${prefix}_baro_link"/>
-        <origin xyz="0 0 0" rpy="0 0 0" />
-      </joint>
-      <link name="${prefix}_temp_left_link" />
-      <joint name="${prefix}_temp_left_joint" type="fixed">
-        <parent link="${prefix}_left_camera_frame"/>
-        <child link="${prefix}_temp_left_link"/>
-        <origin xyz="0 0 0" rpy="0 0 0" />
-      </joint>
-      <link name="${prefix}_temp_right_link" />
-      <joint name="${prefix}_temp_right_joint" type="fixed">
-        <parent link="${prefix}_right_camera_frame"/>
-        <child link="${prefix}_temp_right_link"/>
-        <origin xyz="0 0 0" rpy="0 0 0" />
-      </joint>
-    </xacro:if>
+    <link name="${prefix}_imu_link" />
+    <joint name="${prefix}_imu_joint" type="fixed">
+      <parent link="${prefix}_left_camera_frame"/>
+      <child link="${prefix}_imu_link"/>
+      <origin xyz="0 0 0" rpy="0 0 0" />
+    </joint>
   </xacro:macro>
 </robot>

File: src/edna_description/urdf/robots/edna.urdf.xacro (robot description, xacro)
@@ -46,5 +46,5 @@
   </xacro:swerve_axle>
   <!-- Sensors -->
-  <xacro:zed_camera prefix="zed" model="zed2i" parent="swerve_chassis_link">
+  <xacro:zed_camera prefix="zed2i" model="zed2i" parent="swerve_chassis_link">
     <origin xyz="${cam_pos}" rpy="0 0 0" />
   </xacro:zed_camera>

Commit message: yay it works

File: src/edna_description/urdf/parts/zed_macro.urdf.xacro (robot description, xacro)
@@ -85,9 +85,9 @@
       <parent link="${prefix}_camera_center"/>
       <child link="${prefix}_left_camera_frame"/>
-      <origin xyz="0 ${baseline/2} 0" rpy="-${M_PI/2} 0 -${M_PI/2}" />
+      <origin xyz="0 ${baseline/2} 0" rpy="0 0 0" />
     </joint>
     <link name="${prefix}_left_camera_optical_frame"/>
     <joint name="${prefix}_left_camera_optical_joint" type="fixed">
-      <origin xyz="0 0 ${optical_offset_x}" rpy="${M_PI} 0 0"/>
+      <origin xyz="${optical_offset_x} 0 0" rpy="-${M_PI/2} 0.0 -${M_PI/2}"/>
       <parent link="${prefix}_left_camera_frame"/>
       <child link="${prefix}_left_camera_optical_frame"/>
@@ -98,9 +98,9 @@
       <parent link="${prefix}_camera_center"/>
       <child link="${prefix}_right_camera_frame"/>
-      <origin xyz="0 -${baseline/2} 0" rpy="-${M_PI/2} 0 -${M_PI/2}" />
+      <origin xyz="0 -${baseline/2} 0" rpy="0 0 0" />
     </joint>
     <link name="${prefix}_right_camera_optical_frame"/>
     <joint name="${prefix}_right_camera_optical_joint" type="fixed">
-      <origin xyz="0 0 ${optical_offset_x}" rpy="${M_PI} 0 0"/>
+      <origin xyz="${optical_offset_x} 0 0" rpy="-${M_PI/2} 0.0 -${M_PI/2}"/>
       <parent link="${prefix}_right_camera_frame"/>
       <child link="${prefix}_right_camera_optical_frame"/>

Commit message: Zed + FIELD ORIENTED (looking at you tanush) (#124)
* added zed launch file and config file

* zed launch

* yay it works

---------

Co-authored-by: Gage Miller <gagemiller155@gmail.com>

File: src/edna_description/urdf/parts/zed_macro.urdf.xacro (robot description, xacro)
@@ -85,9 +85,9 @@
       <parent link="${prefix}_camera_center"/>
       <child link="${prefix}_left_camera_frame"/>
-      <origin xyz="0 ${baseline/2} 0" rpy="-${M_PI/2} 0 -${M_PI/2}" />
+      <origin xyz="0 ${baseline/2} 0" rpy="0 0 0" />
     </joint>
     <link name="${prefix}_left_camera_optical_frame"/>
     <joint name="${prefix}_left_camera_optical_joint" type="fixed">
-      <origin xyz="0 0 ${optical_offset_x}" rpy="${M_PI} 0 0"/>
+      <origin xyz="${optical_offset_x} 0 0" rpy="-${M_PI/2} 0.0 -${M_PI/2}"/>
       <parent link="${prefix}_left_camera_frame"/>
       <child link="${prefix}_left_camera_optical_frame"/>
@@ -98,39 +98,18 @@
       <parent link="${prefix}_camera_center"/>
       <child link="${prefix}_right_camera_frame"/>
-      <origin xyz="0 -${baseline/2} 0" rpy="-${M_PI/2} 0 -${M_PI/2}" />
+      <origin xyz="0 -${baseline/2} 0" rpy="0 0 0" />
     </joint>
     <link name="${prefix}_right_camera_optical_frame"/>
     <joint name="${prefix}_right_camera_optical_joint" type="fixed">
-      <origin xyz="0 0 ${optical_offset_x}" rpy="${M_PI} 0 0"/>
+      <origin xyz="${optical_offset_x} 0 0" rpy="-${M_PI/2} 0.0 -${M_PI/2}"/>
       <parent link="${prefix}_right_camera_frame"/>
       <child link="${prefix}_right_camera_optical_frame"/>
     </joint>
-    <!-- ZED2 Sensors -->
-    <xacro:if value="${model == 'zed2'}">
-      <link name="${prefix}_mag_link" />
-      <joint name="${prefix}_mag_joint" type="fixed">
-        <parent link="${prefix}_camera_center"/>
-        <child link="${prefix}_mag_link"/>
-        <origin xyz="0 0 0" rpy="0 0 0" />
-      </joint>
-      <link name="${prefix}_baro_link" />
-      <joint name="${prefix}_baro_joint" type="fixed">
-        <parent link="${prefix}_camera_center"/>
-        <child link="${prefix}_baro_link"/>
-        <origin xyz="0 0 0" rpy="0 0 0" />
-      </joint>
-      <link name="${prefix}_temp_left_link" />
-      <joint name="${prefix}_temp_left_joint" type="fixed">
-        <parent link="${prefix}_left_camera_frame"/>
-        <child link="${prefix}_temp_left_link"/>
-        <origin xyz="0 0 0" rpy="0 0 0" />
-      </joint>
-      <link name="${prefix}_temp_right_link" />
-      <joint name="${prefix}_temp_right_joint" type="fixed">
-        <parent link="${prefix}_right_camera_frame"/>
-        <child link="${prefix}_temp_right_link"/>
-        <origin xyz="0 0 0" rpy="0 0 0" />
-      </joint>
-    </xacro:if>
+    <link name="${prefix}_imu_link" />
+    <joint name="${prefix}_imu_joint" type="fixed">
+      <parent link="${prefix}_left_camera_frame"/>
+      <child link="${prefix}_imu_link"/>
+      <origin xyz="0 0 0" rpy="0 0 0" />
+    </joint>
   </xacro:macro>
 </robot>

Commit message: Update state

File: src/edna_description/urdf/parts/zed_macro.urdf.xacro (robot description, xacro)
@@ -93,4 +93,10 @@
       <child link="${prefix}_left_camera_optical_frame"/>
     </joint>
+    <link name="${prefix}_left_camera_isaac_frame"/>
+    <joint name="${prefix}_left_camera_isaac_joint" type="fixed">
+      <origin xyz="0 0 0" rpy="${M_PI/2} 0.0 -${M_PI/2}"/>
+      <parent link="${prefix}_left_camera_frame"/>
+      <child link="${prefix}_left_camera_isaac_frame"/>
+    </joint>
     <!-- Right Camera -->
     <link name="${prefix}_right_camera_frame" />
@@ -106,4 +112,10 @@
       <child link="${prefix}_right_camera_optical_frame"/>
     </joint>
+    <link name="${prefix}_right_camera_isaac_frame"/>
+    <joint name="${prefix}_right_camera_isaac_joint" type="fixed">
+      <origin xyz="0 0 0" rpy="${M_PI/2} 0.0 -${M_PI/2}"/>
+      <parent link="${prefix}_right_camera_frame"/>
+      <child link="${prefix}_right_camera_isaac_frame"/>
+    </joint>
     <link name="${prefix}_imu_link" />
     <joint name="${prefix}_imu_joint" type="fixed">
