Commit message: Added top slider and gripper

File: src/edna_description/urdf/parts/gripper.xacro (robot description, xacro)
@@ -20,5 +20,5 @@
           <mesh filename="package://edna_description/meshes/center_gripper_bar.stl" scale="0.001 0.001 0.001"/>
         </geometry>
-        <material name="blue"/>
+        <material name="yellow"/>
       </visual>
       <collision>
@@ -92,4 +92,5 @@
       <child link="${prefix}_gripper_right_arm_link"/>
       <axis xyz = "0 0 1"/>
+      <mimic joint = "${prefix}_gripper_left_arm_joint" multiplier = "1" offset = "0"/>
       <limit effort="1000.0" lower="-0.3" upper="0.6" velocity="0.5"/>
     </joint>

File: src/edna_description/urdf/robots/edna.urdf.xacro (robot description, xacro)
@@ -15,4 +15,5 @@
   <xacro:include filename="$(find edna_description)/urdf/parts/elevator.xacro" />
   <xacro:include filename="$(find edna_description)/urdf/parts/gripper.xacro" />
+  <xacro:include filename="$(find edna_description)/urdf/parts/slider.xacro" />
   <!-- Axle Position Variables -->
   <xacro:property name="axle_pos" value="${301.625 / 1000}" />
@@ -21,5 +22,5 @@
   <xacro:property name= "chassis_side_width" value = ".0254" />
   <!-- Camera Position Variables -->
-  <xacro:property name="cam_pos" value="0 0 0.3"/> <!-- Made up values, replace with real ones later. -->
+  <xacro:property name="cam_pos" value="0.2 0 0.3"/> <!-- Made up values, replace with real ones later. -->
   <!-- X IS FORWARD -->
   <!-- Y IS LEFT -->
@@ -66,8 +67,9 @@
     <origin xyz = "-.03 ${elevator_middle_distance / 2} ${back_leg_height - .0215}" rpy = "0 0 0" />
   </xacro:elevator>
-  <!-- Top Gripper -->
-  <!-- <xacro:gripper prefix="top" parent="base_link">
-    <origin xyz = "0 0 0" rpy = "0 0 0" />
-  </xacro:gripper> -->
+  <!-- Top Slider + Gripper -->
+  <xacro:property name= "slider_pos" value = "0.330 -${elevator_middle_distance / 2} ${slider_block_height/2}" />
+  <xacro:slider prefix="top" parent="elevator_left_elevator_outer_2_link">
+    <origin xyz = "${slider_pos}" rpy = "0 0 0" />
+  </xacro:slider>
   <!-- Control -->
   <xacro:swerve_drive_control plugin="$(arg hw_interface_plugin)"/>

Commit message: dpad, gripper stuff

File: src/edna_description/urdf/parts/gripper.xacro (robot description, xacro)
@@ -58,9 +58,9 @@
     </link>
     <joint name="${prefix}_gripper_left_arm_joint" type="revolute">
-      <origin xyz = "0 ${center_to_arm_axle_left} ${arm_axle_lower}" rpy = "0 0 0" />
+      <origin xyz = "0 ${center_to_arm_axle_left} ${arm_axle_lower}" rpy = "0 0 ${pi/10}" />
       <parent link="${prefix}_gripper_bar_link"/>
       <child link="${prefix}_gripper_left_arm_link"/>
       <axis xyz = "0 0 -1"/>
-      <limit effort="1000.0" lower="-0.3" upper="0.6" velocity="0.5"/>
+      <limit effort="1000.0" lower="0" upper="0.9" velocity="0.5"/>
     </joint>
     <!-- Right -->
@@ -88,10 +88,10 @@
     </link>
     <joint name="${prefix}_gripper_right_arm_joint" type="revolute">
-      <origin xyz = "0 ${center_to_arm_axle_right} ${arm_axle_lower}" rpy = "0 0 0" />
+      <origin xyz = "0 ${center_to_arm_axle_right} ${arm_axle_lower}" rpy = "0 0 -${pi/10}" />
       <parent link="${prefix}_gripper_bar_link"/>
       <child link="${prefix}_gripper_right_arm_link"/>
       <axis xyz = "0 0 1"/>
       <mimic joint = "${prefix}_gripper_left_arm_joint" multiplier = "1" offset = "0"/>
-      <limit effort="1000.0" lower="-0.3" upper="0.6" velocity="0.5"/>
+      <limit effort="1000.0" lower="0" upper="0.9" velocity="0.5"/>
     </joint>
   </xacro:macro>

File: src/edna_description/urdf/parts/intake.xacro (robot description, xacro)
@@ -10,5 +10,5 @@
         </xacro:inertial_box>
         <visual>
-            <origin xyz = "${intake_block_length} ${intake_block_width/2} 0" rpy = "${pi/2} 0 0"/>
+            <origin xyz = "${intake_block_length-0.04} ${intake_block_width/2} -0.0508" rpy = "${pi/2} 0 0"/>
             <geometry>
                 <mesh filename = "package://edna_description/meshes/Front_Intake_V2.stl" scale="0.001 0.001 0.001"/>
@@ -17,5 +17,5 @@
         </visual>
         <collision>
-            <origin xyz = "0 0 0" rpy = "0 0 0"/>
+            <origin xyz = "${intake_block_length/2} 0 ${intake_block_height/2}" rpy = "0 0 0"/>
             <geometry>
                 <box size="${intake_block_length} ${intake_block_width} ${intake_block_height}"/>
@@ -27,9 +27,9 @@
         <parent link="${parent}"/>
         <child link="${prefix}_intake_link"/>
-        <axis xyz = "0 1 0"/>
-        <limit effort = "100.0" lower = "0" upper = "0.3" velocity = "1"/>
+        <axis xyz = "0 -1 0"/>
+        <limit effort = "100.0" lower = "0" upper = "1.42" velocity = "1"/>
     </joint>
     <xacro:gripper prefix="${prefix}" parent="${prefix}_intake_link">
-        <origin xyz = "${intake_block_length} 0 0.0127" rpy = "0 0 0" />
+        <origin xyz = "${intake_block_length - 0.1} 0 -0.035" rpy = "0 0 0" />
     </xacro:gripper>
   </xacro:macro>

File: src/edna_description/urdf/robots/edna.urdf.xacro (robot description, xacro)
@@ -70,6 +70,6 @@
   </xacro:slider>
   <!-- Bottom Intake + Gripper -->
-  <xacro:property name= "intake_pos" value = "${chassis_length/2 + 0.17} ${intake_block_width/2 + 0.025} -${elevator_leg_height/2 + 0.23}" />
-  <xacro:intake prefix="bottom" parent="elevator_outer_1_link">
+  <xacro:property name= "intake_pos" value = "0 0 -${elevator_leg_height/4}" />
+  <xacro:intake prefix="bottom" parent="arm_elevator_leg_link">
     <origin xyz = "${intake_pos}" rpy = "0 0 0" />
   </xacro:intake>

Commit message: Finished high teleop

File: src/edna_description/urdf/parts/gripper.xacro (robot description, xacro)
@@ -58,9 +58,9 @@
     </link>
     <joint name="${prefix}_gripper_left_arm_joint" type="revolute">
-      <origin xyz = "0 ${center_to_arm_axle_left} ${arm_axle_lower}" rpy = "0 0 ${pi/10}" />
+      <origin xyz = "0 ${center_to_arm_axle_left} ${arm_axle_lower}" rpy = "0 0 ${-0.9 + pi/10}" />
       <parent link="${prefix}_gripper_bar_link"/>
       <child link="${prefix}_gripper_left_arm_link"/>
       <axis xyz = "0 0 -1"/>
-      <limit effort="1000.0" lower="0" upper="0.9" velocity="0.5"/>
+      <limit effort="1000.0" lower="-0.9" upper="0" velocity="0.5"/>
     </joint>
     <!-- Right -->
@@ -88,10 +88,10 @@
     </link>
     <joint name="${prefix}_gripper_right_arm_joint" type="revolute">
-      <origin xyz = "0 ${center_to_arm_axle_right} ${arm_axle_lower}" rpy = "0 0 -${pi/10}" />
+      <origin xyz = "0 ${center_to_arm_axle_right} ${arm_axle_lower}" rpy = "0 0 ${-pi/10 + 0.9}" />
       <parent link="${prefix}_gripper_bar_link"/>
       <child link="${prefix}_gripper_right_arm_link"/>
       <axis xyz = "0 0 1"/>
       <mimic joint = "${prefix}_gripper_left_arm_joint" multiplier = "1" offset = "0"/>
-      <limit effort="1000.0" lower="0" upper="0.9" velocity="0.5"/>
+      <limit effort="1000.0" lower="-0.9" upper="0" velocity="0.5"/>
     </joint>
   </xacro:macro>
