Commit message: Robot Arm Started

File: isaac/exts/omni.isaac.edna/omni/isaac/edna/edna.urdf (robot description, URDF)
Before this commit: robot edna, 10 links, 9 joints
Links:
- added link swerve_box, mass 1; collision box size=1 1 1; visual box size=1 1 1
Joints:
- added joint swerve_box_joint: type fixed, parent swerve_chassis_link, child swerve_box, origin xyz=0 0 0 rpy=0 0 0

File: src/edna_description/urdf/robots/edna.urdf.xacro (robot description, xacro)
@@ -9,4 +9,5 @@
   <xacro:include filename="$(find edna_description)/urdf/parts/square_chassis.xacro" />
   <xacro:include filename="$(find edna_description)/urdf/parts/swerve_axle.xacro" />
+  <xacro:include filename="$(find edna_description)/urdf/parts/arm.xacro" />
   <!-- <xacro:include filename="$(find edna_description)/urdf/parts/zed_macro.urdf.xacro" /> -->
   <!-- Axle Position Variables -->
@@ -28,4 +29,5 @@
     <origin xyz="-${axle_pos} ${axle_pos_y} -${axle_pos}" rpy="${pi / 2} 0 0" />
   </xacro:swerve_axle>
+  <xacro:arm prefix = "swerve"/>
   <!-- <xacro:zed_camera name="zed_camera" model="zed2i" parent="swerve_chassis_link">
     <origin xyz="${cam_pos}" rpy="${pi/2} 0 0" />

Commit message: update urdf

File: isaac/exts/omni.isaac.edna/omni/isaac/edna/edna.urdf (robot description, URDF)
Before this commit: robot edna, 11 links, 10 joints
Links:
- removed link swerve_box
Joints:
- removed joint swerve_box_joint

File: src/edna_description/urdf/robots/edna.urdf.xacro (robot description, xacro)
@@ -27,5 +27,4 @@
     <origin xyz="-${axle_pos} ${axle_pos_y} -${axle_pos}" rpy="${pi / 2} 0 0" />
   </xacro:swerve_axle>
-  <xacro:arm prefix = "swerve"/>
   <!-- <xacro:zed_camera name="zed_camera" model="zed2i" parent="swerve_chassis_link">
     <origin xyz="${cam_pos}" rpy="${pi/2} 0 0" />

Commit message: Large update to fix motion in sim

File: isaac/exts/omni.isaac.edna/omni/isaac/edna/edna.urdf (robot description, URDF)
Before this commit: robot edna, 10 links, 9 joints
Links:
- link swerve_chassis_link: geometry collision box size=0.7366 0.7366 0.05588; visual mesh filename=package://edna_description/meshes/SwerveChassis.stl scale=0.001 0.001 0.001
Joints:
- joint front_left_axle_joint: axis 0 0 1 -> 0 0 -1; origin xyz=0.301625 0.06905599999999999 0.301625 rpy=1.5707963267948966 0 0 -> xyz=0.301625 0.301625 0.06905599999999999 rpy=0 0 0
- joint front_left_wheel_joint: axis 1 0 0 -> 0 1 0; origin xyz=-0.022 0 0.065 rpy=0 0 0 -> xyz=0 0 -0.063 rpy=0 0 0
- joint front_right_axle_joint: axis 0 0 1 -> 0 0 -1; origin xyz=-0.301625 0.06905599999999999 0.301625 rpy=1.5707963267948966 0 0 -> xyz=0.301625 -0.301625 0.06905599999999999 rpy=0 0 0
- joint front_right_wheel_joint: axis 1 0 0 -> 0 1 0; origin xyz=-0.022 0 0.065 rpy=0 0 0 -> xyz=0 0 -0.063 rpy=0 0 0
- joint rear_left_axle_joint: axis 0 0 1 -> 0 0 -1; origin xyz=0.301625 0.06905599999999999 -0.301625 rpy=1.5707963267948966 0 0 -> xyz=-0.301625 0.301625 0.06905599999999999  rpy=0 0 0
- joint rear_left_wheel_joint: axis 1 0 0 -> 0 1 0; origin xyz=-0.022 0 0.065 rpy=0 0 0 -> xyz=0 0 -0.063 rpy=0 0 0
- joint rear_right_axle_joint: axis 0 0 1 -> 0 0 -1; origin xyz=-0.301625 0.06905599999999999 -0.301625 rpy=1.5707963267948966 0 0 -> xyz=-0.301625 -0.301625 0.06905599999999999 rpy=0 0 0
- joint rear_right_wheel_joint: axis 1 0 0 -> 0 1 0; origin xyz=-0.022 0 0.065 rpy=0 0 0 -> xyz=0 0 -0.063 rpy=0 0 0
- joint swerve_chassis_joint: origin xyz=0 0 0 rpy=1.5707963267948966 0 0 -> xyz=0 0 0 rpy=0 0 0

File: src/edna_description/urdf/parts/swerve_axle.xacro (robot description, xacro)
@@ -30,5 +30,5 @@
             <child link="${prefix}_axle_link" />
             <xacro:insert_block name="origin" />
-            <axis xyz="0 0 1" />
+            <axis xyz="0 0 -1" />
             <dynamics friction="0.1" />
         </joint>

Commit message: turned off gpu dynamics and added imu sim sensor.

File: isaac/exts/omni.isaac.edna/omni/isaac/edna/edna.urdf (robot description, URDF)
Before this commit: robot edna, 10 links, 9 joints
Links:
- added link imu_sensor_link, mass 0.001; collision box size=0.02 0.02 0.02; visual box size=0.02 0.02 0.02
- added link zed_camera_base_link
- added link zed_camera_camera_center; collision mesh filename=package://edna_description/meshes/zed2i.stl; visual mesh filename=package://edna_description/meshes/zed2i.stl
- added link zed_camera_left_camera_frame
- added link zed_camera_left_camera_optical_frame
- added link zed_camera_right_camera_frame
- added link zed_camera_right_camera_optical_frame
Joints:
- added joint imu_sensor_joint: type fixed, parent swerve_chassis_link, child imu_sensor_link, axis 0 0 1
- added joint zed_camera_base_joint: type fixed, parent swerve_chassis_link, child zed_camera_base_link, origin xyz=.3575 0.085 0.0 rpy=1.5707963267948966 0 0
- added joint zed_camera_camera_center_joint: type fixed, parent zed_camera_base_link, child zed_camera_camera_center, origin xyz=0 0 0.015 rpy=0 0.0 0
- added joint zed_camera_left_camera_joint: type fixed, parent zed_camera_camera_center, child zed_camera_left_camera_frame, origin xyz=0 0.06 0 rpy=0 0 0
- added joint zed_camera_left_camera_optical_joint: type fixed, parent zed_camera_left_camera_frame, child zed_camera_left_camera_optical_frame, origin xyz=-0.01 0 0 rpy=-1.5707963267948966 0.0 -1.5707963267948966
- added joint zed_camera_right_camera_joint: type fixed, parent zed_camera_camera_center, child zed_camera_right_camera_frame, origin xyz=0 -0.06 0 rpy=0 0 0
- added joint zed_camera_right_camera_optical_joint: type fixed, parent zed_camera_right_camera_frame, child zed_camera_right_camera_optical_frame, origin xyz=-0.01 0 0 rpy=-1.5707963267948966 0.0 -1.5707963267948966

File: src/edna_description/urdf/edna.urdf (robot description, URDF)
Before this commit: robot edna, 10 links, 9 joints
Links:
- added link imu_sensor_link, mass 0.001; collision box size=0.02 0.02 0.02; visual box size=0.02 0.02 0.02
- added link zed_camera_base_link
- added link zed_camera_camera_center; collision mesh filename=package://edna_description/meshes/zed2i.stl; visual mesh filename=package://edna_description/meshes/zed2i.stl
- added link zed_camera_left_camera_frame
- added link zed_camera_left_camera_optical_frame
- added link zed_camera_right_camera_frame
- added link zed_camera_right_camera_optical_frame
Joints:
- added joint imu_sensor_joint: type fixed, parent swerve_chassis_link, child imu_sensor_link, axis 0 0 1
- added joint zed_camera_base_joint: type fixed, parent swerve_chassis_link, child zed_camera_base_link, origin xyz=.3575 0.085 0.0 rpy=1.5707963267948966 0 0
- added joint zed_camera_camera_center_joint: type fixed, parent zed_camera_base_link, child zed_camera_camera_center, origin xyz=0 0 0.015 rpy=0 0.0 0
- added joint zed_camera_left_camera_joint: type fixed, parent zed_camera_camera_center, child zed_camera_left_camera_frame, origin xyz=0 0.06 0 rpy=0 0 0
- added joint zed_camera_left_camera_optical_joint: type fixed, parent zed_camera_left_camera_frame, child zed_camera_left_camera_optical_frame, origin xyz=-0.01 0 0 rpy=-1.5707963267948966 0.0 -1.5707963267948966
- added joint zed_camera_right_camera_joint: type fixed, parent zed_camera_camera_center, child zed_camera_right_camera_frame, origin xyz=0 -0.06 0 rpy=0 0 0
- added joint zed_camera_right_camera_optical_joint: type fixed, parent zed_camera_right_camera_frame, child zed_camera_right_camera_optical_frame, origin xyz=-0.01 0 0 rpy=-1.5707963267948966 0.0 -1.5707963267948966

File: src/edna_description/urdf/parts/imu.urdf.xacro (robot description, xacro)
@@ -1,8 +1,7 @@
 <?xml version="1.0"?>
 <robot xmlns:xacro="http://www.ros.org/wiki/xacro" name="imu">
-<xacro:macro name="imu_sensor" params="xyz rpy parent">
+<xacro:macro name="imu_sensor" params="parent *origin">
     <joint name="imu_sensor_joint" type="fixed">
         <axis xyz="0 0 1" />
-        <origin xyz="${xyz}" rpy="${rpy}"/>
         <parent link="${parent}"/>
         <child link="imu_sensor_link"/>
@@ -20,5 +19,4 @@
                 <box size="0.02 0.02 0.02"/>
             </geometry>
-            <material/>
         </visual>
         <inertial>
@@ -28,22 +26,4 @@
         </inertial>
     </link>
-    <gazebo reference="imu_sensor_link">
-        <gravity>true</gravity>
-        <sensor name='imu_sensor' type='imu'>
-            <always_on>1</always_on>
-            <update_rate>1000</update_rate>
-            <visualize>1</visualize>
-            <topic>__default_topic__</topic>
-            <plugin name='imu_plugin' filename='libgazebo_ros_imu_sensor.so'>
-                <topicName>imu_data</topicName>
-                <bodyName>imu_sensor_link</bodyName>
-                <updateRateHZ>10.0</updateRateHZ>
-                <gaussianNoise>0.0</gaussianNoise>
-                <xyzOffset>0 0 0</xyzOffset>
-                <rpyOffset>0 0 0</rpyOffset>
-            </plugin>
-            <pose>0 0 0 0 0 0</pose>
-        </sensor>
-    </gazebo>
 </xacro:macro>
 </robot>

File: src/edna_description/urdf/robots/edna.urdf.xacro (robot description, xacro)
@@ -9,4 +9,6 @@
   <xacro:include filename="$(find edna_description)/urdf/parts/square_chassis.xacro" />
   <xacro:include filename="$(find edna_description)/urdf/parts/swerve_axle.xacro" />
+  <xacro:include filename="$(find edna_description)/urdf/parts/zed_macro.urdf.xacro" />
+  <xacro:include filename="$(find edna_description)/urdf/parts/imu.urdf.xacro" />
   <!-- Axle Position Variables -->
   <xacro:property name="axle_pos" value="${301.625 / 1000}" />
@@ -27,7 +29,10 @@
     <origin xyz="-${axle_pos} ${axle_pos_y} -${axle_pos}" rpy="${pi / 2} 0 0" />
   </xacro:swerve_axle>
-  <!-- <xacro:zed_camera name="zed_camera" model="zed2i" parent="swerve_chassis_link">
+  <xacro:zed_camera name="zed_camera" model="zed2i" parent="swerve_chassis_link">
     <origin xyz="${cam_pos}" rpy="${pi/2} 0 0" />
-  </xacro:zed_camera> -->
+  </xacro:zed_camera>
+  <xacro:imu_sensor parent="swerve_chassis_link">
+    <origin xyz="0 0 0" rpy="${pi/2} 0 0" />
+  </xacro:imu_sensor>
   <xacro:swerve_drive_control plugin="$(arg hw_interface_plugin)" />
 </robot>

Commit message: Motion magic sim (#3)
* Add Fixes to the hardware and controller

* Fix urdf and controller output

* add a motion magic files

* Remove bad code

* Updated isaac drive

* Large update to fix motion in sim

* motion magic for sim

* oscillations fixed

* quality of life

* Refine real drive

* Fix controller config

* fixed axle velocities not peing published

---------

Co-authored-by: Gage Miller <gagemiller155@gmail.com>
Co-authored-by: SarangaR <sarnga.raj@gmail.com>
Co-authored-by: Roman Mock <romanjmock@gmail.com>

File: isaac/exts/omni.isaac.edna/omni/isaac/edna/edna.urdf (robot description, URDF)
Before this commit: robot edna, 17 links, 16 joints
Links:
- removed link imu_sensor_link
- removed link zed_camera_base_link
- removed link zed_camera_camera_center
- removed link zed_camera_left_camera_frame
- removed link zed_camera_left_camera_optical_frame
- removed link zed_camera_right_camera_frame
- removed link zed_camera_right_camera_optical_frame
- link swerve_chassis_link: geometry collision box size=0.7366 0.7366 0.05588; visual mesh filename=package://edna_description/meshes/SwerveChassis.stl scale=0.001 0.001 0.001
Joints:
- removed joint imu_sensor_joint
- removed joint zed_camera_base_joint
- removed joint zed_camera_camera_center_joint
- removed joint zed_camera_left_camera_joint
- removed joint zed_camera_left_camera_optical_joint
- removed joint zed_camera_right_camera_joint
- removed joint zed_camera_right_camera_optical_joint
- joint front_left_axle_joint: axis 0 0 1 -> 0 0 -1; origin xyz=0.301625 0.06905599999999999 0.301625 rpy=1.5707963267948966 0 0 -> xyz=0.301625 0.301625 0.06905599999999999 rpy=0 0 0
- joint front_left_wheel_joint: axis 1 0 0 -> 0 1 0; origin xyz=-0.022 0 0.065 rpy=0 0 0 -> xyz=0 0 -0.063 rpy=0 0 0
- joint front_right_axle_joint: axis 0 0 1 -> 0 0 -1; origin xyz=-0.301625 0.06905599999999999 0.301625 rpy=1.5707963267948966 0 0 -> xyz=0.301625 -0.301625 0.06905599999999999 rpy=0 0 0
- joint front_right_wheel_joint: axis 1 0 0 -> 0 1 0; origin xyz=-0.022 0 0.065 rpy=0 0 0 -> xyz=0 0 -0.063 rpy=0 0 0
- joint rear_left_axle_joint: axis 0 0 1 -> 0 0 -1; origin xyz=0.301625 0.06905599999999999 -0.301625 rpy=1.5707963267948966 0 0 -> xyz=-0.301625 0.301625 0.06905599999999999  rpy=0 0 0
- joint rear_left_wheel_joint: axis 1 0 0 -> 0 1 0; origin xyz=-0.022 0 0.065 rpy=0 0 0 -> xyz=0 0 -0.063 rpy=0 0 0
- joint rear_right_axle_joint: axis 0 0 1 -> 0 0 -1; origin xyz=-0.301625 0.06905599999999999 -0.301625 rpy=1.5707963267948966 0 0 -> xyz=-0.301625 -0.301625 0.06905599999999999 rpy=0 0 0
- joint rear_right_wheel_joint: axis 1 0 0 -> 0 1 0; origin xyz=-0.022 0 0.065 rpy=0 0 0 -> xyz=0 0 -0.063 rpy=0 0 0
- joint swerve_chassis_joint: origin xyz=0 0 0 rpy=1.5707963267948966 0 0 -> xyz=0 0 0 rpy=0 0 0

File: src/edna_description/urdf/parts/swerve_axle.xacro (robot description, xacro)
@@ -2,6 +2,6 @@
 <robot xmlns:xacro="http://www.ros.org/wiki/xacro">
     <!-- Chassis Properties -->
-    <xacro:property name="axle_radius" value="0.075" />
-    <xacro:property name="axle_length" value=".1" />
+    <xacro:property name="axle_radius" value="0.05" />
+    <xacro:property name="axle_length" value="0.03" />
     <xacro:property name="axle_mass" value="0.23739" />
     <xacro:property name="wheel_radius" value="0.0508" />
@@ -11,10 +11,10 @@
     <!-- NOTE: The below values are **guesses**-->
     <!-- NOTE: Pretty good **guesses**-->
-    <xacro:property name="wheel_pos_x" value="-0.022"/>
-    <xacro:property name="wheel_pos_y" value="0.065"/>
+    <xacro:property name="wheel_pos_y" value="0.022"/>
+    <xacro:property name="wheel_pos_z" value="0.063"/>
     <xacro:macro name="swerve_axle" params="prefix parent *origin">
         <link name="${prefix}_axle_link">
             <visual>
-                <origin xyz="0 0 0" rpy="0 0 0" />
+                <origin xyz="0 0 0" rpy="${pi} 0 ${pi/2}" />
                 <geometry>
                     <mesh filename="package://edna_description/meshes/SwerveAxle.stl" scale="0.001 0.001 0.001" />
@@ -22,6 +22,6 @@
                 <material name="blue" />
             </visual>
-            <xacro:inertial_cylinder mass="${axle_mass}" radius="${axle_radius}" length="${wheel_length}" >
-                <origin xyz="0 0 0" rpy="0 0 0" />
+            <xacro:inertial_cylinder mass="${axle_mass}" radius="${axle_radius}" length="${axle_length}" >
+                <origin xyz="0 0 -${axle_length/2}" rpy="0 0 0" />
             </xacro:inertial_cylinder>
         </link>
@@ -30,10 +30,10 @@
             <child link="${prefix}_axle_link" />
             <xacro:insert_block name="origin" />
-            <axis xyz="0 0 1" />
+            <axis xyz="0 0 -1" />
             <dynamics friction="0.1" />
         </joint>
         <link name="${prefix}_wheel_link">
             <visual>
-                <origin xyz="0 0 0" rpy="0 ${pi / 4} 0" />
+                <origin xyz="0 -${wheel_pos_y} 0" rpy="0 ${pi/4} ${pi/2}" />
                 <geometry>
                     <mesh filename="package://edna_description/meshes/SwerveWheel.stl" scale="0.001 0.001 0.001" />
@@ -42,5 +42,5 @@
             </visual>
             <collision>
-                <origin xyz="0.021 0 0" rpy="0 ${pi / 2} 0"/>
+                <origin xyz="0 0 0" rpy="${pi / 2} 0 0"/>
                 <geometry>
                     <cylinder  length="${wheel_length}" radius="${wheel_radius}"/>
@@ -48,5 +48,5 @@
             </collision>
             <xacro:inertial_cylinder mass="${wheel_mass}" radius="${wheel_radius}" length="${wheel_length}" >
-                <origin xyz="0 0 0" rpy="0 ${pi / 2} 0" />
+                <origin xyz="0 0 0" rpy="${pi / 2} 0 0" />
             </xacro:inertial_cylinder>
         </link>
@@ -54,6 +54,6 @@
             <parent link="${prefix}_axle_link" />
             <child link="${prefix}_wheel_link" />
-            <origin xyz="${wheel_pos_x} 0 ${wheel_pos_y}" rpy="0 0 0"/>
-            <axis xyz="1 0 0" />
+            <origin xyz="0 0 -${wheel_pos_z}" rpy="0 0 0"/>
+            <axis xyz="0 1 0" />
             <dynamics friction="0.1" />
         </joint>

File: src/edna_description/urdf/robots/edna.urdf.xacro (robot description, xacro)
@@ -13,19 +13,22 @@
   <!-- Axle Position Variables -->
   <xacro:property name="axle_pos" value="${301.625 / 1000}" />
-  <xacro:property name="axle_pos_y" value="${69.056 / 1000}" />
+  <xacro:property name="axle_pos_z" value="${69.056 / 1000}" />
   <!-- Camera Position Variables -->
   <xacro:property name="cam_pos" value=".3575 0.085 0.0"/> <!-- Made up values, replace with real ones later. -->
+  <!-- X IS FORWARD -->
+  <!-- Y IS LEFT -->
+  <!-- Z IS UP -->
   <xacro:square_chassis prefix="swerve" />
   <xacro:swerve_axle prefix="front_left" parent="swerve_chassis_link">
-    <origin xyz="${axle_pos} ${axle_pos_y} ${axle_pos}" rpy="${pi / 2} 0 0" />
+    <origin xyz="${axle_pos} ${axle_pos} ${axle_pos_z}" rpy="0 0 0" />
   </xacro:swerve_axle>
   <xacro:swerve_axle prefix="front_right" parent="swerve_chassis_link">
-    <origin xyz="-${axle_pos} ${axle_pos_y} ${axle_pos}" rpy="${pi / 2} 0 0" />
+    <origin xyz="${axle_pos} -${axle_pos} ${axle_pos_z}" rpy="0 0 0" />
   </xacro:swerve_axle>
   <xacro:swerve_axle prefix="rear_left" parent="swerve_chassis_link">
-    <origin xyz="${axle_pos} ${axle_pos_y} -${axle_pos}" rpy="${pi / 2} 0 0" />
+    <origin xyz="-${axle_pos} ${axle_pos} ${axle_pos_z} " rpy="0 0 0" />
   </xacro:swerve_axle>
   <xacro:swerve_axle prefix="rear_right" parent="swerve_chassis_link">
-    <origin xyz="-${axle_pos} ${axle_pos_y} -${axle_pos}" rpy="${pi / 2} 0 0" />
+    <origin xyz="-${axle_pos} -${axle_pos} ${axle_pos_z}" rpy="0 0 0" />
   </xacro:swerve_axle>
   <xacro:zed_camera name="zed_camera" model="zed2i" parent="swerve_chassis_link">

Commit message: Remove imu fix urdf - Gage

File: isaac/exts/omni.isaac.edna/omni/isaac/edna/edna.urdf (robot description, URDF)
Before this commit: robot edna, 10 links, 9 joints
Links:
- added link imu_sensor_link, mass 0.001; collision box size=0.02 0.02 0.02; visual box size=0.02 0.02 0.02
- added link zed_camera_base_link
- added link zed_camera_camera_center; collision mesh filename=package://edna_description/meshes/zed2i.stl; visual mesh filename=package://edna_description/meshes/zed2i.stl
- added link zed_camera_left_camera_frame
- added link zed_camera_left_camera_optical_frame
- added link zed_camera_right_camera_frame
- added link zed_camera_right_camera_optical_frame
Joints:
- added joint imu_sensor_joint: type fixed, parent swerve_chassis_link, child imu_sensor_link, axis 0 0 1
- added joint zed_camera_base_joint: type fixed, parent swerve_chassis_link, child zed_camera_base_link, origin xyz=.3575 0.085 0.0 rpy=1.5707963267948966 0 0
- added joint zed_camera_camera_center_joint: type fixed, parent zed_camera_base_link, child zed_camera_camera_center, origin xyz=0 0 0.015 rpy=0 0.0 0
- added joint zed_camera_left_camera_joint: type fixed, parent zed_camera_camera_center, child zed_camera_left_camera_frame, origin xyz=0 0.06 0 rpy=0 0 0
- added joint zed_camera_left_camera_optical_joint: type fixed, parent zed_camera_left_camera_frame, child zed_camera_left_camera_optical_frame, origin xyz=-0.01 0 0 rpy=-1.5707963267948966 0.0 -1.5707963267948966
- added joint zed_camera_right_camera_joint: type fixed, parent zed_camera_camera_center, child zed_camera_right_camera_frame, origin xyz=0 -0.06 0 rpy=0 0 0
- added joint zed_camera_right_camera_optical_joint: type fixed, parent zed_camera_right_camera_frame, child zed_camera_right_camera_optical_frame, origin xyz=-0.01 0 0 rpy=-1.5707963267948966 0.0 -1.5707963267948966

File: src/edna_description/urdf/edna.urdf (robot description, URDF)
Before this commit: robot edna, 17 links, 16 joints
Links:
- removed link imu_sensor_link
- removed link zed_camera_base_link
- removed link zed_camera_camera_center
- removed link zed_camera_left_camera_frame
- removed link zed_camera_left_camera_optical_frame
- removed link zed_camera_right_camera_frame
- removed link zed_camera_right_camera_optical_frame
- link swerve_chassis_link: geometry collision box size=0.7366 0.7366 0.05588; visual mesh filename=package://edna_description/meshes/SwerveChassis.stl scale=0.001 0.001 0.001
Joints:
- removed joint imu_sensor_joint
- removed joint zed_camera_base_joint
- removed joint zed_camera_camera_center_joint
- removed joint zed_camera_left_camera_joint
- removed joint zed_camera_left_camera_optical_joint
- removed joint zed_camera_right_camera_joint
- removed joint zed_camera_right_camera_optical_joint
- joint front_left_axle_joint: axis 0 0 1 -> 0 0 -1; origin xyz=0.301625 0.06905599999999999 0.301625 rpy=1.5707963267948966 0 0 -> xyz=0.301625 0.301625 0.06905599999999999 rpy=0 0 0
- joint front_left_wheel_joint: axis 1 0 0 -> 0 1 0; origin xyz=-0.022 0 0.065 rpy=0 0 0 -> xyz=0 0 -0.063 rpy=0 0 0
- joint front_right_axle_joint: axis 0 0 1 -> 0 0 -1; origin xyz=-0.301625 0.06905599999999999 0.301625 rpy=1.5707963267948966 0 0 -> xyz=0.301625 -0.301625 0.06905599999999999 rpy=0 0 0
- joint front_right_wheel_joint: axis 1 0 0 -> 0 1 0; origin xyz=-0.022 0 0.065 rpy=0 0 0 -> xyz=0 0 -0.063 rpy=0 0 0
- joint rear_left_axle_joint: axis 0 0 1 -> 0 0 -1; origin xyz=0.301625 0.06905599999999999 -0.301625 rpy=1.5707963267948966 0 0 -> xyz=-0.301625 0.301625 0.06905599999999999  rpy=0 0 0
- joint rear_left_wheel_joint: axis 1 0 0 -> 0 1 0; origin xyz=-0.022 0 0.065 rpy=0 0 0 -> xyz=0 0 -0.063 rpy=0 0 0
- joint rear_right_axle_joint: axis 0 0 1 -> 0 0 -1; origin xyz=-0.301625 0.06905599999999999 -0.301625 rpy=1.5707963267948966 0 0 -> xyz=-0.301625 -0.301625 0.06905599999999999 rpy=0 0 0
- joint rear_right_wheel_joint: axis 1 0 0 -> 0 1 0; origin xyz=-0.022 0 0.065 rpy=0 0 0 -> xyz=0 0 -0.063 rpy=0 0 0
- joint swerve_chassis_joint: origin xyz=0 0 0 rpy=1.5707963267948966 0 0 -> xyz=0 0 0 rpy=0 0 0

File: src/edna_description/urdf/parts/zed_macro.urdf.xacro (robot description, xacro)
@@ -16,5 +16,4 @@
 -->
 <robot xmlns:xacro="http://wiki.ros.org/xacro">
-  <xacro:include filename="$(find edna_description)/urdf/util/materials.xacro" />
   <xacro:property name="M_PI"     value="3.1415926535897931" />
   <!--

File: src/edna_description/urdf/robots/edna.urdf.xacro (robot description, xacro)
@@ -10,5 +10,4 @@
   <xacro:include filename="$(find edna_description)/urdf/parts/swerve_axle.xacro" />
   <xacro:include filename="$(find edna_description)/urdf/parts/zed_macro.urdf.xacro" />
-  <xacro:include filename="$(find edna_description)/urdf/parts/imu.urdf.xacro" />
   <!-- Axle Position Variables -->
   <xacro:property name="axle_pos" value="${301.625 / 1000}" />
@@ -35,7 +34,4 @@
     <origin xyz="${cam_pos}" rpy="${pi/2} 0 0" />
   </xacro:zed_camera>
-  <xacro:imu_sensor parent="swerve_chassis_link">
-    <origin xyz="0 0 0" rpy="${pi/2} 0 0" />
-  </xacro:imu_sensor>
   <xacro:swerve_drive_control plugin="$(arg hw_interface_plugin)" />
 </robot>
