Commit message: Add prim path change

File: src/edna_description/urdf/edna.urdf (robot description, URDF)
Before this commit: robot edna, 10 links, 9 joints
Links:
- added link zed_camera_base_link
- added link zed_camera_camera_center; collision mesh filename=package://edna_description/meshes/zed2i.stl; visual mesh filename=package://edna_description/meshes/zed2i.stl
- added link zed_camera_left_camera_frame
- added link zed_camera_left_camera_optical_frame
- added link zed_camera_right_camera_frame
- added link zed_camera_right_camera_optical_frame
Joints:
- added joint zed_camera_base_joint: type fixed, parent swerve_chassis_link, child zed_camera_base_link, origin xyz=0 0 0.3 rpy=0 0 0
- added joint zed_camera_camera_center_joint: type fixed, parent zed_camera_base_link, child zed_camera_camera_center, origin xyz=0 0 0.015 rpy=0 0.0 0
- added joint zed_camera_left_camera_joint: type fixed, parent zed_camera_camera_center, child zed_camera_left_camera_frame, origin xyz=0 0.06 0 rpy=0 0 0
- added joint zed_camera_left_camera_optical_joint: type fixed, parent zed_camera_left_camera_frame, child zed_camera_left_camera_optical_frame, origin xyz=-0.01 0 0 rpy=-1.5707963267948966 0.0 -1.5707963267948966
- added joint zed_camera_right_camera_joint: type fixed, parent zed_camera_camera_center, child zed_camera_right_camera_frame, origin xyz=0 -0.06 0 rpy=0 0 0
- added joint zed_camera_right_camera_optical_joint: type fixed, parent zed_camera_right_camera_frame, child zed_camera_right_camera_optical_frame, origin xyz=-0.01 0 0 rpy=-1.5707963267948966 0.0 -1.5707963267948966

Commit message: Add odom transform frame

File: src/edna_description/urdf/edna.urdf (robot description, URDF)
Before this commit: robot edna, 16 links, 15 joints
Joints:
- joint front_left_axle_joint: parent swerve_chassis_link -> base_link
- joint front_right_axle_joint: parent swerve_chassis_link -> base_link
- joint rear_left_axle_joint: parent swerve_chassis_link -> base_link
- joint rear_right_axle_joint: parent swerve_chassis_link -> base_link

File: src/edna_description/urdf/parts/square_chassis.xacro (robot description, xacro)
@@ -6,6 +6,5 @@
   <xacro:property name="chassis_height" value="0.05588" />
   <xacro:property name="chassis_weight" value="19.0508795" />
-  <xacro:macro name="square_chassis" params="prefix">
-    <link name="base_link"></link>
+  <xacro:macro name="square_chassis" params="prefix parent *origin">
     <link name="${prefix}_chassis_link">
       <xacro:inertial_box mass="${chassis_weight}" x="${chassis_length}" y="${chassis_width}" z="${chassis_height}">
@@ -27,7 +26,7 @@
     </link>
     <joint name="${prefix}_chassis_joint" type="fixed">
-      <parent link="base_link" />
+      <parent link="${parent}" />
       <child link="${prefix}_chassis_link" />
-      <origin xyz="0 0 0" rpy="0 0 0" />
+      <xacro:insert_block name="origin" />
     </joint>
   </xacro:macro>

File: src/edna_description/urdf/robots/edna.urdf.xacro (robot description, xacro)
@@ -18,17 +18,23 @@
   <!-- Y IS LEFT -->
   <!-- Z IS UP -->
-  <xacro:square_chassis prefix="swerve" />
-  <xacro:swerve_axle prefix="front_left" parent="swerve_chassis_link">
+  <!-- Chassis -->
+  <link name="base_link"></link>
+  <xacro:square_chassis prefix="swerve" parent="base_link">
+    <origin xyz="0 0 0" rpy="0 0 0" />
+  </xacro:square_chassis>
+  <!-- Drive Train -->
+  <xacro:swerve_axle prefix="front_left" parent="base_link">
     <origin xyz="${axle_pos} ${axle_pos} ${axle_pos_z}" rpy="0 0 0" />
   </xacro:swerve_axle>
-  <xacro:swerve_axle prefix="front_right" parent="swerve_chassis_link">
+  <xacro:swerve_axle prefix="front_right" parent="base_link">
     <origin xyz="${axle_pos} -${axle_pos} ${axle_pos_z}" rpy="0 0 0" />
   </xacro:swerve_axle>
-  <xacro:swerve_axle prefix="rear_left" parent="swerve_chassis_link">
+  <xacro:swerve_axle prefix="rear_left" parent="base_link">
     <origin xyz="-${axle_pos} ${axle_pos} ${axle_pos_z} " rpy="0 0 0" />
   </xacro:swerve_axle>
-  <xacro:swerve_axle prefix="rear_right" parent="swerve_chassis_link">
+  <xacro:swerve_axle prefix="rear_right" parent="base_link">
     <origin xyz="-${axle_pos} -${axle_pos} ${axle_pos_z}" rpy="0 0 0" />
   </xacro:swerve_axle>
+  <!-- Sensors -->
   <xacro:zed_camera name="zed_camera" model="zed2i" parent="swerve_chassis_link">
     <origin xyz="${cam_pos}" rpy="0 0 0" />

Commit message: Add fixes for isaac display and urdf path

File: src/edna_description/urdf/edna.urdf (robot description, URDF)
Before this commit: robot edna, 16 links, 15 joints
Links:
- removed link zed_camera_base_link
- removed link zed_camera_camera_center
- removed link zed_camera_left_camera_frame
- removed link zed_camera_left_camera_optical_frame
- removed link zed_camera_right_camera_frame
- removed link zed_camera_right_camera_optical_frame
- added link zed_base_link
- added link zed_camera_center; collision mesh filename=package://edna_description/meshes/zed2i.stl; visual mesh filename=package://edna_description/meshes/zed2i.stl
- added link zed_left_camera_frame
- added link zed_left_camera_optical_frame
- added link zed_right_camera_frame
- added link zed_right_camera_optical_frame
Joints:
- removed joint zed_camera_base_joint
- removed joint zed_camera_camera_center_joint
- removed joint zed_camera_left_camera_joint
- removed joint zed_camera_left_camera_optical_joint
- removed joint zed_camera_right_camera_joint
- removed joint zed_camera_right_camera_optical_joint
- added joint zed_base_joint: type fixed, parent swerve_chassis_link, child zed_base_link, origin xyz=0 0 0.3 rpy=0 0 0
- added joint zed_camera_center_joint: type fixed, parent zed_base_link, child zed_camera_center, origin xyz=0 0 0.015 rpy=0 0.0 0
- added joint zed_left_camera_joint: type fixed, parent zed_camera_center, child zed_left_camera_frame, origin xyz=0 0.06 0 rpy=0 0 0
- added joint zed_left_camera_optical_joint: type fixed, parent zed_left_camera_frame, child zed_left_camera_optical_frame, origin xyz=-0.01 0 0 rpy=-1.5707963267948966 0.0 -1.5707963267948966
- added joint zed_right_camera_joint: type fixed, parent zed_camera_center, child zed_right_camera_frame, origin xyz=0 -0.06 0 rpy=0 0 0
- added joint zed_right_camera_optical_joint: type fixed, parent zed_right_camera_frame, child zed_right_camera_optical_frame, origin xyz=-0.01 0 0 rpy=-1.5707963267948966 0.0 -1.5707963267948966
- joint front_left_axle_joint: parent base_link -> swerve_chassis_link
- joint front_right_axle_joint: parent base_link -> swerve_chassis_link
- joint rear_left_axle_joint: parent base_link -> swerve_chassis_link
- joint rear_right_axle_joint: parent base_link -> swerve_chassis_link

File: src/edna_description/urdf/parts/zed_macro.urdf.xacro (robot description, xacro)
@@ -24,5 +24,5 @@
       - origin: the xyz/rpy offset from the parent link
   -->
-  <xacro:macro name="zed_camera" params="name=zed model=zed parent *origin">
+  <xacro:macro name="zed_camera" params="prefix=zed model=zed parent *origin">
     <xacro:if value="${model == 'zed'}">
       <xacro:property name="baseline" value="0.12" />
@@ -54,12 +54,12 @@
     </xacro:if>
     <!-- Camera mounting point (the threaded screw hole in the bottom) -->
-    <link name="${name}_base_link" />
-    <joint name="${name}_base_joint" type="fixed">
+    <link name="${prefix}_base_link" />
+    <joint name="${prefix}_base_joint" type="fixed">
       <parent link="${parent}"/>
-      <child link="${name}_base_link"/>
+      <child link="${prefix}_base_link"/>
       <xacro:insert_block name="origin" />
     </joint>
     <!-- Camera Center -->
-    <link name="${name}_camera_center">
+    <link name="${prefix}_camera_center">
       <visual>
         <origin xyz="${screw_offset_x} 0 0" rpy="0 0 0"/>
@@ -75,59 +75,59 @@
       </collision>
     </link>
-    <joint name="${name}_camera_center_joint" type="fixed">
-      <parent link="${name}_base_link"/>
-      <child link="${name}_camera_center"/>
+    <joint name="${prefix}_camera_center_joint" type="fixed">
+      <parent link="${prefix}_base_link"/>
+      <child link="${prefix}_camera_center"/>
       <origin xyz="0 0 ${height/2}" rpy="0 ${bottom_slope} 0" />
     </joint>
     <!-- Left Camera -->
-    <link name="${name}_left_camera_frame" />
-    <joint name="${name}_left_camera_joint" type="fixed">
-      <parent link="${name}_camera_center"/>
-      <child link="${name}_left_camera_frame"/>
+    <link name="${prefix}_left_camera_frame" />
+    <joint name="${prefix}_left_camera_joint" type="fixed">
+      <parent link="${prefix}_camera_center"/>
+      <child link="${prefix}_left_camera_frame"/>
       <origin xyz="0 ${baseline/2} 0" rpy="0 0 0" />
     </joint>
-    <link name="${name}_left_camera_optical_frame"/>
-    <joint name="${name}_left_camera_optical_joint" type="fixed">
+    <link name="${prefix}_left_camera_optical_frame"/>
+    <joint name="${prefix}_left_camera_optical_joint" type="fixed">
       <origin xyz="${optical_offset_x} 0 0" rpy="-${M_PI/2} 0.0 -${M_PI/2}"/>
-      <parent link="${name}_left_camera_frame"/>
-      <child link="${name}_left_camera_optical_frame"/>
+      <parent link="${prefix}_left_camera_frame"/>
+      <child link="${prefix}_left_camera_optical_frame"/>
     </joint>
     <!-- Right Camera -->
-    <link name="${name}_right_camera_frame" />
-    <joint name="${name}_right_camera_joint" type="fixed">
-      <parent link="${name}_camera_center"/>
-      <child link="${name}_right_camera_frame"/>
+    <link name="${prefix}_right_camera_frame" />
+    <joint name="${prefix}_right_camera_joint" type="fixed">
+      <parent link="${prefix}_camera_center"/>
+      <child link="${prefix}_right_camera_frame"/>
       <origin xyz="0 -${baseline/2} 0" rpy="0 0 0" />
     </joint>
-    <link name="${name}_right_camera_optical_frame"/>
-    <joint name="${name}_right_camera_optical_joint" type="fixed">
+    <link name="${prefix}_right_camera_optical_frame"/>
+    <joint name="${prefix}_right_camera_optical_joint" type="fixed">
       <origin xyz="${optical_offset_x} 0 0" rpy="-${M_PI/2} 0.0 -${M_PI/2}"/>
-      <parent link="${name}_right_camera_frame"/>
-      <child link="${name}_right_camera_optical_frame"/>
+      <parent link="${prefix}_right_camera_frame"/>
+      <child link="${prefix}_right_camera_optical_frame"/>
     </joint>
     <!-- ZED2 Sensors -->
     <xacro:if value="${model == 'zed2'}">
-      <link name="${name}_mag_link" />
-      <joint name="${name}_mag_joint" type="fixed">
-        <parent link="${name}_camera_center"/>
-        <child link="${name}_mag_link"/>
+      <link name="${prefix}_mag_link" />
+      <joint name="${prefix}_mag_joint" type="fixed">
+        <parent link="${prefix}_camera_center"/>
+        <child link="${prefix}_mag_link"/>
         <origin xyz="0 0 0" rpy="0 0 0" />
       </joint>
-      <link name="${name}_baro_link" />
-      <joint name="${name}_baro_joint" type="fixed">
-        <parent link="${name}_camera_center"/>
-        <child link="${name}_baro_link"/>
+      <link name="${prefix}_baro_link" />
+      <joint name="${prefix}_baro_joint" type="fixed">
+        <parent link="${prefix}_camera_center"/>
+        <child link="${prefix}_baro_link"/>
         <origin xyz="0 0 0" rpy="0 0 0" />
       </joint>
-      <link name="${name}_temp_left_link" />
-      <joint name="${name}_temp_left_joint" type="fixed">
-        <parent link="${name}_left_camera_frame"/>
-        <child link="${name}_temp_left_link"/>
+      <link name="${prefix}_temp_left_link" />
+      <joint name="${prefix}_temp_left_joint" type="fixed">
+        <parent link="${prefix}_left_camera_frame"/>
+        <child link="${prefix}_temp_left_link"/>
         <origin xyz="0 0 0" rpy="0 0 0" />
       </joint>
-      <link name="${name}_temp_right_link" />
-      <joint name="${name}_temp_right_joint" type="fixed">
-        <parent link="${name}_right_camera_frame"/>
-        <child link="${name}_temp_right_link"/>
+      <link name="${prefix}_temp_right_link" />
+      <joint name="${prefix}_temp_right_joint" type="fixed">
+        <parent link="${prefix}_right_camera_frame"/>
+        <child link="${prefix}_temp_right_link"/>
         <origin xyz="0 0 0" rpy="0 0 0" />
       </joint>

File: src/edna_description/urdf/robots/edna.urdf.xacro (robot description, xacro)
@@ -24,18 +24,18 @@
   </xacro:square_chassis>
   <!-- Drive Train -->
-  <xacro:swerve_axle prefix="front_left" parent="base_link">
+  <xacro:swerve_axle prefix="front_left" parent="swerve_chassis_link">
     <origin xyz="${axle_pos} ${axle_pos} ${axle_pos_z}" rpy="0 0 0" />
   </xacro:swerve_axle>
-  <xacro:swerve_axle prefix="front_right" parent="base_link">
+  <xacro:swerve_axle prefix="front_right" parent="swerve_chassis_link">
     <origin xyz="${axle_pos} -${axle_pos} ${axle_pos_z}" rpy="0 0 0" />
   </xacro:swerve_axle>
-  <xacro:swerve_axle prefix="rear_left" parent="base_link">
+  <xacro:swerve_axle prefix="rear_left" parent="swerve_chassis_link">
     <origin xyz="-${axle_pos} ${axle_pos} ${axle_pos_z} " rpy="0 0 0" />
   </xacro:swerve_axle>
-  <xacro:swerve_axle prefix="rear_right" parent="base_link">
+  <xacro:swerve_axle prefix="rear_right" parent="swerve_chassis_link">
     <origin xyz="-${axle_pos} -${axle_pos} ${axle_pos_z}" rpy="0 0 0" />
   </xacro:swerve_axle>
   <!-- Sensors -->
-  <xacro:zed_camera name="zed_camera" model="zed2i" parent="swerve_chassis_link">
+  <xacro:zed_camera prefix="zed" model="zed2i" parent="swerve_chassis_link">
     <origin xyz="${cam_pos}" rpy="0 0 0" />
   </xacro:zed_camera>

Commit message: Add graphs for cameras

File: src/edna_description/urdf/edna.urdf (robot description, URDF)
Before this commit: robot edna, 16 links, 15 joints
Joints:
- joint zed_left_camera_optical_joint: origin xyz=-0.01 0 0 rpy=-1.5707963267948966 0.0 -1.5707963267948966 -> xyz=-0.01 0 0 rpy=1.5707963267948966 0.0 -1.5707963267948966
- joint zed_right_camera_optical_joint: origin xyz=-0.01 0 0 rpy=-1.5707963267948966 0.0 -1.5707963267948966 -> xyz=-0.01 0 0 rpy=1.5707963267948966 0.0 -1.5707963267948966

File: src/edna_description/urdf/parts/zed_macro.urdf.xacro (robot description, xacro)
@@ -89,5 +89,5 @@
     <link name="${prefix}_left_camera_optical_frame"/>
     <joint name="${prefix}_left_camera_optical_joint" type="fixed">
-      <origin xyz="${optical_offset_x} 0 0" rpy="-${M_PI/2} 0.0 -${M_PI/2}"/>
+      <origin xyz="${optical_offset_x} 0 0" rpy="${M_PI/2} 0.0 -${M_PI/2}"/>
       <parent link="${prefix}_left_camera_frame"/>
       <child link="${prefix}_left_camera_optical_frame"/>
@@ -102,5 +102,5 @@
     <link name="${prefix}_right_camera_optical_frame"/>
     <joint name="${prefix}_right_camera_optical_joint" type="fixed">
-      <origin xyz="${optical_offset_x} 0 0" rpy="-${M_PI/2} 0.0 -${M_PI/2}"/>
+      <origin xyz="${optical_offset_x} 0 0" rpy="${M_PI/2} 0.0 -${M_PI/2}"/>
       <parent link="${prefix}_right_camera_frame"/>
       <child link="${prefix}_right_camera_optical_frame"/>

Commit message: Fix urdf optical transforms

File: src/edna_description/urdf/edna.urdf (robot description, URDF)
Before this commit: robot edna, 16 links, 15 joints
Joints:
- joint zed_left_camera_optical_joint: origin xyz=-0.01 0 0 rpy=1.5707963267948966 0.0 -1.5707963267948966 -> xyz=-0.01 0 0 rpy=1.5707963267948966 0.0 1.5707963267948966
- joint zed_right_camera_optical_joint: origin xyz=-0.01 0 0 rpy=1.5707963267948966 0.0 -1.5707963267948966 -> xyz=-0.01 0 0 rpy=1.5707963267948966 0.0 1.5707963267948966

File: src/edna_description/urdf/parts/zed_macro.urdf.xacro (robot description, xacro)
@@ -89,5 +89,5 @@
     <link name="${prefix}_left_camera_optical_frame"/>
     <joint name="${prefix}_left_camera_optical_joint" type="fixed">
-      <origin xyz="${optical_offset_x} 0 0" rpy="${M_PI/2} 0.0 -${M_PI/2}"/>
+      <origin xyz="${optical_offset_x} 0 0" rpy="${M_PI/2} 0.0 ${M_PI/2}"/>
       <parent link="${prefix}_left_camera_frame"/>
       <child link="${prefix}_left_camera_optical_frame"/>
@@ -102,5 +102,5 @@
     <link name="${prefix}_right_camera_optical_frame"/>
     <joint name="${prefix}_right_camera_optical_joint" type="fixed">
-      <origin xyz="${optical_offset_x} 0 0" rpy="${M_PI/2} 0.0 -${M_PI/2}"/>
+      <origin xyz="${optical_offset_x} 0 0" rpy="${M_PI/2} 0.0 ${M_PI/2}"/>
       <parent link="${prefix}_right_camera_frame"/>
       <child link="${prefix}_right_camera_optical_frame"/>

Commit message: finally fix urdf frames

File: src/edna_description/urdf/edna.urdf (robot description, URDF)
Before this commit: robot edna, 16 links, 15 joints
Joints:
- joint zed_left_camera_joint: origin xyz=0 0.06 0 rpy=0 0 0 -> xyz=0 0.06 0 rpy=-1.5707963267948966 0 -1.5707963267948966
- joint zed_left_camera_optical_joint: origin xyz=-0.01 0 0 rpy=1.5707963267948966 0.0 1.5707963267948966 -> xyz=0 0 -0.01 rpy=3.141592653589793 0 0
- joint zed_right_camera_joint: origin xyz=0 -0.06 0 rpy=0 0 0 -> xyz=0 -0.06 0 rpy=-1.5707963267948966 0 -1.5707963267948966
- joint zed_right_camera_optical_joint: origin xyz=-0.01 0 0 rpy=1.5707963267948966 0.0 1.5707963267948966 -> xyz=0 0 -0.01 rpy=3.141592653589793 0 0

File: src/edna_description/urdf/parts/zed_macro.urdf.xacro (robot description, xacro)
@@ -85,9 +85,9 @@
       <parent link="${prefix}_camera_center"/>
       <child link="${prefix}_left_camera_frame"/>
-      <origin xyz="0 ${baseline/2} 0" rpy="0 0 0" />
+      <origin xyz="0 ${baseline/2} 0" rpy="-${M_PI/2} 0 -${M_PI/2}" />
     </joint>
     <link name="${prefix}_left_camera_optical_frame"/>
     <joint name="${prefix}_left_camera_optical_joint" type="fixed">
-      <origin xyz="${optical_offset_x} 0 0" rpy="${M_PI/2} 0.0 ${M_PI/2}"/>
+      <origin xyz="0 0 ${optical_offset_x}" rpy="${M_PI} 0 0"/>
       <parent link="${prefix}_left_camera_frame"/>
       <child link="${prefix}_left_camera_optical_frame"/>
@@ -98,9 +98,9 @@
       <parent link="${prefix}_camera_center"/>
       <child link="${prefix}_right_camera_frame"/>
-      <origin xyz="0 -${baseline/2} 0" rpy="0 0 0" />
+      <origin xyz="0 -${baseline/2} 0" rpy="-${M_PI/2} 0 -${M_PI/2}" />
     </joint>
     <link name="${prefix}_right_camera_optical_frame"/>
     <joint name="${prefix}_right_camera_optical_joint" type="fixed">
-      <origin xyz="${optical_offset_x} 0 0" rpy="${M_PI/2} 0.0 ${M_PI/2}"/>
+      <origin xyz="0 0 ${optical_offset_x}" rpy="${M_PI} 0 0"/>
       <parent link="${prefix}_right_camera_frame"/>
       <child link="${prefix}_right_camera_optical_frame"/>

Commit message: Sim depth camera (#33)
* Add graphs for cameras

* Fix urdf optical transforms

* finally fix urdf frames

* Added display fixes

File: src/edna_description/urdf/edna.urdf (robot description, URDF)
Before this commit: robot edna, 16 links, 15 joints
Joints:
- joint zed_left_camera_joint: origin xyz=0 0.06 0 rpy=0 0 0 -> xyz=0 0.06 0 rpy=-1.5707963267948966 0 -1.5707963267948966
- joint zed_left_camera_optical_joint: origin xyz=-0.01 0 0 rpy=-1.5707963267948966 0.0 -1.5707963267948966 -> xyz=0 0 -0.01 rpy=3.141592653589793 0 0
- joint zed_right_camera_joint: origin xyz=0 -0.06 0 rpy=0 0 0 -> xyz=0 -0.06 0 rpy=-1.5707963267948966 0 -1.5707963267948966
- joint zed_right_camera_optical_joint: origin xyz=-0.01 0 0 rpy=-1.5707963267948966 0.0 -1.5707963267948966 -> xyz=0 0 -0.01 rpy=3.141592653589793 0 0

File: src/edna_description/urdf/parts/zed_macro.urdf.xacro (robot description, xacro)
@@ -85,9 +85,9 @@
       <parent link="${prefix}_camera_center"/>
       <child link="${prefix}_left_camera_frame"/>
-      <origin xyz="0 ${baseline/2} 0" rpy="0 0 0" />
+      <origin xyz="0 ${baseline/2} 0" rpy="-${M_PI/2} 0 -${M_PI/2}" />
     </joint>
     <link name="${prefix}_left_camera_optical_frame"/>
     <joint name="${prefix}_left_camera_optical_joint" type="fixed">
-      <origin xyz="${optical_offset_x} 0 0" rpy="-${M_PI/2} 0.0 -${M_PI/2}"/>
+      <origin xyz="0 0 ${optical_offset_x}" rpy="${M_PI} 0 0"/>
       <parent link="${prefix}_left_camera_frame"/>
       <child link="${prefix}_left_camera_optical_frame"/>
@@ -98,9 +98,9 @@
       <parent link="${prefix}_camera_center"/>
       <child link="${prefix}_right_camera_frame"/>
-      <origin xyz="0 -${baseline/2} 0" rpy="0 0 0" />
+      <origin xyz="0 -${baseline/2} 0" rpy="-${M_PI/2} 0 -${M_PI/2}" />
     </joint>
     <link name="${prefix}_right_camera_optical_frame"/>
     <joint name="${prefix}_right_camera_optical_joint" type="fixed">
-      <origin xyz="${optical_offset_x} 0 0" rpy="-${M_PI/2} 0.0 -${M_PI/2}"/>
+      <origin xyz="0 0 ${optical_offset_x}" rpy="${M_PI} 0 0"/>
       <parent link="${prefix}_right_camera_frame"/>
       <child link="${prefix}_right_camera_optical_frame"/>

Commit message: Create the Lidar in the description - The lidar is now in the URDF - The graph is fully connected

File: src/edna_description/urdf/edna.urdf (robot description, URDF)
Before this commit: robot edna, 16 links, 15 joints
Links:
- added link lidar_link; collision cylinder length=0.025 radius=0.035; visual cylinder length=0.025 radius=0.035
Joints:
- added joint lidar_joint: type fixed, parent swerve_chassis_link, child lidar_link, origin xyz=0 0 .035 rpy=0 0 0

File: src/edna_description/urdf/robots/edna.urdf.xacro (robot description, xacro)
@@ -10,4 +10,5 @@
   <xacro:include filename="$(find edna_description)/urdf/parts/swerve_axle.xacro" />
   <xacro:include filename="$(find edna_description)/urdf/parts/zed_macro.urdf.xacro" />
+  <xacro:include filename="$(find edna_description)/urdf/parts/lidar.xacro" />
   <!-- Axle Position Variables -->
   <xacro:property name="axle_pos" value="${301.625 / 1000}" />
@@ -40,4 +41,7 @@
     <origin xyz="${cam_pos}" rpy="0 0 0" />
   </xacro:zed_camera>
+  <xacro:lidar parent="swerve_chassis_link" radius="0.035" length="0.025">
+    <origin xyz="0 0 .035" rpy="0 0 0" />
+  </xacro:lidar>
   <xacro:swerve_drive_control plugin="$(arg hw_interface_plugin)" />
 </robot>
