Commit message: Add namespace to all links

File: src/edna_description/urdf/edna.urdf (robot description, URDF)
Before this commit: robot edna, 16 links, 15 joints
Links:
- removed link front_left_axle_link
- removed link front_left_wheel_link
- removed link front_right_axle_link
- removed link front_right_wheel_link
- removed link rear_left_axle_link
- removed link rear_left_wheel_link
- removed link rear_right_axle_link
- removed link rear_right_wheel_link
- removed link swerve_chassis_link
- removed link zed_base_link
- removed link zed_camera_center
- removed link zed_left_camera_frame
- removed link zed_left_camera_optical_frame
- removed link zed_right_camera_frame
- removed link zed_right_camera_optical_frame
- added link default_front_left_axle_link, mass 0.23739; visual mesh filename=package://edna_description/meshes/SwerveAxle.stl scale=0.001 0.001 0.001
- added link default_front_left_wheel_link, mass 0.23133211; collision cylinder length=0.0381 radius=0.0508; visual mesh filename=package://edna_description/meshes/SwerveWheel.stl scale=0.001 0.001 0.001
- added link default_front_right_axle_link, mass 0.23739; visual mesh filename=package://edna_description/meshes/SwerveAxle.stl scale=0.001 0.001 0.001
- added link default_front_right_wheel_link, mass 0.23133211; collision cylinder length=0.0381 radius=0.0508; visual mesh filename=package://edna_description/meshes/SwerveWheel.stl scale=0.001 0.001 0.001
- added link default_rear_left_axle_link, mass 0.23739; visual mesh filename=package://edna_description/meshes/SwerveAxle.stl scale=0.001 0.001 0.001
- added link default_rear_left_wheel_link, mass 0.23133211; collision cylinder length=0.0381 radius=0.0508; visual mesh filename=package://edna_description/meshes/SwerveWheel.stl scale=0.001 0.001 0.001
- added link default_rear_right_axle_link, mass 0.23739; visual mesh filename=package://edna_description/meshes/SwerveAxle.stl scale=0.001 0.001 0.001
- added link default_rear_right_wheel_link, mass 0.23133211; collision cylinder length=0.0381 radius=0.0508; visual mesh filename=package://edna_description/meshes/SwerveWheel.stl scale=0.001 0.001 0.001
- added link default_swerve_chassis_link, mass 19.0508795; collision box size=0.7366 0.7366 0.05588; visual mesh filename=package://edna_description/meshes/SwerveChassis.stl scale=0.001 0.001 0.001
- added link default_zed_base_link
- added link default_zed_camera_center; collision mesh filename=package://edna_description/meshes/zed2i.stl; visual mesh filename=package://edna_description/meshes/zed2i.stl
- added link default_zed_left_camera_frame
- added link default_zed_left_camera_optical_frame
- added link default_zed_right_camera_frame
- added link default_zed_right_camera_optical_frame
Joints:
- removed joint front_left_axle_joint
- removed joint front_left_wheel_joint
- removed joint front_right_axle_joint
- removed joint front_right_wheel_joint
- removed joint rear_left_axle_joint
- removed joint rear_left_wheel_joint
- removed joint rear_right_axle_joint
- removed joint rear_right_wheel_joint
- removed joint swerve_chassis_joint
- removed joint zed_base_joint
- removed joint zed_camera_center_joint
- removed joint zed_left_camera_joint
- removed joint zed_left_camera_optical_joint
- removed joint zed_right_camera_joint
- removed joint zed_right_camera_optical_joint
- added joint default_front_left_axle_joint: type continuous, parent default_swerve_chassis_link, child default_front_left_axle_link, origin xyz=0.301625 0.301625 0.06905599999999999 rpy=0 0 0, axis 0 0 -1
- added joint default_front_left_wheel_joint: type continuous, parent default_front_left_axle_link, child default_front_left_wheel_link, origin xyz=0 0 -0.063 rpy=0 0 0, axis 0 1 0
- added joint default_front_right_axle_joint: type continuous, parent default_swerve_chassis_link, child default_front_right_axle_link, origin xyz=0.301625 -0.301625 0.06905599999999999 rpy=0 0 0, axis 0 0 -1
- added joint default_front_right_wheel_joint: type continuous, parent default_front_right_axle_link, child default_front_right_wheel_link, origin xyz=0 0 -0.063 rpy=0 0 0, axis 0 1 0
- added joint default_rear_left_axle_joint: type continuous, parent default_swerve_chassis_link, child default_rear_left_axle_link, origin xyz=-0.301625 0.301625 0.06905599999999999  rpy=0 0 0, axis 0 0 -1
- added joint default_rear_left_wheel_joint: type continuous, parent default_rear_left_axle_link, child default_rear_left_wheel_link, origin xyz=0 0 -0.063 rpy=0 0 0, axis 0 1 0
- added joint default_rear_right_axle_joint: type continuous, parent default_swerve_chassis_link, child default_rear_right_axle_link, origin xyz=-0.301625 -0.301625 0.06905599999999999 rpy=0 0 0, axis 0 0 -1
- added joint default_rear_right_wheel_joint: type continuous, parent default_rear_right_axle_link, child default_rear_right_wheel_link, origin xyz=0 0 -0.063 rpy=0 0 0, axis 0 1 0
- added joint default_swerve_chassis_joint: type fixed, parent base_link, child default_swerve_chassis_link, origin xyz=0 0 0 rpy=0 0 0
- added joint default_zed_base_joint: type fixed, parent default_swerve_chassis_link, child default_zed_base_link, origin xyz=0 0 0.3 rpy=0 0 0
- added joint default_zed_camera_center_joint: type fixed, parent default_zed_base_link, child default_zed_camera_center, origin xyz=0 0 0.015 rpy=0 0.0 0
- added joint default_zed_left_camera_joint: type fixed, parent default_zed_camera_center, child default_zed_left_camera_frame, origin xyz=0 0.06 0 rpy=-1.5707963267948966 0 -1.5707963267948966
- added joint default_zed_left_camera_optical_joint: type fixed, parent default_zed_left_camera_frame, child default_zed_left_camera_optical_frame, origin xyz=0 0 -0.01 rpy=3.141592653589793 0 0
- added joint default_zed_right_camera_joint: type fixed, parent default_zed_camera_center, child default_zed_right_camera_frame, origin xyz=0 -0.06 0 rpy=-1.5707963267948966 0 -1.5707963267948966
- added joint default_zed_right_camera_optical_joint: type fixed, parent default_zed_right_camera_frame, child default_zed_right_camera_optical_frame, origin xyz=0 0 -0.01 rpy=3.141592653589793 0 0

File: src/edna_description/urdf/robots/edna.urdf.xacro (robot description, xacro)
@@ -3,4 +3,6 @@
   <!-- Args -->
   <xacro:arg name="hw_interface_plugin" default="swerve_hardware/IsaacDriveHardware"/>
+  <xacro:arg name="namespace" default="default"/>
+  <xacro:property name="ns" value="$(arg namespace)" />
   <!-- Include Files -->
   <xacro:include filename="$(find edna_description)/urdf/control/drive.xacro" />
@@ -20,22 +22,22 @@
   <!-- Chassis -->
   <link name="base_link"></link>
-  <xacro:square_chassis prefix="swerve" parent="base_link">
+  <xacro:square_chassis prefix="${ns}_swerve" parent="base_link">
     <origin xyz="0 0 0" rpy="0 0 0" />
   </xacro:square_chassis>
   <!-- Drive Train -->
-  <xacro:swerve_axle prefix="front_left" parent="swerve_chassis_link">
+  <xacro:swerve_axle prefix="${ns}_front_left" parent="${ns}_swerve_chassis_link">
     <origin xyz="${axle_pos} ${axle_pos} ${axle_pos_z}" rpy="0 0 0" />
   </xacro:swerve_axle>
-  <xacro:swerve_axle prefix="front_right" parent="swerve_chassis_link">
+  <xacro:swerve_axle prefix="${ns}_front_right" parent="${ns}_swerve_chassis_link">
     <origin xyz="${axle_pos} -${axle_pos} ${axle_pos_z}" rpy="0 0 0" />
   </xacro:swerve_axle>
-  <xacro:swerve_axle prefix="rear_left" parent="swerve_chassis_link">
+  <xacro:swerve_axle prefix="${ns}_rear_left" parent="${ns}_swerve_chassis_link">
     <origin xyz="-${axle_pos} ${axle_pos} ${axle_pos_z} " rpy="0 0 0" />
   </xacro:swerve_axle>
-  <xacro:swerve_axle prefix="rear_right" parent="swerve_chassis_link">
+  <xacro:swerve_axle prefix="${ns}_rear_right" parent="${ns}_swerve_chassis_link">
     <origin xyz="-${axle_pos} -${axle_pos} ${axle_pos_z}" rpy="0 0 0" />
   </xacro:swerve_axle>
   <!-- Sensors -->
-  <xacro:zed_camera prefix="zed" model="zed2i" parent="swerve_chassis_link">
+  <xacro:zed_camera prefix="${ns}_zed" model="zed2i" parent="${ns}_swerve_chassis_link">
     <origin xyz="${cam_pos}" rpy="0 0 0" />
   </xacro:zed_camera>

Commit message: Namespaced descriptions (#45)
* Add namespace to all links

* Rviz working

* Add Add ns to drive component

* Put joints in launch file

* Add to test_hw and isaa launch

* Add namespaces to links in extension

* Fix autocomplete

File: src/edna_description/urdf/edna.urdf (robot description, URDF)
Before this commit: robot edna, 16 links, 15 joints
Links:
- removed link front_left_axle_link
- removed link front_left_wheel_link
- removed link front_right_axle_link
- removed link front_right_wheel_link
- removed link rear_left_axle_link
- removed link rear_left_wheel_link
- removed link rear_right_axle_link
- removed link rear_right_wheel_link
- removed link swerve_chassis_link
- removed link zed_base_link
- removed link zed_camera_center
- removed link zed_left_camera_frame
- removed link zed_left_camera_optical_frame
- removed link zed_right_camera_frame
- removed link zed_right_camera_optical_frame
- added link default_front_left_axle_link, mass 0.23739; visual mesh filename=package://edna_description/meshes/SwerveAxle.stl scale=0.001 0.001 0.001
- added link default_front_left_wheel_link, mass 0.23133211; collision cylinder length=0.0381 radius=0.0508; visual mesh filename=package://edna_description/meshes/SwerveWheel.stl scale=0.001 0.001 0.001
- added link default_front_right_axle_link, mass 0.23739; visual mesh filename=package://edna_description/meshes/SwerveAxle.stl scale=0.001 0.001 0.001
- added link default_front_right_wheel_link, mass 0.23133211; collision cylinder length=0.0381 radius=0.0508; visual mesh filename=package://edna_description/meshes/SwerveWheel.stl scale=0.001 0.001 0.001
- added link default_rear_left_axle_link, mass 0.23739; visual mesh filename=package://edna_description/meshes/SwerveAxle.stl scale=0.001 0.001 0.001
- added link default_rear_left_wheel_link, mass 0.23133211; collision cylinder length=0.0381 radius=0.0508; visual mesh filename=package://edna_description/meshes/SwerveWheel.stl scale=0.001 0.001 0.001
- added link default_rear_right_axle_link, mass 0.23739; visual mesh filename=package://edna_description/meshes/SwerveAxle.stl scale=0.001 0.001 0.001
- added link default_rear_right_wheel_link, mass 0.23133211; collision cylinder length=0.0381 radius=0.0508; visual mesh filename=package://edna_description/meshes/SwerveWheel.stl scale=0.001 0.001 0.001
- added link default_swerve_chassis_link, mass 19.0508795; collision box size=0.7366 0.7366 0.05588; visual mesh filename=package://edna_description/meshes/SwerveChassis.stl scale=0.001 0.001 0.001
- added link default_zed_base_link
- added link default_zed_camera_center; collision mesh filename=package://edna_description/meshes/zed2i.stl; visual mesh filename=package://edna_description/meshes/zed2i.stl
- added link default_zed_left_camera_frame
- added link default_zed_left_camera_optical_frame
- added link default_zed_right_camera_frame
- added link default_zed_right_camera_optical_frame
Joints:
- removed joint front_left_axle_joint
- removed joint front_left_wheel_joint
- removed joint front_right_axle_joint
- removed joint front_right_wheel_joint
- removed joint rear_left_axle_joint
- removed joint rear_left_wheel_joint
- removed joint rear_right_axle_joint
- removed joint rear_right_wheel_joint
- removed joint swerve_chassis_joint
- removed joint zed_base_joint
- removed joint zed_camera_center_joint
- removed joint zed_left_camera_joint
- removed joint zed_left_camera_optical_joint
- removed joint zed_right_camera_joint
- removed joint zed_right_camera_optical_joint
- added joint default_front_left_axle_joint: type continuous, parent default_swerve_chassis_link, child default_front_left_axle_link, origin xyz=0.301625 0.301625 0.06905599999999999 rpy=0 0 0, axis 0 0 -1
- added joint default_front_left_wheel_joint: type continuous, parent default_front_left_axle_link, child default_front_left_wheel_link, origin xyz=0 0 -0.063 rpy=0 0 0, axis 0 1 0
- added joint default_front_right_axle_joint: type continuous, parent default_swerve_chassis_link, child default_front_right_axle_link, origin xyz=0.301625 -0.301625 0.06905599999999999 rpy=0 0 0, axis 0 0 -1
- added joint default_front_right_wheel_joint: type continuous, parent default_front_right_axle_link, child default_front_right_wheel_link, origin xyz=0 0 -0.063 rpy=0 0 0, axis 0 1 0
- added joint default_rear_left_axle_joint: type continuous, parent default_swerve_chassis_link, child default_rear_left_axle_link, origin xyz=-0.301625 0.301625 0.06905599999999999  rpy=0 0 0, axis 0 0 -1
- added joint default_rear_left_wheel_joint: type continuous, parent default_rear_left_axle_link, child default_rear_left_wheel_link, origin xyz=0 0 -0.063 rpy=0 0 0, axis 0 1 0
- added joint default_rear_right_axle_joint: type continuous, parent default_swerve_chassis_link, child default_rear_right_axle_link, origin xyz=-0.301625 -0.301625 0.06905599999999999 rpy=0 0 0, axis 0 0 -1
- added joint default_rear_right_wheel_joint: type continuous, parent default_rear_right_axle_link, child default_rear_right_wheel_link, origin xyz=0 0 -0.063 rpy=0 0 0, axis 0 1 0
- added joint default_swerve_chassis_joint: type fixed, parent base_link, child default_swerve_chassis_link, origin xyz=0 0 0 rpy=0 0 0
- added joint default_zed_base_joint: type fixed, parent default_swerve_chassis_link, child default_zed_base_link, origin xyz=0 0 0.3 rpy=0 0 0
- added joint default_zed_camera_center_joint: type fixed, parent default_zed_base_link, child default_zed_camera_center, origin xyz=0 0 0.015 rpy=0 0.0 0
- added joint default_zed_left_camera_joint: type fixed, parent default_zed_camera_center, child default_zed_left_camera_frame, origin xyz=0 0.06 0 rpy=-1.5707963267948966 0 -1.5707963267948966
- added joint default_zed_left_camera_optical_joint: type fixed, parent default_zed_left_camera_frame, child default_zed_left_camera_optical_frame, origin xyz=0 0 -0.01 rpy=3.141592653589793 0 0
- added joint default_zed_right_camera_joint: type fixed, parent default_zed_camera_center, child default_zed_right_camera_frame, origin xyz=0 -0.06 0 rpy=-1.5707963267948966 0 -1.5707963267948966
- added joint default_zed_right_camera_optical_joint: type fixed, parent default_zed_right_camera_frame, child default_zed_right_camera_optical_frame, origin xyz=0 0 -0.01 rpy=3.141592653589793 0 0

File: src/edna_description/urdf/robots/edna.urdf.xacro (robot description, xacro)
@@ -3,4 +3,6 @@
   <!-- Args -->
   <xacro:arg name="hw_interface_plugin" default="swerve_hardware/IsaacDriveHardware"/>
+  <xacro:arg name="namespace" default="default"/>
+  <xacro:property name="ns" value="$(arg namespace)" />
   <!-- Include Files -->
   <xacro:include filename="$(find edna_description)/urdf/control/drive.xacro" />
@@ -20,24 +22,24 @@
   <!-- Chassis -->
   <link name="base_link"></link>
-  <xacro:square_chassis prefix="swerve" parent="base_link">
+  <xacro:square_chassis prefix="${ns}_swerve" parent="base_link">
     <origin xyz="0 0 0" rpy="0 0 0" />
   </xacro:square_chassis>
   <!-- Drive Train -->
-  <xacro:swerve_axle prefix="front_left" parent="swerve_chassis_link">
+  <xacro:swerve_axle prefix="${ns}_front_left" parent="${ns}_swerve_chassis_link">
     <origin xyz="${axle_pos} ${axle_pos} ${axle_pos_z}" rpy="0 0 0" />
   </xacro:swerve_axle>
-  <xacro:swerve_axle prefix="front_right" parent="swerve_chassis_link">
+  <xacro:swerve_axle prefix="${ns}_front_right" parent="${ns}_swerve_chassis_link">
     <origin xyz="${axle_pos} -${axle_pos} ${axle_pos_z}" rpy="0 0 0" />
   </xacro:swerve_axle>
-  <xacro:swerve_axle prefix="rear_left" parent="swerve_chassis_link">
+  <xacro:swerve_axle prefix="${ns}_rear_left" parent="${ns}_swerve_chassis_link">
     <origin xyz="-${axle_pos} ${axle_pos} ${axle_pos_z} " rpy="0 0 0" />
   </xacro:swerve_axle>
-  <xacro:swerve_axle prefix="rear_right" parent="swerve_chassis_link">
+  <xacro:swerve_axle prefix="${ns}_rear_right" parent="${ns}_swerve_chassis_link">
     <origin xyz="-${axle_pos} -${axle_pos} ${axle_pos_z}" rpy="0 0 0" />
   </xacro:swerve_axle>
   <!-- Sensors -->
-  <xacro:zed_camera prefix="zed" model="zed2i" parent="swerve_chassis_link">
+  <xacro:zed_camera prefix="${ns}_zed" model="zed2i" parent="${ns}_swerve_chassis_link">
     <origin xyz="${cam_pos}" rpy="0 0 0" />
   </xacro:zed_camera>
-  <xacro:swerve_drive_control plugin="$(arg hw_interface_plugin)" />
+  <xacro:swerve_drive_control plugin="$(arg hw_interface_plugin)" ns="${ns}"/>
 </robot>
