Commit message: Add namespaces to URDF and import script

File: src/edna_description/urdf/edna.urdf (robot description, URDF)
Before this commit: robot edna, 17 links, 16 joints
Links:
- removed link default_front_left_axle_link
- removed link default_front_left_wheel_link
- removed link default_front_right_axle_link
- removed link default_front_right_wheel_link
- removed link default_rear_left_axle_link
- removed link default_rear_left_wheel_link
- removed link default_rear_right_axle_link
- removed link default_rear_right_wheel_link
- removed link default_swerve_chassis_link
- removed link default_zed_base_link
- removed link default_zed_camera_center
- removed link default_zed_left_camera_frame
- removed link default_zed_left_camera_optical_frame
- removed link default_zed_right_camera_frame
- removed link default_zed_right_camera_optical_frame
- removed link lidar_link
- added link liam_front_left_axle_link, mass 0.23739; visual mesh filename=package://edna_description/meshes/SwerveAxle.stl scale=0.001 0.001 0.001
- added link liam_front_left_wheel_link, mass 0.23133211; collision cylinder length=0.0381 radius=0.0508; visual mesh filename=package://edna_description/meshes/SwerveWheel.stl scale=0.001 0.001 0.001
- added link liam_front_right_axle_link, mass 0.23739; visual mesh filename=package://edna_description/meshes/SwerveAxle.stl scale=0.001 0.001 0.001
- added link liam_front_right_wheel_link, mass 0.23133211; collision cylinder length=0.0381 radius=0.0508; visual mesh filename=package://edna_description/meshes/SwerveWheel.stl scale=0.001 0.001 0.001
- added link liam_lidar_link; collision cylinder length=0.025 radius=0.035; visual cylinder length=0.025 radius=0.035
- added link liam_rear_left_axle_link, mass 0.23739; visual mesh filename=package://edna_description/meshes/SwerveAxle.stl scale=0.001 0.001 0.001
- added link liam_rear_left_wheel_link, mass 0.23133211; collision cylinder length=0.0381 radius=0.0508; visual mesh filename=package://edna_description/meshes/SwerveWheel.stl scale=0.001 0.001 0.001
- added link liam_rear_right_axle_link, mass 0.23739; visual mesh filename=package://edna_description/meshes/SwerveAxle.stl scale=0.001 0.001 0.001
- added link liam_rear_right_wheel_link, mass 0.23133211; collision cylinder length=0.0381 radius=0.0508; visual mesh filename=package://edna_description/meshes/SwerveWheel.stl scale=0.001 0.001 0.001
- added link liam_swerve_chassis_link, mass 19.0508795; collision box size=0.7366 0.7366 0.05588; visual mesh filename=package://edna_description/meshes/SwerveChassis.stl scale=0.001 0.001 0.001
- added link liam_zed_base_link
- added link liam_zed_camera_center; collision mesh filename=package://edna_description/meshes/zed2i.stl; visual mesh filename=package://edna_description/meshes/zed2i.stl
- added link liam_zed_left_camera_frame
- added link liam_zed_left_camera_optical_frame
- added link liam_zed_right_camera_frame
- added link liam_zed_right_camera_optical_frame
Joints:
- removed joint default_front_left_axle_joint
- removed joint default_front_left_wheel_joint
- removed joint default_front_right_axle_joint
- removed joint default_front_right_wheel_joint
- removed joint default_rear_left_axle_joint
- removed joint default_rear_left_wheel_joint
- removed joint default_rear_right_axle_joint
- removed joint default_rear_right_wheel_joint
- removed joint default_swerve_chassis_joint
- removed joint default_zed_base_joint
- removed joint default_zed_camera_center_joint
- removed joint default_zed_left_camera_joint
- removed joint default_zed_left_camera_optical_joint
- removed joint default_zed_right_camera_joint
- removed joint default_zed_right_camera_optical_joint
- removed joint lidar_joint
- added joint liam_front_left_axle_joint: type continuous, parent liam_swerve_chassis_link, child liam_front_left_axle_link, origin xyz=0.301625 0.301625 0.06905599999999999 rpy=0 0 0, axis 0 0 -1
- added joint liam_front_left_wheel_joint: type continuous, parent liam_front_left_axle_link, child liam_front_left_wheel_link, origin xyz=0 0 -0.063 rpy=0 0 0, axis 0 1 0
- added joint liam_front_right_axle_joint: type continuous, parent liam_swerve_chassis_link, child liam_front_right_axle_link, origin xyz=0.301625 -0.301625 0.06905599999999999 rpy=0 0 0, axis 0 0 -1
- added joint liam_front_right_wheel_joint: type continuous, parent liam_front_right_axle_link, child liam_front_right_wheel_link, origin xyz=0 0 -0.063 rpy=0 0 0, axis 0 1 0
- added joint liam_lidar_joint: type fixed, parent liam_swerve_chassis_link, child liam_lidar_link, origin xyz=0 0 .035 rpy=0 0 0
- added joint liam_rear_left_axle_joint: type continuous, parent liam_swerve_chassis_link, child liam_rear_left_axle_link, origin xyz=-0.301625 0.301625 0.06905599999999999  rpy=0 0 0, axis 0 0 -1
- added joint liam_rear_left_wheel_joint: type continuous, parent liam_rear_left_axle_link, child liam_rear_left_wheel_link, origin xyz=0 0 -0.063 rpy=0 0 0, axis 0 1 0
- added joint liam_rear_right_axle_joint: type continuous, parent liam_swerve_chassis_link, child liam_rear_right_axle_link, origin xyz=-0.301625 -0.301625 0.06905599999999999 rpy=0 0 0, axis 0 0 -1
- added joint liam_rear_right_wheel_joint: type continuous, parent liam_rear_right_axle_link, child liam_rear_right_wheel_link, origin xyz=0 0 -0.063 rpy=0 0 0, axis 0 1 0
- added joint liam_swerve_chassis_joint: type fixed, parent base_link, child liam_swerve_chassis_link, origin xyz=0 0 0 rpy=0 0 0
- added joint liam_zed_base_joint: type fixed, parent liam_swerve_chassis_link, child liam_zed_base_link, origin xyz=0 0 0.3 rpy=0 0 0
- added joint liam_zed_camera_center_joint: type fixed, parent liam_zed_base_link, child liam_zed_camera_center, origin xyz=0 0 0.015 rpy=0 0.0 0
- added joint liam_zed_left_camera_joint: type fixed, parent liam_zed_camera_center, child liam_zed_left_camera_frame, origin xyz=0 0.06 0 rpy=-1.5707963267948966 0 -1.5707963267948966
- added joint liam_zed_left_camera_optical_joint: type fixed, parent liam_zed_left_camera_frame, child liam_zed_left_camera_optical_frame, origin xyz=0 0 -0.01 rpy=3.141592653589793 0 0
- added joint liam_zed_right_camera_joint: type fixed, parent liam_zed_camera_center, child liam_zed_right_camera_frame, origin xyz=0 -0.06 0 rpy=-1.5707963267948966 0 -1.5707963267948966
- added joint liam_zed_right_camera_optical_joint: type fixed, parent liam_zed_right_camera_frame, child liam_zed_right_camera_optical_frame, origin xyz=0 0 -0.01 rpy=3.141592653589793 0 0

File: src/edna_description/urdf/parts/lidar.xacro (robot description, xacro)
@@ -1,6 +1,6 @@
 <?xml version="1.0" ?>
 <robot xmlns:xacro="http://www.ros.org/wiki/xacro">
-  <xacro:macro name="lidar" params="radius length parent *origin">
-    <link name="lidar_link">
+  <xacro:macro name="lidar" params="radius length prefix parent *origin">
+    <link name="${prefix}_link">
       <visual>
         <origin xyz="0 0 0" rpy="0 0 0"/>
@@ -17,8 +17,8 @@
       </collision>
     </link>
-    <joint name="lidar_joint" type="fixed">
+    <joint name="${prefix}_joint" type="fixed">
       <xacro:insert_block name="origin" />
       <parent link="${parent}"/>
-      <child link="lidar_link"/>
+      <child link="${prefix}_link"/>
     </joint>
   </xacro:macro>

File: src/edna_description/urdf/robots/edna.urdf.xacro (robot description, xacro)
@@ -43,5 +43,5 @@
     <origin xyz="${cam_pos}" rpy="0 0 0" />
   </xacro:zed_camera>
-  <xacro:lidar parent="swerve_chassis_link" radius="0.035" length="0.025">
+  <xacro:lidar prefix="${ns}_lidar" parent="${ns}_swerve_chassis_link" radius="0.035" length="0.025">
     <origin xyz="0 0 .035" rpy="0 0 0" />
   </xacro:lidar>

Commit message: Add LiDAR to sim (#48)
- Create the Lidar in the description
- Add graph to import script
- Add namespaces to URDF and import script

File: src/edna_description/urdf/edna.urdf (robot description, URDF)
Before this commit: robot edna, 16 links, 15 joints
Links:
- removed link default_front_left_axle_link
- removed link default_front_left_wheel_link
- removed link default_front_right_axle_link
- removed link default_front_right_wheel_link
- removed link default_rear_left_axle_link
- removed link default_rear_left_wheel_link
- removed link default_rear_right_axle_link
- removed link default_rear_right_wheel_link
- removed link default_swerve_chassis_link
- removed link default_zed_base_link
- removed link default_zed_camera_center
- removed link default_zed_left_camera_frame
- removed link default_zed_left_camera_optical_frame
- removed link default_zed_right_camera_frame
- removed link default_zed_right_camera_optical_frame
- added link liam_front_left_axle_link, mass 0.23739; visual mesh filename=package://edna_description/meshes/SwerveAxle.stl scale=0.001 0.001 0.001
- added link liam_front_left_wheel_link, mass 0.23133211; collision cylinder length=0.0381 radius=0.0508; visual mesh filename=package://edna_description/meshes/SwerveWheel.stl scale=0.001 0.001 0.001
- added link liam_front_right_axle_link, mass 0.23739; visual mesh filename=package://edna_description/meshes/SwerveAxle.stl scale=0.001 0.001 0.001
- added link liam_front_right_wheel_link, mass 0.23133211; collision cylinder length=0.0381 radius=0.0508; visual mesh filename=package://edna_description/meshes/SwerveWheel.stl scale=0.001 0.001 0.001
- added link liam_lidar_link; collision cylinder length=0.025 radius=0.035; visual cylinder length=0.025 radius=0.035
- added link liam_rear_left_axle_link, mass 0.23739; visual mesh filename=package://edna_description/meshes/SwerveAxle.stl scale=0.001 0.001 0.001
- added link liam_rear_left_wheel_link, mass 0.23133211; collision cylinder length=0.0381 radius=0.0508; visual mesh filename=package://edna_description/meshes/SwerveWheel.stl scale=0.001 0.001 0.001
- added link liam_rear_right_axle_link, mass 0.23739; visual mesh filename=package://edna_description/meshes/SwerveAxle.stl scale=0.001 0.001 0.001
- added link liam_rear_right_wheel_link, mass 0.23133211; collision cylinder length=0.0381 radius=0.0508; visual mesh filename=package://edna_description/meshes/SwerveWheel.stl scale=0.001 0.001 0.001
- added link liam_swerve_chassis_link, mass 19.0508795; collision box size=0.7366 0.7366 0.05588; visual mesh filename=package://edna_description/meshes/SwerveChassis.stl scale=0.001 0.001 0.001
- added link liam_zed_base_link
- added link liam_zed_camera_center; collision mesh filename=package://edna_description/meshes/zed2i.stl; visual mesh filename=package://edna_description/meshes/zed2i.stl
- added link liam_zed_left_camera_frame
- added link liam_zed_left_camera_optical_frame
- added link liam_zed_right_camera_frame
- added link liam_zed_right_camera_optical_frame
Joints:
- removed joint default_front_left_axle_joint
- removed joint default_front_left_wheel_joint
- removed joint default_front_right_axle_joint
- removed joint default_front_right_wheel_joint
- removed joint default_rear_left_axle_joint
- removed joint default_rear_left_wheel_joint
- removed joint default_rear_right_axle_joint
- removed joint default_rear_right_wheel_joint
- removed joint default_swerve_chassis_joint
- removed joint default_zed_base_joint
- removed joint default_zed_camera_center_joint
- removed joint default_zed_left_camera_joint
- removed joint default_zed_left_camera_optical_joint
- removed joint default_zed_right_camera_joint
- removed joint default_zed_right_camera_optical_joint
- added joint liam_front_left_axle_joint: type continuous, parent liam_swerve_chassis_link, child liam_front_left_axle_link, origin xyz=0.301625 0.301625 0.06905599999999999 rpy=0 0 0, axis 0 0 -1
- added joint liam_front_left_wheel_joint: type continuous, parent liam_front_left_axle_link, child liam_front_left_wheel_link, origin xyz=0 0 -0.063 rpy=0 0 0, axis 0 1 0
- added joint liam_front_right_axle_joint: type continuous, parent liam_swerve_chassis_link, child liam_front_right_axle_link, origin xyz=0.301625 -0.301625 0.06905599999999999 rpy=0 0 0, axis 0 0 -1
- added joint liam_front_right_wheel_joint: type continuous, parent liam_front_right_axle_link, child liam_front_right_wheel_link, origin xyz=0 0 -0.063 rpy=0 0 0, axis 0 1 0
- added joint liam_lidar_joint: type fixed, parent liam_swerve_chassis_link, child liam_lidar_link, origin xyz=0 0 .035 rpy=0 0 0
- added joint liam_rear_left_axle_joint: type continuous, parent liam_swerve_chassis_link, child liam_rear_left_axle_link, origin xyz=-0.301625 0.301625 0.06905599999999999  rpy=0 0 0, axis 0 0 -1
- added joint liam_rear_left_wheel_joint: type continuous, parent liam_rear_left_axle_link, child liam_rear_left_wheel_link, origin xyz=0 0 -0.063 rpy=0 0 0, axis 0 1 0
- added joint liam_rear_right_axle_joint: type continuous, parent liam_swerve_chassis_link, child liam_rear_right_axle_link, origin xyz=-0.301625 -0.301625 0.06905599999999999 rpy=0 0 0, axis 0 0 -1
- added joint liam_rear_right_wheel_joint: type continuous, parent liam_rear_right_axle_link, child liam_rear_right_wheel_link, origin xyz=0 0 -0.063 rpy=0 0 0, axis 0 1 0
- added joint liam_swerve_chassis_joint: type fixed, parent base_link, child liam_swerve_chassis_link, origin xyz=0 0 0 rpy=0 0 0
- added joint liam_zed_base_joint: type fixed, parent liam_swerve_chassis_link, child liam_zed_base_link, origin xyz=0 0 0.3 rpy=0 0 0
- added joint liam_zed_camera_center_joint: type fixed, parent liam_zed_base_link, child liam_zed_camera_center, origin xyz=0 0 0.015 rpy=0 0.0 0
- added joint liam_zed_left_camera_joint: type fixed, parent liam_zed_camera_center, child liam_zed_left_camera_frame, origin xyz=0 0.06 0 rpy=-1.5707963267948966 0 -1.5707963267948966
- added joint liam_zed_left_camera_optical_joint: type fixed, parent liam_zed_left_camera_frame, child liam_zed_left_camera_optical_frame, origin xyz=0 0 -0.01 rpy=3.141592653589793 0 0
- added joint liam_zed_right_camera_joint: type fixed, parent liam_zed_camera_center, child liam_zed_right_camera_frame, origin xyz=0 -0.06 0 rpy=-1.5707963267948966 0 -1.5707963267948966
- added joint liam_zed_right_camera_optical_joint: type fixed, parent liam_zed_right_camera_frame, child liam_zed_right_camera_optical_frame, origin xyz=0 0 -0.01 rpy=3.141592653589793 0 0

File: src/edna_description/urdf/robots/edna.urdf.xacro (robot description, xacro)
@@ -12,4 +12,5 @@
   <xacro:include filename="$(find edna_description)/urdf/parts/swerve_axle.xacro" />
   <xacro:include filename="$(find edna_description)/urdf/parts/zed_macro.urdf.xacro" />
+  <xacro:include filename="$(find edna_description)/urdf/parts/lidar.xacro" />
   <!-- Axle Position Variables -->
   <xacro:property name="axle_pos" value="${301.625 / 1000}" />
@@ -42,4 +43,7 @@
     <origin xyz="${cam_pos}" rpy="0 0 0" />
   </xacro:zed_camera>
+  <xacro:lidar prefix="${ns}_lidar" parent="${ns}_swerve_chassis_link" radius="0.035" length="0.025">
+    <origin xyz="0 0 .035" rpy="0 0 0" />
+  </xacro:lidar>
   <xacro:swerve_drive_control plugin="$(arg hw_interface_plugin)" ns="${ns}"/>
 </robot>

Commit message: tried to commit

File: src/edna_description/urdf/edna.urdf (robot description, URDF)
Before this commit: robot edna, 17 links, 16 joints
Links:
- removed link liam_front_left_axle_link
- removed link liam_front_left_wheel_link
- removed link liam_front_right_axle_link
- removed link liam_front_right_wheel_link
- removed link liam_lidar_link
- removed link liam_rear_left_axle_link
- removed link liam_rear_left_wheel_link
- removed link liam_rear_right_axle_link
- removed link liam_rear_right_wheel_link
- removed link liam_swerve_chassis_link
- removed link liam_zed_base_link
- removed link liam_zed_camera_center
- removed link liam_zed_left_camera_frame
- removed link liam_zed_left_camera_optical_frame
- removed link liam_zed_right_camera_frame
- removed link liam_zed_right_camera_optical_frame
- added link real_front_left_axle_link, mass 0.23739; visual mesh filename=package://edna_description/meshes/SwerveAxle.stl scale=0.001 0.001 0.001
- added link real_front_left_wheel_link, mass 0.23133211; collision cylinder length=0.0381 radius=0.0508; visual mesh filename=package://edna_description/meshes/SwerveWheel.stl scale=0.001 0.001 0.001
- added link real_front_right_axle_link, mass 0.23739; visual mesh filename=package://edna_description/meshes/SwerveAxle.stl scale=0.001 0.001 0.001
- added link real_front_right_wheel_link, mass 0.23133211; collision cylinder length=0.0381 radius=0.0508; visual mesh filename=package://edna_description/meshes/SwerveWheel.stl scale=0.001 0.001 0.001
- added link real_lidar_link; collision cylinder length=0.025 radius=0.035; visual cylinder length=0.025 radius=0.035
- added link real_rear_left_axle_link, mass 0.23739; visual mesh filename=package://edna_description/meshes/SwerveAxle.stl scale=0.001 0.001 0.001
- added link real_rear_left_wheel_link, mass 0.23133211; collision cylinder length=0.0381 radius=0.0508; visual mesh filename=package://edna_description/meshes/SwerveWheel.stl scale=0.001 0.001 0.001
- added link real_rear_right_axle_link, mass 0.23739; visual mesh filename=package://edna_description/meshes/SwerveAxle.stl scale=0.001 0.001 0.001
- added link real_rear_right_wheel_link, mass 0.23133211; collision cylinder length=0.0381 radius=0.0508; visual mesh filename=package://edna_description/meshes/SwerveWheel.stl scale=0.001 0.001 0.001
- added link real_swerve_chassis_link, mass 19.0508795; collision box size=0.7366 0.7366 0.05588; visual mesh filename=package://edna_description/meshes/SwerveChassis.stl scale=0.001 0.001 0.001
- added link real_zed_base_link
- added link real_zed_camera_center; collision mesh filename=package://edna_description/meshes/zed2i.stl; visual mesh filename=package://edna_description/meshes/zed2i.stl
- added link real_zed_left_camera_frame
- added link real_zed_left_camera_optical_frame
- added link real_zed_right_camera_frame
- added link real_zed_right_camera_optical_frame
Joints:
- removed joint liam_front_left_axle_joint
- removed joint liam_front_left_wheel_joint
- removed joint liam_front_right_axle_joint
- removed joint liam_front_right_wheel_joint
- removed joint liam_lidar_joint
- removed joint liam_rear_left_axle_joint
- removed joint liam_rear_left_wheel_joint
- removed joint liam_rear_right_axle_joint
- removed joint liam_rear_right_wheel_joint
- removed joint liam_swerve_chassis_joint
- removed joint liam_zed_base_joint
- removed joint liam_zed_camera_center_joint
- removed joint liam_zed_left_camera_joint
- removed joint liam_zed_left_camera_optical_joint
- removed joint liam_zed_right_camera_joint
- removed joint liam_zed_right_camera_optical_joint
- added joint real_front_left_axle_joint: type continuous, parent real_swerve_chassis_link, child real_front_left_axle_link, origin xyz=0.301625 0.301625 0.06905599999999999 rpy=0 0 0, axis 0 0 -1
- added joint real_front_left_wheel_joint: type continuous, parent real_front_left_axle_link, child real_front_left_wheel_link, origin xyz=0 0 -0.063 rpy=0 0 0, axis 0 1 0
- added joint real_front_right_axle_joint: type continuous, parent real_swerve_chassis_link, child real_front_right_axle_link, origin xyz=0.301625 -0.301625 0.06905599999999999 rpy=0 0 0, axis 0 0 -1
- added joint real_front_right_wheel_joint: type continuous, parent real_front_right_axle_link, child real_front_right_wheel_link, origin xyz=0 0 -0.063 rpy=0 0 0, axis 0 1 0
- added joint real_lidar_joint: type fixed, parent real_swerve_chassis_link, child real_lidar_link, origin xyz=0 0 .035 rpy=0 0 0
- added joint real_rear_left_axle_joint: type continuous, parent real_swerve_chassis_link, child real_rear_left_axle_link, origin xyz=-0.301625 0.301625 0.06905599999999999  rpy=0 0 0, axis 0 0 -1
- added joint real_rear_left_wheel_joint: type continuous, parent real_rear_left_axle_link, child real_rear_left_wheel_link, origin xyz=0 0 -0.063 rpy=0 0 0, axis 0 1 0
- added joint real_rear_right_axle_joint: type continuous, parent real_swerve_chassis_link, child real_rear_right_axle_link, origin xyz=-0.301625 -0.301625 0.06905599999999999 rpy=0 0 0, axis 0 0 -1
- added joint real_rear_right_wheel_joint: type continuous, parent real_rear_right_axle_link, child real_rear_right_wheel_link, origin xyz=0 0 -0.063 rpy=0 0 0, axis 0 1 0
- added joint real_swerve_chassis_joint: type fixed, parent base_link, child real_swerve_chassis_link, origin xyz=0 0 0 rpy=0 0 0
- added joint real_zed_base_joint: type fixed, parent real_swerve_chassis_link, child real_zed_base_link, origin xyz=0 0 0.3 rpy=0 0 0
- added joint real_zed_camera_center_joint: type fixed, parent real_zed_base_link, child real_zed_camera_center, origin xyz=0 0 0.015 rpy=0 0.0 0
- added joint real_zed_left_camera_joint: type fixed, parent real_zed_camera_center, child real_zed_left_camera_frame, origin xyz=0 0.06 0 rpy=-1.5707963267948966 0 -1.5707963267948966
- added joint real_zed_left_camera_optical_joint: type fixed, parent real_zed_left_camera_frame, child real_zed_left_camera_optical_frame, origin xyz=0 0 -0.01 rpy=3.141592653589793 0 0
- added joint real_zed_right_camera_joint: type fixed, parent real_zed_camera_center, child real_zed_right_camera_frame, origin xyz=0 -0.06 0 rpy=-1.5707963267948966 0 -1.5707963267948966
- added joint real_zed_right_camera_optical_joint: type fixed, parent real_zed_right_camera_frame, child real_zed_right_camera_optical_frame, origin xyz=0 0 -0.01 rpy=3.141592653589793 0 0
