Commit message: Add Add ns to drive component

File: src/edna_description/urdf/control/drive.xacro (robot description, xacro)
@@ -1,5 +1,5 @@
 <?xml version="1.0"?>
 <robot name="robot" xmlns:xacro="http://www.ros.org/wiki/xacro" >
-  <xacro:macro name="swerve_drive_control" params="plugin">
+  <xacro:macro name="swerve_drive_control" params="plugin ns">
     <ros2_control name="swerve_drive" type="system">
       <hardware>
@@ -8,5 +8,5 @@
         <param name="example_param_hw_stop_duration_sec">3.0</param>
       </hardware>
-      <joint name="front_right_wheel_joint">
+      <joint name="${ns}_front_right_wheel_joint">
         <command_interface name="velocity">
           <param name="min">-1</param>
@@ -16,5 +16,5 @@
         <state_interface name="velocity"/>
       </joint>
-      <joint name="rear_left_wheel_joint">
+      <joint name="${ns}_rear_left_wheel_joint">
         <command_interface name="velocity">
           <param name="min">-1</param>
@@ -24,5 +24,5 @@
         <state_interface name="velocity"/>
       </joint>
-      <joint name="front_left_wheel_joint">
+      <joint name="${ns}_front_left_wheel_joint">
         <command_interface name="velocity">
           <param name="min">-1</param>
@@ -32,5 +32,5 @@
         <state_interface name="velocity"/>
       </joint>
-      <joint name="rear_right_wheel_joint">
+      <joint name="${ns}_rear_right_wheel_joint">
         <command_interface name="velocity">
           <param name="min">-1</param>
@@ -40,5 +40,5 @@
         <state_interface name="velocity"/>
       </joint>
-      <joint name="front_right_axle_joint">
+      <joint name="${ns}_front_right_axle_joint">
         <command_interface name="position">
           <param name="min">-1</param>
@@ -48,5 +48,5 @@
         <state_interface name="velocity"/>
       </joint>
-      <joint name="rear_left_axle_joint">
+      <joint name="${ns}_rear_left_axle_joint">
         <command_interface name="position">
           <param name="min">-1</param>
@@ -56,5 +56,5 @@
         <state_interface name="velocity"/>
       </joint>
-      <joint name="front_left_axle_joint">
+      <joint name="${ns}_front_left_axle_joint">
         <command_interface name="position">
           <param name="min">-1</param>
@@ -64,5 +64,5 @@
         <state_interface name="velocity"/>
       </joint>
-      <joint name="rear_right_axle_joint">
+      <joint name="${ns}_rear_right_axle_joint">
         <command_interface name="position">
           <param name="min">-1</param>

File: src/edna_description/urdf/robots/edna.urdf.xacro (robot description, xacro)
@@ -42,4 +42,4 @@
     <origin xyz="${cam_pos}" rpy="0 0 0" />
   </xacro:zed_camera>
-  <xacro:swerve_drive_control plugin="$(arg hw_interface_plugin)" />
+  <xacro:swerve_drive_control plugin="$(arg hw_interface_plugin)" ns="${ns}"/>
 </robot>

Commit message: back leg and elevator leg URDF

File: src/edna_description/urdf/control/drive.xacro (robot description, xacro)
@@ -72,4 +72,12 @@
         <state_interface name="velocity"/>
       </joint>
+      <joint name="${ns}_arm_roller_bar_joint">
+        <command_interface name="position">
+          <param name="min">-1</param>
+          <param name="max">1</param>
+        </command_interface>
+        <state_interface name="position"/>
+        <state_interface name="velocity"/>
+      </joint>
     </ros2_control>
   </xacro:macro>

File: src/edna_description/urdf/parts/back_leg.xacro (robot description, xacro)
@@ -1,14 +1,14 @@
 <?xml version = "1.0"?>
 <robot xmlns:xacro = "http://www.ros.org/wiki/xacro">
-    <xacro:property name="back_leg_length" value="0.052" />
-    <xacro:property name="back_leg_width" value="0.635" />
-    <xacro:property name="back_leg_height" value="0.527" />
+    <xacro:property name="back_leg_length" value="0.0508" />
+    <xacro:property name="back_leg_width" value="0.457" />
+    <xacro:property name="back_leg_height" value="0.812" />
     <xacro:macro name = "back_leg" params = "prefix parent *origin">
-        <link name = "${prefix}_link">
+        <link name = "${prefix}_back_leg_link">
             <xacro:inertial_box mass = "1" x = "${back_leg_length}" y = "${back_leg_width}" z = "${back_leg_height}">
                 <origin xyz = "0 0 ${back_leg_height/2}" rpy = "0 0 0"/>
             </xacro:inertial_box>
             <visual>
-                <origin xyz = "${0.7366/2} 0 ${back_leg_height/2 + 0.2}" rpy = "0 0 0"/>
+                <origin xyz = "0 0 0" rpy = "0 0 0"/>
                 <geometry>
                     <mesh filename="package://edna_description/meshes/back_legs.stl" scale="0.001 0.001 0.001"/>
@@ -17,13 +17,14 @@
             </visual>
             <collision>
-                <origin xyz = "0 0 ${back_leg_height/2}" rpy = "0 0 0"/>
+                <origin xyz = "0 0 0" rpy = "0 0 0"/>
                 <geometry>
                     <box size = "${back_leg_length} ${back_leg_width} ${back_leg_height}"/>
                 </geometry>
+                <material name = "ghost"/>
             </collision>
         </link>
-        <joint name = "${prefix}_box_joint" type = "fixed">
+        <joint name = "${prefix}_back_leg_joint" type = "fixed">
             <parent link = "${parent}"/>
-            <child link = "${prefix}_link"/>
+            <child link = "${prefix}_back_leg_link"/>
             <xacro:insert_block name = "origin"/>
         </joint>

File: src/edna_description/urdf/parts/elevator_leg.xacro (robot description, xacro)
@@ -4,11 +4,14 @@
     <xacro:property name="elevator_leg_width" value="0.330" />
     <xacro:property name="elevator_leg_height" value="0.527" />
-    <xacro:macro name = "elevator_leg" params = "prefix parent *origin">
-        <link name = "${prefix}_link">
+    <xacro:property name="roller_bar_length" value="0.0508" />
+    <xacro:property name="roller_bar_width" value="0.711" />
+    <xacro:property name="roller_bar_height" value="0.527" />
+    <xacro:macro name = "elevator_leg" params = "prefix parent *origin *origin2">
+        <link name = "${prefix}_elevator_leg_link">
             <xacro:inertial_box mass = "1" x = "${elevator_leg_length}" y = "${elevator_leg_width}" z = "${elevator_leg_height}">
                 <origin xyz = "0 0 ${elevator_leg_height/2}" rpy = "0 0 0"/>
             </xacro:inertial_box>
             <visual>
-                <origin xyz = "0 0 ${elevator_leg_height/2 + 0.082}" rpy = "0 0 0"/>
+                <origin xyz = "0 0 0" rpy = "0 0 0"/>
                 <geometry>
                     <mesh filename="package://edna_description/meshes/elevator_legs.stl" scale="0.001 0.001 0.001"/>
@@ -17,5 +20,5 @@
             </visual>
             <collision>
-                <origin xyz = "0 0 ${elevator_leg_height/2}" rpy = "0 0 0"/>
+                <origin xyz = "0 0 0" rpy = "0 0 0"/>
                 <geometry>
                     <box size = "${elevator_leg_length} ${elevator_leg_width} ${elevator_leg_height}"/>
@@ -23,8 +26,33 @@
             </collision>
         </link>
-        <joint name = "${prefix}_box_joint" type = "fixed">
+        <joint name = "${prefix}_elevator_leg_joint" type = "fixed">
             <parent link = "${parent}"/>
-            <child link = "${prefix}_link"/>
+            <child link = "${prefix}_elevator_leg_link"/>
             <xacro:insert_block name = "origin"/>
+        </joint>
+        <link name = "${prefix}_roller_bar_link">
+            <xacro:inertial_box mass = "1" x = "${roller_bar_length}" y = "${roller_bar_width}" z = "${roller_bar_height}">
+                <origin xyz = "0 0 ${roller_bar_height/2}" rpy = "${pi/2} 0 0"/>
+            </xacro:inertial_box>
+            <visual>
+                <origin xyz = "0 0 0" rpy = "0 0 0"/>
+                <geometry>
+                    <mesh filename="package://edna_description/meshes/Roller_Bar.stl" scale="0.001 0.001 0.001"/>
+                </geometry>
+                <material name = "blue"/>
+            </visual>
+            <collision>
+                <origin xyz = "0 0 0" rpy = "0 0 0"/>
+                <geometry>
+                    <box size = "${roller_bar_length} ${roller_bar_width} ${roller_bar_height}"/>
+                </geometry>
+            </collision>
+        </link>
+        <joint name = "${prefix}_roller_bar_joint" type = "prismatic">
+            <parent link = "${prefix}_elevator_leg_link"/>
+            <child link = "${prefix}_roller_bar_link"/>
+            <axis xyz = "0 1 0"/>
+            <limit effort = "100.0" lower = "0" upper = "0.06985" velocity = "0.1"/>
+            <xacro:insert_block name = "origin2"/>
         </joint>
     </xacro:macro>

File: src/edna_description/urdf/robots/edna.urdf.xacro (robot description, xacro)
@@ -46,12 +46,10 @@
     <origin xyz="${cam_pos}" rpy="0 0 0" />
   </xacro:zed_camera>
-  <xacro:roller_bar prefix="roller_bar" parent="swerve_chassis_link">
-    <origin xyz="0 0 0" rpy="0 0 0" />
-  </xacro:roller_bar>
-  <xacro:elevator_leg prefix="elevator_leg" parent="swerve_chassis_link">
-    <origin xyz="0 0 0" rpy="0 0 0" />
+  <xacro:elevator_leg prefix="${ns}_arm" parent="${ns}_swerve_chassis_link">
+    <origin xyz = "-0.1905 0 ${0.527/2 + 0.03}" rpy = "0 0 0"/>
+    <origin xyz = "0 0 ${0.527/5}" rpy = "${pi/2} 0 0"/>
   </xacro:elevator_leg>
-  <xacro:back_leg prefix="back_leg" parent="swerve_chassis_link">
-    <origin xyz="0 0 0" rpy="0 0 0" />
+  <xacro:back_leg prefix="${ns}_arm" parent="${ns}_swerve_chassis_link">
+    <origin xyz = "${0.7366/2 - 0.0508/2} 0 ${back_leg_height/2 + 0.05588}" rpy = "0 0 0" />
   </xacro:back_leg>
   <xacro:lidar prefix="${ns}_lidar" parent="${ns}_swerve_chassis_link" radius="0.035" length="0.025">

File: src/edna_description/urdf/util/materials.xacro (robot description, xacro)
@@ -9,4 +9,7 @@
   <material name="green">
     <color rgba="0.0 0.8 0.0 1.0" />
+  </material>
+  <material name="ghost">
+    <color rgba="0.0 0.8 0.0 0.5" />
   </material>
   <material name="grey">

Commit message: robot arm/elevator URDF

File: src/edna_description/urdf/control/drive.xacro (robot description, xacro)
@@ -80,4 +80,52 @@
         <state_interface name="velocity"/>
       </joint>
+      <joint name = "${ns}_elevator_left_elevator_outer_1_joint" type = "revolute">
+          <command_interface name="position">
+            <param name="min">-1</param>
+            <param name="max">1</param>
+          </command_interface>
+          <state_interface name="position"/>
+          <state_interface name="velocity"/>
+      </joint>
+      <joint name = "${ns}_elevator_left_elevator_center_joint" type = "prismatic">
+          <command_interface name="position">
+            <param name="min">-1</param>
+            <param name="max">1</param>
+          </command_interface>
+          <state_interface name="position"/>
+          <state_interface name="velocity"/>
+      </joint>
+      <joint name = "${ns}_elevator_left_elevator_outer_2_joint" type = "prismatic">
+          <command_interface name="position">
+            <param name="min">-1</param>
+            <param name="max">1</param>
+          </command_interface>
+          <state_interface name="position"/>
+          <state_interface name="velocity"/>
+      </joint>
+      <joint name = "${ns}_elevator_right_elevator_outer_1_joint" type = "revolute">
+          <command_interface name="position">
+            <param name="min">-1</param>
+            <param name="max">1</param>
+          </command_interface>
+          <state_interface name="position"/>
+          <state_interface name="velocity"/>
+      </joint>
+      <joint name = "${ns}_elevator_right_elevator_center_joint" type = "prismatic">
+          <command_interface name="position">
+            <param name="min">-1</param>
+            <param name="max">1</param>
+          </command_interface>
+          <state_interface name="position"/>
+          <state_interface name="velocity"/>
+      </joint>
+      <joint name = "${ns}_elevator_right_elevator_outer_2_joint" type = "prismatic">
+          <command_interface name="position">
+            <param name="min">-1</param>
+            <param name="max">1</param>
+          </command_interface>
+          <state_interface name="position"/>
+          <state_interface name="velocity"/>
+      </joint>
     </ros2_control>
   </xacro:macro>

File: src/edna_description/urdf/parts/back_leg.xacro (robot description, xacro)
@@ -14,5 +14,5 @@
                     <mesh filename="package://edna_description/meshes/back_legs.stl" scale="0.001 0.001 0.001"/>
                 </geometry>
-                <material name = "blue"/>
+                <material name = "red"/>
             </visual>
             <collision>
@@ -21,5 +21,4 @@
                     <box size = "${back_leg_length} ${back_leg_width} ${back_leg_height}"/>
                 </geometry>
-                <material name = "ghost"/>
             </collision>
         </link>

File: src/edna_description/urdf/parts/elevator_leg.xacro (robot description, xacro)
@@ -17,5 +17,5 @@
                     <mesh filename="package://edna_description/meshes/elevator_legs.stl" scale="0.001 0.001 0.001"/>
                 </geometry>
-                <material name = "blue"/>
+                <material name = "red"/>
             </visual>
             <collision>
@@ -40,5 +40,5 @@
                     <mesh filename="package://edna_description/meshes/Roller_Bar.stl" scale="0.001 0.001 0.001"/>
                 </geometry>
-                <material name = "blue"/>
+                <material name = "red"/>
             </visual>
             <collision>
@@ -53,5 +53,5 @@
             <child link = "${prefix}_roller_bar_link"/>
             <axis xyz = "0 1 0"/>
-            <limit effort = "100.0" lower = "0" upper = "0.06985" velocity = "0.1"/>
+            <limit effort = "100.0" lower = "0" upper = "0.06985" velocity = "0.5"/>
             <xacro:insert_block name = "origin2"/>
         </joint>

File: src/edna_description/urdf/robots/edna.urdf.xacro (robot description, xacro)
@@ -12,8 +12,8 @@
   <xacro:include filename="$(find edna_description)/urdf/parts/swerve_axle.xacro" />
   <xacro:include filename="$(find edna_description)/urdf/parts/zed_macro.urdf.xacro" />
-  <xacro:include filename="$(find edna_description)/urdf/parts/roller_bar.xacro" />
   <xacro:include filename="$(find edna_description)/urdf/parts/elevator_leg.xacro" />
   <xacro:include filename="$(find edna_description)/urdf/parts/back_leg.xacro" />
   <xacro:include filename="$(find edna_description)/urdf/parts/lidar.xacro" />
+  <xacro:include filename="$(find edna_description)/urdf/parts/elevator.xacro" />
   <!-- Axle Position Variables -->
   <xacro:property name="axle_pos" value="${301.625 / 1000}" />
@@ -47,10 +47,18 @@
   </xacro:zed_camera>
   <xacro:elevator_leg prefix="${ns}_arm" parent="${ns}_swerve_chassis_link">
-    <origin xyz = "-0.1905 0 ${0.527/2 + 0.03}" rpy = "0 0 0"/>
-    <origin xyz = "0 0 ${0.527/5}" rpy = "${pi/2} 0 0"/>
+    <origin xyz = "-0.1905 0 ${0.527/2 + 0.03}" rpy = "0 0 ${pi}"/>
+    <origin xyz = "0 0 ${0.527/5 + 0.01}" rpy = "${pi/2} 0 0"/>
   </xacro:elevator_leg>
   <xacro:back_leg prefix="${ns}_arm" parent="${ns}_swerve_chassis_link">
-    <origin xyz = "${0.7366/2 - 0.0508/2} 0 ${back_leg_height/2 + 0.05588}" rpy = "0 0 0" />
+    <origin xyz = "${0.7366/2 - 0.0508/2} 0 ${back_leg_height/2 + 0.05588}" rpy = "0 0 ${pi}" />
   </xacro:back_leg>
+  <!--Right Elevator-->
+  <xacro:elevator prefix="${ns}_elevator_right" parent="${ns}_arm_back_leg_link" ns="${ns}">
+    <origin xyz = "0.00253 -0.152 0.3738731" rpy = "${pi} ${(0.0174533*16.3)} 0" />
+  </xacro:elevator>
+  <!--Left Elevator-->
+  <xacro:elevator prefix="${ns}_elevator_left" parent="${ns}_arm_back_leg_link" ns="${ns}">
+    <origin xyz = "0.00253 0.28 0.3738731" rpy = "${pi} ${(0.0174533*16.3)} 0" />
+  </xacro:elevator>
   <xacro:lidar prefix="${ns}_lidar" parent="${ns}_swerve_chassis_link" radius="0.035" length="0.025">
     <origin xyz="0 0 .035" rpy="0 0 0" />

Commit message: added urdf stuff

File: src/edna_description/urdf/control/drive.xacro (robot description, xacro)
@@ -72,4 +72,60 @@
         <state_interface name="velocity"/>
       </joint>
+      <joint name="${ns}_arm_roller_bar_joint">
+        <command_interface name="position">
+          <param name="min">-1</param>
+          <param name="max">1</param>
+        </command_interface>
+        <state_interface name="position"/>
+        <state_interface name="velocity"/>
+      </joint>
+      <joint name = "${ns}_elevator_left_elevator_outer_1_joint" type = "revolute">
+          <command_interface name="position">
+            <param name="min">-1</param>
+            <param name="max">1</param>
+          </command_interface>
+          <state_interface name="position"/>
+          <state_interface name="velocity"/>
+      </joint>
+      <joint name = "${ns}_elevator_left_elevator_center_joint" type = "prismatic">
+          <command_interface name="position">
+            <param name="min">-1</param>
+            <param name="max">1</param>
+          </command_interface>
+          <state_interface name="position"/>
+          <state_interface name="velocity"/>
+      </joint>
+      <joint name = "${ns}_elevator_left_elevator_outer_2_joint" type = "prismatic">
+          <command_interface name="position">
+            <param name="min">-1</param>
+            <param name="max">1</param>
+          </command_interface>
+          <state_interface name="position"/>
+          <state_interface name="velocity"/>
+      </joint>
+      <joint name = "${ns}_elevator_right_elevator_outer_1_joint" type = "revolute">
+          <command_interface name="position">
+            <param name="min">-1</param>
+            <param name="max">1</param>
+          </command_interface>
+          <state_interface name="position"/>
+          <state_interface name="velocity"/>
+      </joint>
+      <joint name = "${ns}_elevator_right_elevator_center_joint" type = "prismatic">
+          <command_interface name="position">
+            <param name="min">-1</param>
+            <param name="max">1</param>
+          </command_interface>
+          <state_interface name="position"/>
+          <state_interface name="velocity"/>
+      </joint>
+      <joint name = "${ns}_elevator_right_elevator_outer_2_joint" type = "prismatic">
+          <command_interface name="position">
+            <param name="min">-1</param>
+            <param name="max">1</param>
+          </command_interface>
+          <state_interface name="position"/>
+          <state_interface name="velocity"/>
+      </joint>
     </ros2_control>
   </xacro:macro>

File: src/edna_description/urdf/robots/edna.urdf.xacro (robot description, xacro)
@@ -12,5 +12,8 @@
   <xacro:include filename="$(find edna_description)/urdf/parts/swerve_axle.xacro" />
   <xacro:include filename="$(find edna_description)/urdf/parts/zed_macro.urdf.xacro" />
+  <xacro:include filename="$(find edna_description)/urdf/parts/elevator_leg.xacro" />
+  <xacro:include filename="$(find edna_description)/urdf/parts/back_leg.xacro" />
   <xacro:include filename="$(find edna_description)/urdf/parts/lidar.xacro" />
+  <xacro:include filename="$(find edna_description)/urdf/parts/elevator.xacro" />
   <!-- Axle Position Variables -->
   <xacro:property name="axle_pos" value="${301.625 / 1000}" />
@@ -43,4 +46,19 @@
     <origin xyz="${cam_pos}" rpy="0 0 0" />
   </xacro:zed_camera>
+  <xacro:property name="elevator_leg_z" value="0.527"/>
+  <xacro:elevator_leg prefix="${ns}_arm" parent="${ns}_swerve_chassis_link">
+    <origin xyz = "0.1905 0 ${elevator_leg_z/2 + 0.03}" rpy = "0 0 0"/>
+  </xacro:elevator_leg>
+  <xacro:back_leg prefix="${ns}_arm" parent="${ns}_swerve_chassis_link">
+    <origin xyz = "-${chassis_length/2 - back_leg_length/2} 0 ${back_leg_height/2 + chassis_height}" rpy = "0 0 0" />
+  </xacro:back_leg>
+  <!--Right Elevator-->
+  <xacro:elevator prefix="${ns}_elevator_right" parent="${ns}_arm_back_leg_link" ns="${ns}" suffix="right">
+    <origin xyz = "0 ${-back_leg_width/2 - 0.04} ${back_leg_height/2 - 0.02}" rpy = "0 0 0" />
+  </xacro:elevator>
+  <!--Left Elevator-->
+  <xacro:elevator prefix="${ns}_elevator_left" parent="${ns}_arm_back_leg_link" ns="${ns}" suffix="left">
+    <origin xyz = "0 ${back_leg_width/2 + 0.04} ${back_leg_height/2 - 0.02}" rpy = "0 0 0" />
+  </xacro:elevator>
   <xacro:lidar prefix="${ns}_lidar" parent="${ns}_swerve_chassis_link" radius="0.035" length="0.025">
     <origin xyz="0 0 .035" rpy="0 0 0" />
