Commit message: Using frame_prefix

File: src/edna_description/urdf/control/drive.xacro (robot description, xacro)
@@ -1,5 +1,5 @@
 <?xml version="1.0"?>
 <robot name="robot" xmlns:xacro="http://www.ros.org/wiki/xacro" >
-  <xacro:macro name="swerve_drive_control" params="plugin ns">
+  <xacro:macro name="swerve_drive_control" params="plugin">
     <ros2_control name="swerve_drive" type="system">
       <hardware>
@@ -8,5 +8,5 @@
         <param name="example_param_hw_stop_duration_sec">3.0</param>
       </hardware>
-      <joint name="${ns}_front_right_wheel_joint">
+      <joint name="front_right_wheel_joint">
         <command_interface name="velocity">
           <param name="min">-1</param>
@@ -16,5 +16,5 @@
         <state_interface name="velocity"/>
       </joint>
-      <joint name="${ns}_rear_left_wheel_joint">
+      <joint name="rear_left_wheel_joint">
         <command_interface name="velocity">
           <param name="min">-1</param>
@@ -24,5 +24,5 @@
         <state_interface name="velocity"/>
       </joint>
-      <joint name="${ns}_front_left_wheel_joint">
+      <joint name="front_left_wheel_joint">
         <command_interface name="velocity">
           <param name="min">-1</param>
@@ -32,5 +32,5 @@
         <state_interface name="velocity"/>
       </joint>
-      <joint name="${ns}_rear_right_wheel_joint">
+      <joint name="rear_right_wheel_joint">
         <command_interface name="velocity">
           <param name="min">-1</param>
@@ -40,5 +40,5 @@
         <state_interface name="velocity"/>
       </joint>
-      <joint name="${ns}_front_right_axle_joint">
+      <joint name="front_right_axle_joint">
         <command_interface name="position">
           <param name="min">-1</param>
@@ -48,5 +48,5 @@
         <state_interface name="velocity"/>
       </joint>
-      <joint name="${ns}_rear_left_axle_joint">
+      <joint name="rear_left_axle_joint">
         <command_interface name="position">
           <param name="min">-1</param>
@@ -56,5 +56,5 @@
         <state_interface name="velocity"/>
       </joint>
-      <joint name="${ns}_front_left_axle_joint">
+      <joint name="front_left_axle_joint">
         <command_interface name="position">
           <param name="min">-1</param>
@@ -64,5 +64,5 @@
         <state_interface name="velocity"/>
       </joint>
-      <joint name="${ns}_rear_right_axle_joint">
+      <joint name="rear_right_axle_joint">
         <command_interface name="position">
           <param name="min">-1</param>

File: src/edna_description/urdf/robots/edna.urdf.xacro (robot description, xacro)
@@ -3,6 +3,4 @@
   <!-- Args -->
   <xacro:arg name="hw_interface_plugin" default="swerve_hardware/IsaacDriveHardware"/>
-  <xacro:arg name="namespace" default="default"/>
-  <xacro:property name="ns" value="$(arg namespace)" />
   <!-- Include Files -->
   <xacro:include filename="$(find edna_description)/urdf/control/drive.xacro" />
@@ -23,27 +21,27 @@
   <!-- Chassis -->
   <link name="base_link"></link>
-  <xacro:square_chassis prefix="${ns}_swerve" parent="base_link">
+  <xacro:square_chassis prefix="swerve" parent="base_link">
     <origin xyz="0 0 0" rpy="0 0 0" />
   </xacro:square_chassis>
   <!-- Drive Train -->
-  <xacro:swerve_axle prefix="${ns}_front_left" parent="${ns}_swerve_chassis_link">
+  <xacro:swerve_axle prefix="front_left" parent="swerve_chassis_link">
     <origin xyz="${axle_pos} ${axle_pos} ${axle_pos_z}" rpy="0 0 0" />
   </xacro:swerve_axle>
-  <xacro:swerve_axle prefix="${ns}_front_right" parent="${ns}_swerve_chassis_link">
+  <xacro:swerve_axle prefix="front_right" parent="swerve_chassis_link">
     <origin xyz="${axle_pos} -${axle_pos} ${axle_pos_z}" rpy="0 0 0" />
   </xacro:swerve_axle>
-  <xacro:swerve_axle prefix="${ns}_rear_left" parent="${ns}_swerve_chassis_link">
+  <xacro:swerve_axle prefix="rear_left" parent="swerve_chassis_link">
     <origin xyz="-${axle_pos} ${axle_pos} ${axle_pos_z} " rpy="0 0 0" />
   </xacro:swerve_axle>
-  <xacro:swerve_axle prefix="${ns}_rear_right" parent="${ns}_swerve_chassis_link">
+  <xacro:swerve_axle prefix="rear_right" parent="swerve_chassis_link">
     <origin xyz="-${axle_pos} -${axle_pos} ${axle_pos_z}" rpy="0 0 0" />
   </xacro:swerve_axle>
   <!-- Sensors -->
-  <xacro:zed_camera prefix="${ns}_zed" model="zed2i" parent="${ns}_swerve_chassis_link">
+  <xacro:zed_camera prefix="zed" model="zed2i" parent="swerve_chassis_link">
     <origin xyz="${cam_pos}" rpy="0 0 0" />
   </xacro:zed_camera>
-  <xacro:lidar prefix="${ns}_lidar" parent="${ns}_swerve_chassis_link" radius="0.035" length="0.025">
+  <xacro:lidar prefix="lidar" parent="swerve_chassis_link" radius="0.035" length="0.025">
     <origin xyz="0 0 .035" rpy="0 0 0" />
   </xacro:lidar>
-  <xacro:swerve_drive_control plugin="$(arg hw_interface_plugin)" ns="${ns}"/>
+  <xacro:swerve_drive_control plugin="$(arg hw_interface_plugin)"/>
 </robot>

Commit message: Added arm urdf  #23 (#66)
* added urdf stuff

* Small view change

---------

Co-authored-by: Gage Miller <gagemiller155@gmail.com>

File: src/edna_description/urdf/control/drive.xacro (robot description, xacro)
@@ -72,4 +72,60 @@
         <state_interface name="velocity"/>
       </joint>
+      <joint name="arm_roller_bar_joint">
+        <command_interface name="position">
+          <param name="min">-1</param>
+          <param name="max">1</param>
+        </command_interface>
+        <state_interface name="position"/>
+        <state_interface name="velocity"/>
+      </joint>
+      <joint name = "elevator_left_elevator_outer_1_joint" type = "revolute">
+          <command_interface name="position">
+            <param name="min">-1</param>
+            <param name="max">1</param>
+          </command_interface>
+          <state_interface name="position"/>
+          <state_interface name="velocity"/>
+      </joint>
+      <joint name = "elevator_left_elevator_center_joint" type = "prismatic">
+          <command_interface name="position">
+            <param name="min">-1</param>
+            <param name="max">1</param>
+          </command_interface>
+          <state_interface name="position"/>
+          <state_interface name="velocity"/>
+      </joint>
+      <joint name = "elevator_left_elevator_outer_2_joint" type = "prismatic">
+          <command_interface name="position">
+            <param name="min">-1</param>
+            <param name="max">1</param>
+          </command_interface>
+          <state_interface name="position"/>
+          <state_interface name="velocity"/>
+      </joint>
+      <joint name = "elevator_right_elevator_outer_1_joint" type = "revolute">
+          <command_interface name="position">
+            <param name="min">-1</param>
+            <param name="max">1</param>
+          </command_interface>
+          <state_interface name="position"/>
+          <state_interface name="velocity"/>
+      </joint>
+      <joint name = "elevator_right_elevator_center_joint" type = "prismatic">
+          <command_interface name="position">
+            <param name="min">-1</param>
+            <param name="max">1</param>
+          </command_interface>
+          <state_interface name="position"/>
+          <state_interface name="velocity"/>
+      </joint>
+      <joint name = "elevator_right_elevator_outer_2_joint" type = "prismatic">
+          <command_interface name="position">
+            <param name="min">-1</param>
+            <param name="max">1</param>
+          </command_interface>
+          <state_interface name="position"/>
+          <state_interface name="velocity"/>
+      </joint>
     </ros2_control>
   </xacro:macro>

File: src/edna_description/urdf/robots/edna.urdf.xacro (robot description, xacro)
@@ -10,5 +10,8 @@
   <xacro:include filename="$(find edna_description)/urdf/parts/swerve_axle.xacro" />
   <xacro:include filename="$(find edna_description)/urdf/parts/zed_macro.urdf.xacro" />
+  <xacro:include filename="$(find edna_description)/urdf/parts/elevator_leg.xacro" />
+  <xacro:include filename="$(find edna_description)/urdf/parts/back_leg.xacro" />
   <xacro:include filename="$(find edna_description)/urdf/parts/lidar.xacro" />
+  <xacro:include filename="$(find edna_description)/urdf/parts/elevator.xacro" />
   <!-- Axle Position Variables -->
   <xacro:property name="axle_pos" value="${301.625 / 1000}" />
@@ -44,4 +47,21 @@
     <origin xyz="0 0 .035" rpy="0 0 0" />
   </xacro:lidar>
+  <!-- Arm -->
+  <xacro:property name="elevator_leg_z" value="0.527"/>
+  <xacro:elevator_leg prefix="arm" parent="swerve_chassis_link">
+    <origin xyz = "0.1905 0 ${elevator_leg_z/2 + 0.03}" rpy = "0 0 0"/>
+  </xacro:elevator_leg>
+  <xacro:back_leg prefix="arm" parent="swerve_chassis_link">
+    <origin xyz = "-${chassis_length/2 - back_leg_length/2} 0 ${back_leg_height/2 + chassis_height}" rpy = "0 0 0" />
+  </xacro:back_leg>
+  <!--Right Elevator-->
+  <xacro:elevator prefix="elevator_right" parent="arm_back_leg_link" suffix="right">
+    <origin xyz = "0 ${-back_leg_width/2 - 0.04} ${back_leg_height/2 - 0.02}" rpy = "0 0 0" />
+  </xacro:elevator>
+  <!--Left Elevator-->
+  <xacro:elevator prefix="elevator_left" parent="arm_back_leg_link" suffix="left">
+    <origin xyz = "0 ${back_leg_width/2 + 0.04} ${back_leg_height/2 - 0.02}" rpy = "0 0 0" />
+  </xacro:elevator>
+  <!-- Control -->
   <xacro:swerve_drive_control plugin="$(arg hw_interface_plugin)"/>
 </robot>

Commit message: added gripper, merged elevator left/right

File: src/edna_description/urdf/control/drive.xacro (robot description, xacro)
@@ -80,5 +80,5 @@
         <state_interface name="velocity"/>
       </joint>
-      <joint name = "elevator_left_elevator_outer_1_joint" type = "revolute">
+      <joint name = "elevator_outer_1_joint" type = "revolute">
           <command_interface name="position">
             <param name="min">-1</param>
@@ -88,5 +88,5 @@
           <state_interface name="velocity"/>
       </joint>
-      <joint name = "elevator_left_elevator_center_joint" type = "prismatic">
+      <joint name = "elevator_center_joint" type = "prismatic">
           <command_interface name="position">
             <param name="min">0</param>
@@ -96,5 +96,5 @@
           <state_interface name="velocity"/>
       </joint>
-      <joint name = "elevator_left_elevator_outer_2_joint" type = "prismatic">
+      <joint name = "elevator_outer_2_joint" type = "prismatic">
           <command_interface name="position">
             <param name="min">-1</param>
@@ -104,5 +104,5 @@
           <state_interface name="velocity"/>
       </joint>
-      <joint name = "elevator_right_elevator_outer_1_joint" type = "revolute">
+      <joint name = "top_slider_joint" type = "prismatic">
           <command_interface name="position">
             <param name="min">-1</param>
@@ -112,5 +112,5 @@
           <state_interface name="velocity"/>
       </joint>
-      <joint name = "elevator_right_elevator_center_joint" type = "prismatic">
+      <joint name = "top_gripper_left_arm_joint" type = "revolute">
           <command_interface name="position">
             <param name="min">-1</param>
@@ -120,5 +120,5 @@
           <state_interface name="velocity"/>
       </joint>
-      <joint name = "elevator_right_elevator_outer_2_joint" type = "prismatic">
+      <joint name = "top_gripper_right_arm_joint" type = "prismatic">
           <command_interface name="position">
             <param name="min">-1</param>

File: src/edna_description/urdf/parts/elevator.xacro (robot description, xacro)
@@ -12,6 +12,6 @@
     <xacro:property name="elevator_outer_offset_z" value="0.07"/>
     <xacro:include filename="$(find edna_description)/urdf/parts/elevator_leg.xacro" />
-    <xacro:macro name = "elevator" params = "prefix parent *origin suffix">
-        <link name = "${prefix}_elevator_outer_1_link">
+    <xacro:macro name = "elevator" params = "prefix parent *origin">
+        <link name = "${prefix}_outer_1_link">
             <xacro:inertial_box mass = "1" x = "${elevator_outer_length}" y = "${elevator_outer_width}" z = "${elevator_outer_height}">
                 <origin xyz = "0 0 ${elevator_outer_height/2}" rpy = "0 0 0"/>
@@ -25,4 +25,11 @@
                 <material name = "blue"/>
             </visual>
+            <visual>
+                <origin xyz = "${elevator_outer_length/2 - 0.08} ${0.07+elevator_middle_distance} 0.062" rpy = "${pi} 0 0"/>
+                <geometry>
+                    <mesh filename="package://edna_description/meshes/elevator_outer_updated.stl" scale="0.001 0.001 0.001"/>
+                </geometry>
+                <material name = "blue"/>
+            </visual>
             <collision>
                 <origin xyz = "${elevator_outer_length/2 - 0.0104} -0.0025 0.023" rpy = "0 0 0"/>
@@ -31,8 +38,14 @@
                 </geometry>
             </collision>
+            <collision>
+                <origin xyz = "${elevator_outer_length/2 - 0.0104} ${-0.0025+elevator_middle_distance} 0.023" rpy = "0 0 0"/>
+                <geometry>
+                    <box size = "${elevator_outer_length + 0.0004} ${elevator_outer_width + 0.0004} ${elevator_outer_height+0.002}"/>
+                </geometry>
+            </collision>
         </link>
-        <joint name = "${prefix}_elevator_outer_1_joint" type = "revolute">
+        <joint name = "${prefix}_outer_1_joint" type = "revolute">
             <parent link = "${parent}"/>
-            <child link = "${prefix}_elevator_outer_1_link"/>
+            <child link = "${prefix}_outer_1_link"/>
             <axis xyz = "0 -1 0"/>
             <limit effort="1000.0" lower="0.0" upper="0.548" velocity="0.5"/>
@@ -40,5 +53,5 @@
             <xacro:insert_block name = "origin"/>
         </joint>
-        <link name = "${prefix}_elevator_center_link">
+        <link name = "${prefix}_center_link">
             <xacro:inertial_box mass = "1" x = "${elevator_outer_length}" y = "${elevator_outer_width}" z = "${elevator_outer_height}">
                 <origin xyz = "0 0 ${elevator_outer_height/2}" rpy = "0 0 0"/>
@@ -46,4 +59,11 @@
             <visual>
                 <origin xyz = "${0.265+elevator_center_offset_x} 0.004 ${-0.085+elevator_center_offset_z}" rpy = "0 0 ${pi}"/>
+                <geometry>
+                    <mesh filename="package://edna_description/meshes/elevator_center.stl" scale="0.001 0.001 0.001"/>
+                </geometry>
+                <material name = "blue"/>
+            </visual>
+            <visual>
+                <origin xyz = "${0.265+elevator_center_offset_x} ${0.004+elevator_middle_distance} ${-0.085+elevator_center_offset_z}" rpy = "0 0 ${pi}"/>
                 <geometry>
                     <mesh filename="package://edna_description/meshes/elevator_center.stl" scale="0.001 0.001 0.001"/>
@@ -58,16 +78,20 @@
                 <material name="ghost"/>
             </collision>
+            <collision>
+                <origin xyz = "${elevator_center_length/2 - 0.03} ${elevator_middle_distance} 0" rpy = "0 0 0"/>
+                <geometry>
+                    <box size = "${elevator_center_length + 0.01} ${elevator_center_width} ${elevator_center_height}"/>
+                </geometry>
+                <material name="ghost"/>
+            </collision>
         </link>
-        <joint name = "${prefix}_elevator_center_joint" type = "prismatic">
-            <parent link = "${prefix}_elevator_outer_1_link" joint = "${prefix}_elevator_outer_1_joint"/>
-            <child link = "${prefix}_elevator_center_link"/>
+        <joint name = "${prefix}_center_joint" type = "prismatic">
+            <parent link = "${prefix}_outer_1_link" joint = "${prefix}_outer_1_joint"/>
+            <child link = "${prefix}_center_link"/>
             <axis xyz = "1 0 0"/>
             <limit effort="1000.0" lower="0.0" upper="0.56" velocity="0.5"/>
-            <xacro:if value="${suffix == 'right'}">
-                <mimic joint = "elevator_left_elevator_center_joint" multiplier = "1" offset = "0"/>
-            </xacro:if>
             <origin xyz = "${0.1-elevator_center_offset_x} 0 ${elevator_center_offset_z}" rpy = "0 0 0"/>
         </joint>
-        <link name = "${prefix}_elevator_outer_2_link">
+        <link name = "${prefix}_outer_2_link">
             <xacro:inertial_box mass = "1" x = "${elevator_outer_length}" y = "${elevator_outer_width}" z = "${elevator_outer_height}">
                 <origin xyz = "0 0 ${elevator_outer_height/2}" rpy = "0 0 0"/>
@@ -81,4 +105,12 @@
                 <material name = "blue"/>
             </visual>
+            <visual>
+                <!-- <origin xyz = "${elevator_outer_offset_x+0.34} -0.07 ${-1*(elevator_outer_offset_z+0.015)}" rpy = "0 0 ${pi}"/> -->
+                 <origin xyz = "${elevator_outer_length/2 + 0.045} ${0.075+elevator_middle_distance} -0.06" rpy = "0 0 ${pi}"/>
+                <geometry>
+                    <mesh filename="package://edna_description/meshes/elevator_outer_updated.stl" scale="0.001 0.001 0.001"/>
+                </geometry>
+                <material name = "blue"/>
+            </visual>
             <collision>
                 <origin xyz = "${elevator_outer_length/2 - 0.025} 0 0" rpy = "0 0 ${pi}"/>
@@ -87,11 +119,17 @@
                 </geometry>
             </collision>
+            <collision>
+                <origin xyz = "${elevator_outer_length/2 - 0.025} ${elevator_middle_distance} 0" rpy = "0 0 ${pi}"/>
+                <geometry>
+                    <box size = "${elevator_outer_length + 0.025} ${elevator_outer_width} ${elevator_outer_height}"/>
+                </geometry>
+            </collision>
         </link>
-        <joint name = "${prefix}_elevator_outer_2_joint" type = "prismatic">
+        <joint name = "${prefix}_outer_2_joint" type = "prismatic">
             <axis xyz = "1 0 0"/>
             <limit effort="1000.0" lower="0.0" upper="0.568" velocity="0.5"/>
-            <parent link = "${prefix}_elevator_center_link"/>
-            <child link = "${prefix}_elevator_outer_2_link"/>
-            <mimic joint = "${prefix}_elevator_center_joint" multiplier = "1" offset = "0"/>
+            <parent link = "${prefix}_center_link"/>
+            <child link = "${prefix}_outer_2_link"/>
+            <mimic joint = "${prefix}_center_joint" multiplier = "1" offset = "0"/>
             <origin xyz = "${elevator_outer_offset_x} 0 ${elevator_outer_offset_z}" rpy = "0 0 0"/>
         </joint>

File: src/edna_description/urdf/parts/slider.xacro (robot description, xacro)
@@ -28,5 +28,5 @@
         <child link="${prefix}_slider_link"/>
         <axis xyz = "1 0 0"/>
-        <limit effort = "100.0" lower = "0" upper = "0.2" velocity = "1"/>
+        <limit effort = "100.0" lower = "0" upper = "0.4" velocity = "1"/>
     </joint>
     <xacro:gripper prefix="${prefix}" parent="${prefix}_slider_link">

File: src/edna_description/urdf/robots/edna.urdf.xacro (robot description, xacro)
@@ -59,15 +59,11 @@
     <origin xyz = "-${chassis_length/2 - each_leg_width * 2} 0 ${chassis_height}" rpy = "0 0 0" />
   </xacro:back_leg>
-  <!--Right Elevator-->
-  <xacro:elevator prefix="elevator_right" parent="arm_back_leg_link" suffix="right">
+  <!--Elevator-->
+  <xacro:elevator prefix="elevator" parent="arm_back_leg_link">
     <origin xyz = "-.03 -${elevator_middle_distance / 2} ${back_leg_height - .0215}" rpy = "0 0 0" />
   </xacro:elevator>
-  <!--Left Elevator-->
-  <xacro:elevator prefix="elevator_left" parent="arm_back_leg_link" suffix="left">
-    <origin xyz = "-.03 ${elevator_middle_distance / 2} ${back_leg_height - .0215}" rpy = "0 0 0" />
-  </xacro:elevator>
   <!-- Top Slider + Gripper -->
-  <xacro:property name= "slider_pos" value = "0.330 -${elevator_middle_distance / 2} ${slider_block_height/2}" />
-  <xacro:slider prefix="top" parent="elevator_left_elevator_outer_2_link">
+  <xacro:property name= "slider_pos" value = "0.330 ${elevator_middle_distance / 2} ${slider_block_height/2}" />
+  <xacro:slider prefix="top" parent="elevator_outer_2_link">
     <origin xyz = "${slider_pos}" rpy = "0 0 0" />
   </xacro:slider>

Commit message: gripper stuff

File: src/edna_description/urdf/control/drive.xacro (robot description, xacro)
@@ -128,4 +128,28 @@
           <state_interface name="velocity"/>
       </joint>
+       <joint name = "bottom_intake_joint" type = "revolute">
+          <command_interface name="position">
+            <param name="min">-1</param>
+            <param name="max">1</param>
+          </command_interface>
+          <state_interface name="position"/>
+          <state_interface name="velocity"/>
+      </joint>
+      <joint name = "bottom_gripper_left_arm_joint" type = "revolute">
+          <command_interface name="position">
+            <param name="min">-1</param>
+            <param name="max">1</param>
+          </command_interface>
+          <state_interface name="position"/>
+          <state_interface name="velocity"/>
+      </joint>
+      <joint name = "bottom_gripper_right_arm_joint" type = "prismatic">
+          <command_interface name="position">
+            <param name="min">-1</param>
+            <param name="max">1</param>
+          </command_interface>
+          <state_interface name="position"/>
+          <state_interface name="velocity"/>
+      </joint>
     </ros2_control>
   </xacro:macro>

File: src/edna_description/urdf/parts/intake.xacro (robot description, xacro)
@@ -17,5 +17,5 @@
         </visual>
         <collision>
-            <origin xyz = "${intake_block_length/2} 0 ${intake_block_height/2}" rpy = "0 0 0"/>
+            <origin xyz = "${intake_block_length/2 - 0.03} 0 0" rpy = "0 0 0"/>
             <geometry>
                 <box size="${intake_block_length} ${intake_block_width} ${intake_block_height}"/>
@@ -31,5 +31,5 @@
     </joint>
     <xacro:gripper prefix="${prefix}" parent="${prefix}_intake_link">
-        <origin xyz = "${intake_block_length - 0.1} 0 -0.035" rpy = "0 0 0" />
+        <origin xyz = "${intake_block_length - 0.05} 0 -0.035" rpy = "0 0 0" />
     </xacro:gripper>
   </xacro:macro>

File: src/edna_description/urdf/robots/edna.urdf.xacro (robot description, xacro)
@@ -70,5 +70,5 @@
   </xacro:slider>
   <!-- Bottom Intake + Gripper -->
-  <xacro:property name= "intake_pos" value = "0 0 -${elevator_leg_height/4}" />
+  <xacro:property name= "intake_pos" value = "0 0 -${elevator_leg_height/4 + 0.06}" />
   <xacro:intake prefix="bottom" parent="arm_elevator_leg_link">
     <origin xyz = "${intake_pos}" rpy = "0 0 0" />
