Commit message: Isaac arm (#77)
* initial commit

* joint_trajectory

* delete joint trajectory

* made publish trajectory msg file

* trajectory message publish fix

* I hate yamls

* yamls again

* i suddenly love yamls

* jjoint trajectory added to rosdep

* Cmake updated

* deleted .env finally

* now isaac isnt working...

* extension change

* fixed isaac drive

* fixed naming

* add gripper

* Added top slider and gripper

* updated real_hw_interface without gripper

* added gripper to real hw

* removed motion magic for elevator

* added gripper, merged elevator left/right

* adding joint trajectory publish to launch

* its working

* liam comitted

* removed lidar

* needs fixing

* updated stl

* bottom gripper

* dpad, gripper stuff

* bottom arm

* gripper stuff

* teleop

---------

Co-authored-by: SarangaR <sarnga.raj@gmail.com>
Co-authored-by: Kunwar Kalra <kkalra1003@gmail.com>
Co-authored-by: Gage Miller <gagemiller155@gmail.com>

File: src/edna_description/urdf/control/drive.xacro (robot description, xacro)
@@ -74,11 +74,11 @@
       <joint name="arm_roller_bar_joint">
         <command_interface name="position">
-          <param name="min">-1</param>
-          <param name="max">1</param>
+          <param name="min">0</param>
+          <param name="max">0.07</param>
         </command_interface>
         <state_interface name="position"/>
         <state_interface name="velocity"/>
       </joint>
-      <joint name = "elevator_left_elevator_outer_1_joint" type = "revolute">
+      <joint name = "elevator_outer_1_joint" type = "revolute">
           <command_interface name="position">
             <param name="min">-1</param>
@@ -88,5 +88,13 @@
           <state_interface name="velocity"/>
       </joint>
-      <joint name = "elevator_left_elevator_center_joint" type = "prismatic">
+      <joint name = "elevator_center_joint" type = "prismatic">
+          <command_interface name="position">
+            <param name="min">0</param>
+            <param name="max">0.56</param>
+          </command_interface>
+          <state_interface name="position"/>
+          <state_interface name="velocity"/>
+      </joint>
+      <joint name = "elevator_outer_2_joint" type = "prismatic">
           <command_interface name="position">
             <param name="min">-1</param>
@@ -96,5 +104,5 @@
           <state_interface name="velocity"/>
       </joint>
-      <joint name = "elevator_left_elevator_outer_2_joint" type = "prismatic">
+      <joint name = "top_slider_joint" type = "prismatic">
           <command_interface name="position">
             <param name="min">-1</param>
@@ -104,5 +112,5 @@
           <state_interface name="velocity"/>
       </joint>
-      <joint name = "elevator_right_elevator_outer_1_joint" type = "revolute">
+      <joint name = "top_gripper_left_arm_joint" type = "revolute">
           <command_interface name="position">
             <param name="min">-1</param>
@@ -112,5 +120,5 @@
           <state_interface name="velocity"/>
       </joint>
-      <joint name = "elevator_right_elevator_center_joint" type = "prismatic">
+      <joint name = "top_gripper_right_arm_joint" type = "prismatic">
           <command_interface name="position">
             <param name="min">-1</param>
@@ -120,5 +128,21 @@
           <state_interface name="velocity"/>
       </joint>
-      <joint name = "elevator_right_elevator_outer_2_joint" type = "prismatic">
+       <joint name = "bottom_intake_joint" type = "revolute">
+          <command_interface name="position">
+            <param name="min">-1</param>
+            <param name="max">1</param>
+          </command_interface>
+          <state_interface name="position"/>
+          <state_interface name="velocity"/>
+      </joint>
+      <joint name = "bottom_gripper_left_arm_joint" type = "revolute">
+          <command_interface name="position">
+            <param name="min">-1</param>
+            <param name="max">1</param>
+          </command_interface>
+          <state_interface name="position"/>
+          <state_interface name="velocity"/>
+      </joint>
+      <joint name = "bottom_gripper_right_arm_joint" type = "prismatic">
           <command_interface name="position">
             <param name="min">-1</param>

File: src/edna_description/urdf/parts/elevator_leg.xacro (robot description, xacro)
@@ -1,9 +1,9 @@
 <?xml version = "1.0"?>
 <robot xmlns:xacro = "http://www.ros.org/wiki/xacro">
-    <xacro:property name="elevator_leg_length" value="0.052" />
-    <xacro:property name="elevator_leg_width" value="0.330" />
-    <xacro:property name="elevator_leg_height" value="0.59" />
+    <xacro:property name="elevator_leg_length" value="0.0508" />
+    <xacro:property name="elevator_leg_width" value="0.3302" />
+    <xacro:property name="elevator_leg_height" value="0.5842" />
     <xacro:property name="roller_bar_length" value="0.0508" />
-    <xacro:property name="roller_bar_width" value="0.711" />
+    <xacro:property name="roller_bar_width" value="0.7112" />
     <!-- <xacro:property name="roller_bar_height" value="0.527" /> -->
     <xacro:property name="roller_bar_height" value="0.1" />
@@ -17,5 +17,5 @@
                 <origin xyz = "0 0 0" rpy = "0 0 0"/>
                 <geometry>
-                    <mesh filename="package://edna_description/meshes/elevator_legs.stl" scale="0.001 0.001 0.001"/>
+                    <mesh filename="package://edna_description/meshes/Front_Legs_V2.stl" scale="0.001 0.001 0.001"/>
                 </geometry>
                 <material name = "red"/>
@@ -38,7 +38,7 @@
             </xacro:inertial_box>
             <visual>
-                <origin xyz = "0 0 -0.19" rpy = "${pi/2} 0 0"/>
+                <origin xyz = "0 0 -0.24" rpy = "0 0 0"/>
                 <geometry>
-                    <mesh filename="package://edna_description/meshes/Roller_Bar.stl" scale="0.001 0.001 0.001"/>
+                    <mesh filename="package://edna_description/meshes/Roller_Bar_V2.stl" scale="0.001 0.001 0.001"/>
                 </geometry>
                 <material name = "red"/>

File: src/edna_description/urdf/robots/edna.urdf.xacro (robot description, xacro)
@@ -14,4 +14,7 @@
   <xacro:include filename="$(find edna_description)/urdf/parts/lidar.xacro" />
   <xacro:include filename="$(find edna_description)/urdf/parts/elevator.xacro" />
+  <xacro:include filename="$(find edna_description)/urdf/parts/gripper.xacro" />
+  <xacro:include filename="$(find edna_description)/urdf/parts/slider.xacro" />
+  <xacro:include filename="$(find edna_description)/urdf/parts/intake.xacro" />
   <!-- Axle Position Variables -->
   <xacro:property name="axle_pos" value="${301.625 / 1000}" />
@@ -21,5 +24,4 @@
   <!-- Camera Position Variables -->
   <xacro:property name="cam_pos" value="0.2 0 0.3"/> <!-- Made up values, replace with real ones later. -->
-  <xacro:property name="lidar_pos" value="0 0 0.035"/>
   <!-- X IS FORWARD -->
   <!-- Y IS LEFT -->
@@ -47,7 +49,7 @@
     <origin xyz="${cam_pos}" rpy="0 0 0" />
   </xacro:zed_camera>
-  <xacro:lidar prefix="lidar" parent="swerve_chassis_link" radius="0.035" length="0.025">
+  <!-- <xacro:lidar prefix="lidar" parent="swerve_chassis_link" radius="0.035" length="0.025">
     <origin xyz="${lidar_pos}" rpy="0 0 0" />
-  </xacro:lidar>
+  </xacro:lidar> -->
   <!-- Arm -->
   <xacro:property name="elevator_leg_z" value="0.527"/>
@@ -58,12 +60,18 @@
     <origin xyz = "-${chassis_length/2 - each_leg_width * 2} 0 ${chassis_height}" rpy = "0 0 0" />
   </xacro:back_leg>
-  <!--Right Elevator-->
-  <xacro:elevator prefix="elevator_right" parent="arm_back_leg_link" suffix="right">
+  <!--Elevator-->
+  <xacro:elevator prefix="elevator" parent="arm_back_leg_link">
     <origin xyz = "-.03 -${elevator_middle_distance / 2} ${back_leg_height - .0215}" rpy = "0 0 0" />
   </xacro:elevator>
-  <!--Left Elevator-->
-  <xacro:elevator prefix="elevator_left" parent="arm_back_leg_link" suffix="left">
-    <origin xyz = "-.03 ${elevator_middle_distance / 2} ${back_leg_height - .0215}" rpy = "0 0 0" />
-  </xacro:elevator>
+  <!-- Top Slider + Gripper -->
+  <xacro:property name= "slider_pos" value = "0.330 ${elevator_middle_distance / 2} ${slider_block_height/2}" />
+  <xacro:slider prefix="top" parent="elevator_outer_2_link">
+    <origin xyz = "${slider_pos}" rpy = "0 0 0" />
+  </xacro:slider>
+  <!-- Bottom Intake + Gripper -->
+  <xacro:property name= "intake_pos" value = "0 0 -${elevator_leg_height/4 + 0.06}" />
+  <xacro:intake prefix="bottom" parent="arm_elevator_leg_link">
+    <origin xyz = "${intake_pos}" rpy = "0 0 0" />
+  </xacro:intake>
   <!-- Control -->
   <xacro:swerve_drive_control plugin="$(arg hw_interface_plugin)"/>

Commit message: Add new and improved real drive hardware

File: src/edna_description/urdf/control/drive.xacro (robot description, xacro)
@@ -3,4 +3,5 @@
   <xacro:macro name="swerve_drive_control" params="plugin">
     <ros2_control name="swerve_drive" type="system">
+      <!-- USING A SINGLE HARDWARE INTERFACE TO REDUCE DDS AND THREAD LOAD ON RIO -->
       <hardware>
         <plugin>${plugin}</plugin>
@@ -8,68 +9,46 @@
         <param name="example_param_hw_stop_duration_sec">3.0</param>
       </hardware>
+      <!-- DRIVE TRAIN COMPONENTS -->
       <joint name="front_right_wheel_joint">
-        <command_interface name="velocity">
-          <param name="min">-1</param>
-          <param name="max">1</param>
-        </command_interface>
+        <command_interface name="velocity"/>
         <state_interface name="position"/>
         <state_interface name="velocity"/>
       </joint>
       <joint name="rear_left_wheel_joint">
-        <command_interface name="velocity">
-          <param name="min">-1</param>
-          <param name="max">1</param>
-        </command_interface>
+        <command_interface name="velocity"/>
         <state_interface name="position"/>
         <state_interface name="velocity"/>
       </joint>
       <joint name="front_left_wheel_joint">
-        <command_interface name="velocity">
-          <param name="min">-1</param>
-          <param name="max">1</param>
-        </command_interface>
+        <command_interface name="velocity"/>
         <state_interface name="position"/>
         <state_interface name="velocity"/>
       </joint>
       <joint name="rear_right_wheel_joint">
-        <command_interface name="velocity">
-          <param name="min">-1</param>
-          <param name="max">1</param>
-        </command_interface>
+        <command_interface name="velocity"/>
         <state_interface name="position"/>
         <state_interface name="velocity"/>
       </joint>
       <joint name="front_right_axle_joint">
-        <command_interface name="position">
-          <param name="min">-1</param>
-          <param name="max">1</param>
-        </command_interface>
+        <command_interface name="position"/>
         <state_interface name="position"/>
         <state_interface name="velocity"/>
       </joint>
       <joint name="rear_left_axle_joint">
-        <command_interface name="position">
-          <param name="min">-1</param>
-          <param name="max">1</param>
-        </command_interface>
+        <command_interface name="position"/>
         <state_interface name="position"/>
         <state_interface name="velocity"/>
       </joint>
       <joint name="front_left_axle_joint">
-        <command_interface name="position">
-          <param name="min">-1</param>
-          <param name="max">1</param>
-        </command_interface>
+        <command_interface name="position"/>
         <state_interface name="position"/>
         <state_interface name="velocity"/>
       </joint>
       <joint name="rear_right_axle_joint">
-        <command_interface name="position">
-          <param name="min">-1</param>
-          <param name="max">1</param>
-        </command_interface>
+        <command_interface name="position"/>
         <state_interface name="position"/>
         <state_interface name="velocity"/>
       </joint>
+      <!-- ARM COMPONENTS -->
       <joint name="arm_roller_bar_joint">
         <command_interface name="position">
@@ -79,6 +58,7 @@
         <state_interface name="position"/>
         <state_interface name="velocity"/>
+        <param name="arm_group">true</param>
       </joint>
-      <joint name = "elevator_outer_1_joint" type = "revolute">
+      <joint name = "elevator_outer_1_joint">
           <command_interface name="position">
             <param name="min">-1</param>
@@ -87,6 +67,8 @@
           <state_interface name="position"/>
           <state_interface name="velocity"/>
+          <param name="arm_group">true</param>
+          <param name="mimic">arm_roller_bar_joint</param>
       </joint>
-      <joint name = "elevator_center_joint" type = "prismatic">
+      <joint name = "elevator_center_joint">
           <command_interface name="position">
             <param name="min">0</param>
@@ -95,6 +77,7 @@
           <state_interface name="position"/>
           <state_interface name="velocity"/>
+          <param name="arm_group">true</param>
       </joint>
-      <joint name = "elevator_outer_2_joint" type = "prismatic">
+      <joint name = "elevator_outer_2_joint">
           <command_interface name="position">
             <param name="min">-1</param>
@@ -103,6 +86,7 @@
           <state_interface name="position"/>
           <state_interface name="velocity"/>
+          <param name="mimic">elevator_center_joint</param>
       </joint>
-      <joint name = "top_slider_joint" type = "prismatic">
+      <joint name = "top_slider_joint">
           <command_interface name="position">
             <param name="min">-1</param>
@@ -111,6 +95,8 @@
           <state_interface name="position"/>
           <state_interface name="velocity"/>
+          <param name="arm_group">true</param>
+          <param name="primary">true</param>
       </joint>
-      <joint name = "top_gripper_left_arm_joint" type = "revolute">
+      <joint name = "top_gripper_left_arm_joint">
           <command_interface name="position">
             <param name="min">-1</param>
@@ -119,6 +105,7 @@
           <state_interface name="position"/>
           <state_interface name="velocity"/>
+          <param name="arm_group">true</param>
       </joint>
-      <joint name = "top_gripper_right_arm_joint" type = "prismatic">
+      <joint name = "top_gripper_right_arm_joint">
           <command_interface name="position">
             <param name="min">-1</param>
@@ -127,6 +114,8 @@
           <state_interface name="position"/>
           <state_interface name="velocity"/>
+          <param name="arm_grouping">true</param>
+          <param name="mimic">top_gripper_left_arm_joint</param>
       </joint>
-       <joint name = "bottom_intake_joint" type = "revolute">
+       <joint name = "bottom_intake_joint">
           <command_interface name="position">
             <param name="min">-1</param>
@@ -135,6 +124,8 @@
           <state_interface name="position"/>
           <state_interface name="velocity"/>
+          <param name="arm_group">true</param>
+          <param name="primary">true</param>
       </joint>
-      <joint name = "bottom_gripper_left_arm_joint" type = "revolute">
+      <joint name = "bottom_gripper_left_arm_joint">
           <command_interface name="position">
             <param name="min">-1</param>
@@ -143,6 +134,7 @@
           <state_interface name="position"/>
           <state_interface name="velocity"/>
+          <param name="arm_group">true</param>
       </joint>
-      <joint name = "bottom_gripper_right_arm_joint" type = "prismatic">
+      <joint name = "bottom_gripper_right_arm_joint">
           <command_interface name="position">
             <param name="min">-1</param>
@@ -151,4 +143,6 @@
           <state_interface name="position"/>
           <state_interface name="velocity"/>
+          <param name="arm_group">true</param>
+          <param name="mimic">bottom_gripper_left_arm_joint</param>
       </joint>
     </ros2_control>

Commit message: tanush's macros (working in sim), BOTTOM GRIPPER IS GONE

File: src/edna_description/urdf/control/drive.xacro (robot description, xacro)
@@ -127,23 +127,4 @@
           <param name="primary">true</param>
       </joint>
-      <joint name = "bottom_gripper_left_arm_joint">
-          <command_interface name="position">
-            <param name="min">-1</param>
-            <param name="max">1</param>
-          </command_interface>
-          <state_interface name="position"/>
-          <state_interface name="velocity"/>
-          <param name="arm_group">true</param>
-      </joint>
-      <joint name = "bottom_gripper_right_arm_joint">
-          <command_interface name="position">
-            <param name="min">-1</param>
-            <param name="max">1</param>
-          </command_interface>
-          <state_interface name="position"/>
-          <state_interface name="velocity"/>
-          <param name="arm_group">true</param>
-          <param name="mimic">bottom_gripper_left_arm_joint</param>
-      </joint>
     </ros2_control>
   </xacro:macro>

File: src/edna_description/urdf/parts/intake.xacro (robot description, xacro)
@@ -30,7 +30,7 @@
         <limit effort = "100.0" lower = "0" upper = "1.42" velocity = "1"/>
     </joint>
-    <xacro:gripper prefix="${prefix}" parent="${prefix}_intake_link">
+    <!-- <xacro:gripper prefix="${prefix}" parent="${prefix}_intake_link">
         <origin xyz = "${intake_block_length - 0.05} 0 -0.035" rpy = "0 0 0" />
-    </xacro:gripper>
+    </xacro:gripper> -->
   </xacro:macro>
 </robot>
