Commit message: ZED Camera URDF - Moved ZED xacro and stl files into edna - Added the camera to the robot

File: src/edna_description/urdf/robots/edna.urdf.xacro (robot description, xacro)
@@ -9,7 +9,10 @@
   <xacro:include filename="$(find edna_description)/urdf/parts/square_chassis.xacro" />
   <xacro:include filename="$(find edna_description)/urdf/parts/swerve_axle.xacro" />
-    <!-- Axle Position Variables -->
-    <xacro:property name="axle_pos" value="${301.625 / 1000}" />
-    <xacro:property name="axle_pos_y" value="${69.056 / 1000}" />
+  <xacro:include filename="$(find edna_description)/urdf/parts/zed_macro.urdf.xacro" />
+  <!-- Axle Position Variables -->
+  <xacro:property name="axle_pos" value="${301.625 / 1000}" />
+  <xacro:property name="axle_pos_y" value="${69.056 / 1000}" />
+  <!-- Camera Position Variables -->
+  <xacro:property name="cam_pos" value=".3575 0.085 0.0"/> <!-- Made up values, replace with real ones later. -->
   <xacro:square_chassis prefix="swerve" />
   <xacro:swerve_axle prefix="front_left" parent="swerve_chassis_link">
@@ -25,4 +28,7 @@
     <origin xyz="-${axle_pos} ${axle_pos_y} -${axle_pos}" rpy="${pi / 2} 0 0" />
   </xacro:swerve_axle>
+  <xacro:zed_camera name="zed_camera" model="zed2i" parent="swerve_chassis_link">
+    <origin xyz="${cam_pos}" rpy="${pi/2} 0 0" />
+  </xacro:zed_camera>
   <xacro:swerve_drive_control plugin="$(arg hw_interface_plugin)" />
 </robot>

File: src/edna_description/urdf/util/materials.xacro (robot description, xacro)
@@ -31,3 +31,6 @@
     <color rgba="0.700 0.700 0.700 1.000" />
   </material>
+  <material name="zed2i_mat">
+    <color rgba="0.25 0.25 0.25 0.99"/>
+  </material>
 </robot>

File: src/zed_wrapper/urdf/zed_descr.urdf.xacro (robot description, xacro)
@@ -17,5 +17,5 @@
 <robot name="stereolabs_camera" xmlns:xacro="http://ros.org/wiki/xacro">
   <xacro:arg name="camera_name"   default="zed" />
-  <xacro:arg name="camera_model"  default="zed" />
+  <xacro:arg name="camera_model"  default="zed2i" />
   <xacro:arg name="base_frame"    default="base_link" />
   <xacro:arg name="cam_pos_x"     default="0.0" />

Commit message: Remove zed cam temp

File: src/edna_description/urdf/robots/edna.urdf.xacro (robot description, xacro)
@@ -31,7 +31,7 @@
     <origin xyz="-${axle_pos} -${axle_pos} ${axle_pos_z}" rpy="0 0 0" />
   </xacro:swerve_axle>
-  <xacro:zed_camera name="zed_camera" model="zed2i" parent="swerve_chassis_link">
-    <origin xyz="${cam_pos}" rpy="${pi/2} 0 0" />
-  </xacro:zed_camera>
+  <!-- <xacro:zed_camera name="zed_camera" model="zed2i" parent="swerve_chassis_link">
+    <origin xyz="${cam_pos}" rpy="0 0 0" />
+  </xacro:zed_camera>  -->
   <xacro:swerve_drive_control plugin="$(arg hw_interface_plugin)" />
 </robot>

Commit message: Fix isaac ext imu sensor

File: src/edna_description/urdf/robots/edna.urdf.xacro (robot description, xacro)
@@ -14,5 +14,5 @@
   <xacro:property name="axle_pos_z" value="${69.056 / 1000}" />
   <!-- Camera Position Variables -->
-  <xacro:property name="cam_pos" value=".3575 0.085 0.0"/> <!-- Made up values, replace with real ones later. -->
+  <xacro:property name="cam_pos" value="0 0 0.3"/> <!-- Made up values, replace with real ones later. -->
   <!-- X IS FORWARD -->
   <!-- Y IS LEFT -->
@@ -31,7 +31,7 @@
     <origin xyz="-${axle_pos} -${axle_pos} ${axle_pos_z}" rpy="0 0 0" />
   </xacro:swerve_axle>
-  <!-- <xacro:zed_camera name="zed_camera" model="zed2i" parent="swerve_chassis_link">
+  <xacro:zed_camera name="zed_camera" model="zed2i" parent="swerve_chassis_link">
     <origin xyz="${cam_pos}" rpy="0 0 0" />
-  </xacro:zed_camera>  -->
+  </xacro:zed_camera>
   <xacro:swerve_drive_control plugin="$(arg hw_interface_plugin)" />
 </robot>

Commit message: urdf for elevator

File: src/edna_description/urdf/robots/edna.urdf.xacro (robot description, xacro)
@@ -10,5 +10,7 @@
   <xacro:include filename="$(find edna_description)/urdf/parts/swerve_axle.xacro" />
   <xacro:include filename="$(find edna_description)/urdf/parts/zed_macro.urdf.xacro" />
-  <xacro:include filename="$(find edna_description)/urdf/parts/arm.xacro" />
+  <xacro:include filename="$(find edna_description)/urdf/parts/roller_bar.xacro" />
+  <xacro:include filename="$(find edna_description)/urdf/parts/elevator_leg.xacro" />
+  <xacro:include filename="$(find edna_description)/urdf/parts/back_leg.xacro" />
   <!-- Axle Position Variables -->
   <xacro:property name="axle_pos" value="${301.625 / 1000}" />
@@ -42,6 +44,12 @@
   </xacro:zed_camera>
   <xacro:swerve_drive_control plugin="$(arg hw_interface_plugin)" />
-  <xacro:arm prefix="arm" parent="swerve_chassis_link">
+  <xacro:roller_bar prefix="roller_bar" parent="swerve_chassis_link">
     <origin xyz="0 0 0" rpy="0 0 0" />
-  </xacro:arm>
+  </xacro:roller_bar>
+  <xacro:elevator_leg prefix="elevator_leg" parent="swerve_chassis_link">
+    <origin xyz="0 0 0" rpy="0 0 0" />
+  </xacro:elevator_leg>
+  <xacro:back_leg prefix="back_leg" parent="swerve_chassis_link">
+    <origin xyz="0 0 0" rpy="0 0 0" />
+  </xacro:back_leg>
 </robot>

Commit message: Mapping Works (somewhat) - Added footprint joint - Added `slam_toolbox` - Added a launch file for `slam_toolbox` - Reduced minimum radius of LiDAR and moved it up

File: src/edna_description/urdf/robots/edna.urdf.xacro (robot description, xacro)
@@ -43,6 +43,12 @@
     <origin xyz="${cam_pos}" rpy="0 0 0" />
   </xacro:zed_camera>
+  <link name="${ns}_footprint" />
+  <joint name="${ns}_footprint_joint" type="fixed">
+    <parent link="base_link" />
+    <child link="${ns}_footprint" />
+    <origin xyz="0 0 0" rpy="0 0 0" />
+  </joint>
   <xacro:lidar prefix="${ns}_lidar" parent="${ns}_swerve_chassis_link" radius="0.035" length="0.025">
-    <origin xyz="0 0 .035" rpy="0 0 0" />
+    <origin xyz="0 0 .065" rpy="0 0 0" />
   </xacro:lidar>
   <xacro:swerve_drive_control plugin="$(arg hw_interface_plugin)" ns="${ns}"/>

Commit message: it might work but every time i try to test it my computer crashes

File: src/edna_description/urdf/robots/edna.urdf.xacro (robot description, xacro)
@@ -22,6 +22,6 @@
   <!-- Z IS UP -->
   <!-- Chassis -->
-  <link name="base_link"></link>
-  <xacro:square_chassis prefix="${ns}_swerve" parent="base_link">
+  <link name="${ns}_base_link"></link>
+  <xacro:square_chassis prefix="${ns}_swerve" parent="${ns}_base_link">
     <origin xyz="0 0 0" rpy="0 0 0" />
   </xacro:square_chassis>
@@ -45,7 +45,7 @@
   <link name="${ns}_footprint" />
   <joint name="${ns}_footprint_joint" type="fixed">
-    <parent link="base_link" />
+    <parent link="${ns}_base_link" />
     <child link="${ns}_footprint" />
-    <origin xyz="0 0 0" rpy="0 0 0" />
+    <origin xyz="0 0 -0.0508" rpy="0 0 0" />
   </joint>
   <xacro:lidar prefix="${ns}_lidar" parent="${ns}_swerve_chassis_link" radius="0.035" length="0.025">

Commit message: Works (but the LiDAR is detecting the robot, meaning that some of the lidar beams are colliding with itself and screwing up SLAM)

File: src/edna_description/urdf/robots/edna.urdf.xacro (robot description, xacro)
@@ -45,6 +45,13 @@
   </xacro:zed_camera>
   <xacro:lidar prefix="lidar" parent="swerve_chassis_link" radius="0.035" length="0.025">
-    <origin xyz="0 0 .035" rpy="0 0 0" />
+    <origin xyz="0 0 .065" rpy="0 0 0" />
   </xacro:lidar>
+  <!-- Footprint (for Navigation) -->
+  <link name="base_footprint" />
+  <joint name="base_footprint_joint" type="fixed">
+    <parent link="base_link" />
+    <child link="base_footprint" />
+    <origin xyz="0 0 -0.0508" rpy="0 0 0" />
+  </joint>
   <!-- Arm -->
   <xacro:property name="elevator_leg_z" value="0.527"/>

Commit message: Move camera forward

File: src/edna_description/urdf/robots/edna.urdf.xacro (robot description, xacro)
@@ -20,5 +20,6 @@
   <xacro:property name= "chassis_side_width" value = ".0254" />
   <!-- Camera Position Variables -->
-  <xacro:property name="cam_pos" value="0 0 0.3"/> <!-- Made up values, replace with real ones later. -->
+  <xacro:property name="cam_pos" value="0.2 0 0.3"/> <!-- Made up values, replace with real ones later. -->
+  <xacro:property name="lidar_pos" value="0 0 0.035"/>
   <!-- X IS FORWARD -->
   <!-- Y IS LEFT -->
@@ -47,5 +48,5 @@
   </xacro:zed_camera>
   <xacro:lidar prefix="lidar" parent="swerve_chassis_link" radius="0.035" length="0.025">
-    <origin xyz="0 0 .035" rpy="0 0 0" />
+    <origin xyz="${lidar_pos}" rpy="0 0 0" />
   </xacro:lidar>
   <!-- Arm -->

Commit message: add gripper

File: src/edna_description/urdf/robots/edna.urdf.xacro (robot description, xacro)
@@ -14,4 +14,5 @@
   <xacro:include filename="$(find edna_description)/urdf/parts/lidar.xacro" />
   <xacro:include filename="$(find edna_description)/urdf/parts/elevator.xacro" />
+  <xacro:include filename="$(find edna_description)/urdf/parts/gripper.xacro" />
   <!-- Axle Position Variables -->
   <xacro:property name="axle_pos" value="${301.625 / 1000}" />
@@ -65,4 +66,8 @@
     <origin xyz = "-.03 ${elevator_middle_distance / 2} ${back_leg_height - .0215}" rpy = "0 0 0" />
   </xacro:elevator>
+  <!-- Top Gripper -->
+  <!-- <xacro:gripper prefix="top" parent="base_link">
+    <origin xyz = "0 0 0" rpy = "0 0 0" />
+  </xacro:gripper> -->
   <!-- Control -->
   <xacro:swerve_drive_control plugin="$(arg hw_interface_plugin)"/>

Commit message: IT WORKS

File: src/edna_description/urdf/robots/edna.urdf.xacro (robot description, xacro)
@@ -70,5 +70,5 @@
   </xacro:slider>
   <!-- Bottom Intake + Gripper -->
-  <xacro:property name= "intake_pos" value = "0 0 -${elevator_leg_height/4 + 0.06}" />
+  <xacro:property name= "intake_pos" value = "0 0 -${elevator_leg_height/4 + 0.01}" />
   <xacro:intake prefix="bottom" parent="arm_elevator_leg_link">
     <origin xyz = "${intake_pos}" rpy = "0 0 0" />

Commit message: Revert random changes that weren't in here a moment ago

File: src/edna_description/urdf/robots/edna.urdf.xacro (robot description, xacro)
@@ -70,5 +70,5 @@
   </xacro:slider>
   <!-- Bottom Intake + Gripper -->
-  <xacro:property name= "intake_pos" value = "0 0 -${elevator_leg_height/4 + 0.01}" />
+  <xacro:property name= "intake_pos" value = "0 0 -${elevator_leg_height/4 + 0.06}" />
   <xacro:intake prefix="bottom" parent="arm_elevator_leg_link">
     <origin xyz = "${intake_pos}" rpy = "0 0 0" />

Commit message: Move camera position up

File: src/edna_description/urdf/robots/edna.urdf.xacro (robot description, xacro)
@@ -23,5 +23,5 @@
   <xacro:property name= "chassis_side_width" value = ".0254" />
   <!-- Camera Position Variables -->
-  <xacro:property name="cam_pos" value="0.2 0 0.3"/> <!-- Made up values, replace with real ones later. -->
+  <xacro:property name="cam_pos" value="0.2 0 0.35"/> <!-- Made up values, replace with real ones later. -->
   <!-- X IS FORWARD -->
   <!-- Y IS LEFT -->
